File: pcb/v3/dac.kicad_sch (KiCad schematic)
At the start: 68 parts, among them U10 1, U11 OPA1622, U9 1, Y3 24.576MHz, Y4 24.576MHz

Commit message: up
Parts:
- removed C40, C41, C42, C43: 10pF, Capacitor_SMD:C_0402_1005Metric_Pad0.74x0.62mm_HandSolder, symbol Device:C
- removed CN1: ~, coloryr:AUDIO-TH_PJ-3136-B, symbol coloryr:PJ-3136-B
- removed R51, R52: 0, Resistor_SMD:R_0402_1005Metric_Pad0.72x0.64mm_HandSolder, symbol Device:R
- removed Y3, Y4: 24.576MHz, Crystal:Crystal_SMD_3225-4Pin_3.2x2.5mm_HandSoldering, symbol Oscillator:ECS-2520MV-xxx-xx
- added C79: 1uF, Capacitor_SMD:C_0402_1005Metric_Pad0.74x0.62mm_HandSolder, symbol Device:C
- added R11: 10K, Resistor_SMD:R_0402_1005Metric_Pad0.72x0.64mm_HandSolder, symbol Device:R
- U11: renamed from U9; value 1 -> CS43198
- U12: renamed from U10; value 1 -> CS43198
- renumbered C44 to C45, C45 to C46, C46 to C47, C47 to C48, C48 to C49, C49 to C50, C50 to C51, C51 to C52, C52 to C53, C53 to C54, C54 to C55, C55 to C56, C56 to C57, C57 to C58, C58 to C59, C59 to C60, C60 to C61, C61 to C62, C62 to C63, C63 to C64, C64 to C65, C65 to C66, C66 to C67, C67 to C68, C68 to C69, C69 to C70, C70 to C71, C71 to C72, C72 to C73, C73 to C74, C74 to C75, C75 to C76, C76 to C77, C77 to C78, CN2 to CN1, R47 to R57, R48 to R58, R49 to R59, R50 to R60, R53 to R61, R54 to R62, R55 to R63, R56 to R64, R57 to R65, R58 to R66, R59 to R67, R60 to R68, R61 to R69, R62 to R70, R63 to R71, R64 to R72, R65 to R73, R66 to R74, R67 to R75, R68 to R76, R69 to R77, U11 to U13
Connections:
- net 1.8V: now also R11.2
- net GND: now also R69.1, R70.1, C79.2
- net HP_DETECT: now also C79.1, R11.1
- net at CN1.3, R72.1: now also CN1.4 (3)
- net at CN1.2, R73.1: now also CN1.5
- net at R71.1: now also CN1.6; no longer CN1.4 (3)
- net DAC_INT: now reaches U12.27 (INT)
- net DAC_MCLK: now reaches U12.37 (XTI/MCLK)
- net DAC_MCLK: now also U11.37 (XTI/MCLK)
- net RESET renamed DAC_RESET
