File: pcb/v3/dac.kicad_sch (KiCad schematic)
At the start: 62 parts, among them U14 CS43198, U15 CS43198, U16 OPA1622

Commit message: up
Connections:
- net +INA: now also R70.2; no longer R68.2
- net +INB: now also R68.2; no longer R70.2
- net -INA: now also R69.2; no longer R67.2
- net -INB: now also R67.2; no longer R69.2
- net GND: no longer CN1.6
- net OUT_A: now also C76.1, R72.1, U16.7; no longer C75.1, R71.1, U16.9
- net OUT_B: now also C75.1, R71.1, U16.9; no longer C76.1, R72.1, U16.7
- net at CN1.2, PJ1.2, R77.1: no longer CN1.5
Changed lines of the file:
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@@
 	(paper "A4")
 	(junction
-		(at 242.57 38.1)
-		(diameter 0)
-		(color 0 0 0 0)
-	)
-	(junction
 		(at 168.91 59.69)
 		(diameter 0)
@@
 	)
 	(junction
-		(at 243.84 40.64)
-		(diameter 0)
-		(color 0 0 0 0)
-	)
-	(junction
 		(at 223.52 83.82)
 		(diameter 0)
@@
 	(wire
 		(pts
-			(xy 243.84 27.94) (xy 243.84 40.64)
-		)
-		(stroke
-			(width 0)
-			(type default)
-		)
-	)
-	(wire
-		(pts
 			(xy 113.03 187.96) (xy 113.03 190.5)
 		)
@@
 	(wire
 		(pts
-			(xy 242.57 30.48) (xy 242.57 38.1)
-		)
-		(stroke
-			(width 0)
-			(type default)
-		)
-	)
-	(wire
-		(pts
 			(xy 152.4 72.39) (xy 148.59 72.39)
 		)
@@
 	(wire
 		(pts
-			(xy 248.92 27.94) (xy 243.84 27.94)
-		)
-		(stroke
-			(width 0)
-			(type default)
-		)
-	)
-	(wire
-		(pts
 			(xy 74.93 31.75) (xy 74.93 34.29)
 		)
@@
 	(wire
 		(pts
-			(xy 242.57 30.48) (xy 248.92 30.48)
-		)
-		(stroke
-			(width 0)
-			(type default)
-		)
-	)
-	(wire
-		(pts
 			(xy 243.84 83.82) (xy 243.84 95.25)
 		)
@@
 		)
 	)
+	(global_label "+INA"
+		(shape input)
+		(at 209.55 128.27 180)
+		(fields_autoplaced yes)
+		(effects
+			(font
+				(size 1.27 1.27)
+			)
+			(justify right)
+		)
+		(property "Intersheetrefs" "${INTERSHEET_REFS}"
+			(at 201.9685 128.27 0)
+			(effects
+				(font
+					(size 1.27 1.27)
+				)
+				(justify right)
+				(hide yes)
+			)
+		)
+	)
 	(global_label "DAC_LRCK"
 		(shape input)
@@
 		)
 	)
+	(global_label "OUT_A"
+		(shape input)
+		(at 246.38 125.73 0)
+		(fields_autoplaced yes)
+		(effects
+			(font
+				(size 1.27 1.27)
+			)
+			(justify left)
+		)
+		(property "Intersheetrefs" "${INTERSHEET_REFS}"
+			(at 255.05 125.73 0)
+			(effects
+				(font
+					(size 1.27 1.27)
+				)
+				(justify left)
+				(hide yes)
+			)
+		)
+	)
 	(global_label "-INB"
 		(shape input)
@@
 		)
 	)
+	(global_label "-INB"
+		(shape input)
+		(at 209.55 92.71 180)
+		(fields_autoplaced yes)
+		(effects
+			(font
+				(size 1.27 1.27)
+			)
+			(justify right)
+		)
+		(property "Intersheetrefs" "${INTERSHEET_REFS}"
+			(at 201.7871 92.71 0)
+			(effects
+				(font
+					(size 1.27 1.27)
+				)
+				(justify right)
+				(hide yes)
+			)
+		)
+	)
 	(global_label "-INA"
 		(shape input)
@@
 		)
 	)
-	(global_label "-INA"
-		(shape input)
-		(at 209.55 92.71 180)
-		(fields_autoplaced yes)
-		(effects
-			(font
-				(size 1.27 1.27)
-			)
-			(justify right)
-		)
-		(property "Intersheetrefs" "${INTERSHEET_REFS}"
-			(at 201.9685 92.71 0)
-			(effects
-				(font
-					(size 1.27 1.27)
-				)
-				(justify right)
-				(hide yes)
-			)
-		)
-	)
 	(global_label "DAC_RESET"
 		(shape input)
@@
 		)
 	)
-	(global_label "-INB"
+	(global_label "DAC_SCL_1"
 		(shape input)
-		(at 209.55 123.19 180)
+		(at 77.47 86.36 180)
 		(fields_autoplaced yes)
 		(effects
@@
 		)
 		(property "Intersheetrefs" "${INTERSHEET_REFS}"
-			(at 201.7871 123.19 0)
+			(at 64.2039 86.36 0)
 			(effects
 				(font
@@
 		)
 	)
-	(global_label "DAC_SCL_1"
+	(global_label "DAC_MCLK_1"
 		(shape input)
-		(at 77.47 86.36 180)
+		(at 77.47 49.53 180)
 		(fields_autoplaced yes)
 		(effects
@@
 		)
 		(property "Intersheetrefs" "${INTERSHEET_REFS}"
-			(at 64.2039 86.36 0)
+			(at 62.692 49.53 0)
 			(effects
 				(font
@@
 		)
 	)
-	(global_label "+INA"
+	(global_label "+INB"
 		(shape input)
 		(at 209.55 97.79 180)
@@
 		)
 		(property "Intersheetrefs" "${INTERSHEET_REFS}"
-			(at 201.9685 97.79 0)
+			(at 201.7871 97.79 0)
 			(effects
 				(font
@@
 		)
 	)
-	(global_label "DAC_MCLK_1"
+	(global_label "REF_A"
 		(shape input)
-		(at 77.47 49.53 180)
+		(at 144.78 177.8 0)
 		(fields_autoplaced yes)
 		(effects
@@
 				(size 1.27 1.27)
 			)
-			(justify right)
+			(justify left)
 		)
 		(property "Intersheetrefs" "${INTERSHEET_REFS}"
-			(at 62.692 49.53 0)
+			(at 153.329 177.8 0)
 			(effects
 				(font
 					(size 1.27 1.27)
 				)
-				(justify right)
+				(justify left)
 				(hide yes)
 			)
 		)
 	)
-	(global_label "REF_A"
+	(global_label "OP+"
 		(shape input)
-		(at 144.78 177.8 0)
+		(at 255.27 138.43 0)
 		(fields_autoplaced yes)
 		(effects
@@
 		)
 		(property "Intersheetrefs" "${INTERSHEET_REFS}"
-			(at 153.329 177.8 0)
+			(at 262.4281 138.43 0)
 			(effects
 				(font
@@
 		)
 	)
-	(global_label "OP+"
+	(global_label "DAC_SDIN"
 		(shape input)
-		(at 255.27 138.43 0)
+		(at 77.47 63.5 180)
 		(fields_autoplaced yes)
 		(effects
@@
 				(size 1.27 1.27)
 			)
-			(justify left)
+			(justify right)
 		)
 		(property "Intersheetrefs" "${INTERSHEET_REFS}"
-			(at 262.4281 138.43 0)
+			(at 65.4738 63.5 0)
 			(effects
 				(font
 					(size 1.27 1.27)
 				)
-				(justify left)
+				(justify right)
 				(hide yes)
 			)
 		)
 	)
-	(global_label "DAC_SDIN"
+	(global_label "-INA"
 		(shape input)
-		(at 77.47 63.5 180)
+		(at 209.55 123.19 180)
 		(fields_autoplaced yes)
 		(effects
@@
 		)
 		(property "Intersheetrefs" "${INTERSHEET_REFS}"
-			(at 65.4738 63.5 0)
+			(at 201.9685 123.19 0)
 			(effects
 				(font
@@
 		)
 	)
-	(global_label "+INB"
-		(shape input)
-		(at 209.55 128.27 180)
-		(fields_autoplaced yes)
-		(effects
-			(font
-				(size 1.27 1.27)
-			)
-			(justify right)
-		)
-		(property "Intersheetrefs" "${INTERSHEET_REFS}"
-			(at 201.7871 128.27 0)
-			(effects
-				(font
-					(size 1.27 1.27)
-				)
-				(justify right)
-				(hide yes)
-			)
-		)
-	)
 	(global_label "DAC_INT_2"
 		(shape input)
@@
 	(global_label "OUT_B"
 		(shape input)
-		(at 246.38 125.73 0)
-		(fields_autoplaced yes)
-		(effects
-			(font
-				(size 1.27 1.27)
-			)
-			(justify left)
-		)
-		(property "Intersheetrefs" "${INTERSHEET_REFS}"
-			(at 255.2314 125.73 0)
-			(effects
-				(font
-					(size 1.27 1.27)
-				)
-				(justify left)
-				(hide yes)
-			)
-		)
-	)
-	(global_label "OUT_A"
-		(shape input)
 		(at 246.38 95.25 0)
 		(fields_autoplaced yes)
@@
 		)
 		(property "Intersheetrefs" "${INTERSHEET_REFS}"
-			(at 255.05 95.25 0)
+			(at 255.2314 95.25 0)
 			(effects
 				(font

Commit message: up
Parts:
- added R82: 12.7K, Resistor_SMD:R_0402_1005Metric_Pad0.72x0.64mm_HandSolder, symbol Device:R
- added R83: 22.6K, Resistor_SMD:R_0402_1005Metric_Pad0.72x0.64mm_HandSolder, symbol Device:R
Connections:
- net GND: now also R82.1
- net OP+: now also R83.1; no longer U16.8 (EN)
- new net: R82.2, R83.2, U16.8 (EN)
Other:
- moved on the sheet: C75, R67, R68, R71, U16A

Commit message: up
Parts:
- removed R82: 12.7K, Resistor_SMD:R_0402_1005Metric_Pad0.72x0.64mm_HandSolder, symbol Device:R
- removed R83: 22.6K, Resistor_SMD:R_0402_1005Metric_Pad0.72x0.64mm_HandSolder, symbol Device:R
Connections:
- net OUT_EN: now reaches U16.8 (EN)

Commit message: up
Parts:
- added R82: 22.6K, Resistor_SMD:R_0402_1005Metric_Pad0.72x0.64mm_HandSolder, symbol Device:R
- added R83: 12.7K, Resistor_SMD:R_0402_1005Metric_Pad0.72x0.64mm_HandSolder, symbol Device:R
Connections:
- net GND: now also R83.1
- net OP+: now also R82.1
- net OUT_EN: now also R82.2, R83.2

Commit message: up
Parts:
- removed R82: 22.6K, Resistor_SMD:R_0402_1005Metric_Pad0.72x0.64mm_HandSolder, symbol Device:R
- removed R83: 12.7K, Resistor_SMD:R_0402_1005Metric_Pad0.72x0.64mm_HandSolder, symbol Device:R
- added R84: 22.6K, Capacitor_SMD:C_0402_1005Metric_Pad0.74x0.62mm_HandSolder, symbol Device:R
- added R86: 12.7K, Capacitor_SMD:C_0402_1005Metric_Pad0.74x0.62mm_HandSolder, symbol Device:R
Connections:
- net GND: now also R86.1
- net OP+: now also R84.1
- net OUT_EN: now also R84.2, R86.2

Commit message: up
Parts:
- removed R93: 0, Resistor_SMD:R_0805_2012Metric, symbol Device:R
- added R87, R89: 10K, Capacitor_SMD:C_0402_1005Metric_Pad0.74x0.62mm_HandSolder, symbol Device:R
Connections:
- net GND: now also R87.2, R89.2; no longer PJ1.1
- net HP_TIP: now reaches CN1.3, PJ1.3, R76.1
- net HP_DET: now reaches PJ1.4, R80.1
- net HP_DET: now also R87.1
- net HP_RING2: now reaches PJ1.5
- net at CN1.4 (3), R75.1: now also R89.1
- net HP_DETECT_IO: now reaches CN1.6
- new net HP_SLEEVE: PJ1.1
Other:
- moved on the sheet: CN1, PJ1

Commit message: up
Parts:
- removed R75, R80: 0, Resistor_SMD:R_0805_2012Metric, symbol Device:R
- removed R89: 10K, Capacitor_SMD:C_0402_1005Metric_Pad0.74x0.62mm_HandSolder, symbol Device:R
- added C79: 10uF, Capacitor_SMD:C_0603_1608Metric_Pad1.08x0.95mm_HandSolder, symbol Device:C
Connections:
- net HP_DET is gone; now on net HP_DETECT_IO: PJ1.4, R87.1
- net HP_DETECT: now also CN1.6; no longer U14.22 (HP_DETECT)
- net HP_DETECT_IO: no longer CN1.6
- net HP_TIP: now also C79.2; no longer CN1.3, R76.1
- net DAC_INT_1: no longer names the net of U14.27 (INT)
- net DAC_INT_2: no longer names the net of U15.27 (INT)
- net HP_DETECT1: no longer names the net of U15.22 (HP_DETECT)
- new net: C79.1, CN1.3, R76.1

Commit message: up
Parts:
- added C36: 10uF, Capacitor_SMD:C_0603_1608Metric_Pad1.08x0.95mm_HandSolder, symbol Device:C
- added R55: 10K, Capacitor_SMD:C_0402_1005Metric_Pad0.74x0.62mm_HandSolder, symbol Device:R
Connections:
- net GND: now also R55.2
- net HP_DETECT_IO: no longer R87.1
- net HP_TIP: now also C79.1, R87.1; no longer C79.2
- net at CN1.3, R76.1: now also C79.2; no longer C79.1
- net at CN1.2, R77.1: now also C36.2; no longer PJ1.2
- new net: C36.1, PJ1.2, R55.1
Other:
- moved on the sheet: C79, R87
