File: pcb/v3/dac.kicad_sch (KiCad schematic)
At the start: 65 parts, among them U14 CS43198, U15 CS43198, U16 OPA1622

Commit message: pcb 3.9
Parts:
- C73, C77: value 1.0uF -> 1uF
Connections:
- net DAC_INT_A: now reaches U14.27 (INT)
- net DAC_INT_B: now reaches U15.27 (INT)
- net DAC_LRCK renamed DAC_LRCK_1
- net DAC_SCLK renamed DAC_SCLK_1
- net DAC_SDIN renamed DAC_SDIN_1
Changed lines of the file:
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@@
 	(wire
 		(pts
+			(xy 77.47 92.71) (xy 87.63 92.71)
+		)
+		(stroke
+			(width 0)
+			(type default)
+		)
+	)
+	(wire
+		(pts
 			(xy 134.62 148.59) (xy 151.13 148.59)
 		)
@@
 	(wire
 		(pts
+			(xy 76.2 180.34) (xy 86.36 180.34)
+		)
+		(stroke
+			(width 0)
+			(type default)
+		)
+	)
+	(wire
+		(pts
 			(xy 177.8 130.81) (xy 182.88 130.81)
 		)
@@
 		)
 	)
-	(global_label "DAC_LRCK"
+	(global_label "DAC_LRCK_1"
 		(shape input)
 		(at 77.47 66.04 180)
@@
 		)
 		(property "Intersheetrefs" "${INTERSHEET_REFS}"
-			(at 65.0505 66.04 0)
+			(at 62.8734 66.04 0)
 			(effects
 				(font
@@
 		)
 	)
+	(global_label "DAC_SDIN_1"
+		(shape input)
+		(at 76.2 151.13 180)
+		(fields_autoplaced yes)
+		(effects
+			(font
+				(size 1.27 1.27)
+			)
+			(justify right)
+		)
+		(property "Intersheetrefs" "${INTERSHEET_REFS}"
+			(at 62.0267 151.13 0)
+			(effects
+				(font
+					(size 1.27 1.27)
+				)
+				(justify right)
+				(hide yes)
+			)
+		)
+	)
 	(global_label "-INA"
 		(shape input)
@@
 		)
 	)
-	(global_label "DAC_SCL_1"
+	(global_label "DAC_LRCK_1"
 		(shape input)
-		(at 76.2 173.99 180)
+		(at 76.2 153.67 180)
 		(fields_autoplaced yes)
 		(effects
@@
 		)
 		(property "Intersheetrefs" "${INTERSHEET_REFS}"
-			(at 62.9339 173.99 0)
+			(at 61.6034 153.67 0)
 			(effects
 				(font
@@
 		)
 	)
-	(global_label "DAC_LRCK"
+	(global_label "DAC_SCL_1"
 		(shape input)
-		(at 76.2 153.67 180)
+		(at 76.2 173.99 180)
 		(fields_autoplaced yes)
 		(effects
@@
 		)
 		(property "Intersheetrefs" "${INTERSHEET_REFS}"
-			(at 63.7805 153.67 0)
+			(at 62.9339 173.99 0)
 			(effects
 				(font
@@
 		)
 	)
+	(global_label "DAC_INT_B"
+		(shape input)
+		(at 76.2 180.34 180)
+		(fields_autoplaced yes)
+		(effects
+			(font
+				(size 1.27 1.27)
+			)
+			(justify right)
+		)
+		(property "Intersheetrefs" "${INTERSHEET_REFS}"
+			(at 63.4781 180.34 0)
+			(effects
+				(font
+					(size 1.27 1.27)
+				)
+				(justify right)
+				(hide yes)
+			)
+		)
+	)
 	(global_label "DAC_RESET"
 		(shape input)
@@
 		)
 	)
-	(global_label "DAC_SDIN"
+	(global_label "REF_A"
 		(shape input)
-		(at 76.2 151.13 180)
+		(at 146.05 90.17 0)
 		(fields_autoplaced yes)
 		(effects
@@
 				(size 1.27 1.27)
 			)
-			(justify right)
+			(justify left)
 		)
 		(property "Intersheetrefs" "${INTERSHEET_REFS}"
-			(at 64.2038 151.13 0)
+			(at 154.599 90.17 0)
 			(effects
 				(font
 					(size 1.27 1.27)
 				)
-				(justify right)
+				(justify left)
 				(hide yes)
 			)
 		)
 	)
-	(global_label "REF_A"
+	(global_label "DAC_INT_A"
 		(shape input)
-		(at 146.05 90.17 0)
+		(at 77.47 92.71 180)
 		(fields_autoplaced yes)
 		(effects
@@
 				(size 1.27 1.27)
 			)
-			(justify left)
+			(justify right)
 		)
 		(property "Intersheetrefs" "${INTERSHEET_REFS}"
-			(at 154.599 90.17 0)
+			(at 64.9295 92.71 0)
 			(effects
 				(font
 					(size 1.27 1.27)
 				)
-				(justify left)
+				(justify right)
 				(hide yes)
 			)
@@
 		)
 	)
-	(global_label "DAC_SDIN"
+	(global_label "DAC_SDIN_1"
 		(shape input)
 		(at 77.47 63.5 180)
@@
 		)
 		(property "Intersheetrefs" "${INTERSHEET_REFS}"
-			(at 65.4738 63.5 0)
+			(at 63.2967 63.5 0)
 			(effects
 				(font
@@
 		)
 	)
-	(global_label "DAC_SCLK"
+	(global_label "OP-"
 		(shape input)
-		(at 76.2 156.21 180)
+		(at 207.01 138.43 180)
 		(fields_autoplaced yes)
 		(effects
@@
 		)
 		(property "Intersheetrefs" "${INTERSHEET_REFS}"
-			(at 63.841 156.21 0)
+			(at 199.8519 138.43 0)
 			(effects
 				(font
@@
 		)
 	)
-	(global_label "OP-"
+	(global_label "+INA"
 		(shape input)
-		(at 207.01 138.43 180)
+		(at 161.29 171.45 0)
 		(fields_autoplaced yes)
 		(effects
@@
 				(size 1.27 1.27)
 			)
-			(justify right)
+			(justify left)
 		)
 		(property "Intersheetrefs" "${INTERSHEET_REFS}"
-			(at 199.8519 138.43 0)
+			(at 168.8715 171.45 0)
 			(effects
 				(font
 					(size 1.27 1.27)
 				)
-				(justify right)
+				(justify left)
 				(hide yes)
 			)
 		)
 	)
-	(global_label "+INA"
+	(global_label "OP+"
 		(shape input)
-		(at 161.29 171.45 0)
+		(at 264.16 95.25 0)
 		(fields_autoplaced yes)
 		(effects
@@
 		)
 		(property "Intersheetrefs" "${INTERSHEET_REFS}"
-			(at 168.8715 171.45 0)
+			(at 271.3181 95.25 0)
 			(effects
 				(font
@@
 		)
 	)
-	(global_label "OP+"
+	(global_label "REF_B"
 		(shape input)
-		(at 264.16 95.25 0)
+		(at 209.55 26.67 180)
 		(fields_autoplaced yes)
 		(effects
@@
 				(size 1.27 1.27)
 			)
-			(justify left)
+			(justify right)
 		)
 		(property "Intersheetrefs" "${INTERSHEET_REFS}"
-			(at 271.3181 95.25 0)
+			(at 200.8196 26.67 0)
 			(effects
 				(font
 					(size 1.27 1.27)
 				)
-				(justify left)
+				(justify right)
 				(hide yes)
 			)
 		)
 	)
-	(global_label "REF_B"
+	(global_label "DAC_SCLK_1"
 		(shape input)
-		(at 209.55 26.67 180)
+		(at 76.2 156.21 180)
 		(fields_autoplaced yes)
 		(effects
@@
 		)
 		(property "Intersheetrefs" "${INTERSHEET_REFS}"
-			(at 200.8196 26.67 0)
+			(at 61.6639 156.21 0)
 			(effects
 				(font
@@
 		)
 	)
-	(global_label "DAC_SCLK"
+	(global_label "DAC_SCLK_1"
 		(shape input)
 		(at 77.47 68.58 180)
@@
 		)
 		(property "Intersheetrefs" "${INTERSHEET_REFS}"
-			(at 65.111 68.58 0)
+			(at 62.9339 68.58 0)
 			(effects
 				(font
@@
 			)
 		)
-		(property "Value" "1.0uF"
+		(property "Value" "1uF"
 			(at 208.788 142.24 0)
 			(effects
@@
 			)
 		)
-		(property "Value" "1.0uF"
+		(property "Value" "1uF"
 			(at 243.078 142.24 0)
 			(effects

Commit message: 3.11
Parts:
- PJ1: renamed from CN1; value ~ -> PJ-265G; footprint coloryr:AUDIO-TH_PJ-625G -> Connector_PinHeader_2.54mm:PinHeader_1x06_P2.54mm_Vertical
- PJ2: renamed from PJ1; value ~ -> PJ-327A; footprint coloryr:AUDIO-IN-SMD_PJ-327A_C22355751 -> Connector_PinHeader_2.54mm:PinHeader_1x05_P2.54mm_Vertical
Changed lines of the file:
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@@
 		(on_board yes)
 		(dnp no)
-		(fields_autoplaced yes)
-		(property "Reference" "PJ1"
-			(at 278.13 52.7049 0)
+		(property "Reference" "PJ2"
+			(at 268.732 43.18 0)
 			(effects
 				(font
@@
 			)
 		)
-		(property "Value" "~"
-			(at 278.13 54.61 0)
+		(property "Value" "PJ-327A"
+			(at 266.7 45.72 0)
 			(effects
 				(font
@@
 			)
 		)
-		(property "Footprint" "coloryr:AUDIO-IN-SMD_PJ-327A_C22355751"
+		(property "Footprint" "Connector_PinHeader_2.54mm:PinHeader_1x05_P2.54mm_Vertical"
 			(at 270.51 53.34 0)
 			(effects
@@
 			(project ""
 				(path "/9e6d55f4-a9e8-48fa-bb52-b4e4e3117f8b/8a8efada-1d6d-4bcc-828e-939af60bb626"
-					(reference "PJ1")
+					(reference "PJ2")
 					(unit 1)
 				)
@@
 		(on_board yes)
 		(dnp no)
-		(property "Reference" "CN1"
-			(at 276.86 33.6549 0)
+		(property "Reference" "PJ1"
+			(at 269.24 22.606 0)
 			(effects
 				(font
@@
 			)
 		)
-		(property "Value" "~"
-			(at 276.86 35.56 0)
+		(property "Value" "PJ-265G"
+			(at 267.208 25.0191 0)
 			(effects
 				(font
@@
 			)
 		)
-		(property "Footprint" "coloryr:AUDIO-TH_PJ-625G"
+		(property "Footprint" "Connector_PinHeader_2.54mm:PinHeader_1x06_P2.54mm_Vertical"
 			(at 268.986 42.418 0)
 			(effects
@@
 			(project "coloryr"
 				(path "/9e6d55f4-a9e8-48fa-bb52-b4e4e3117f8b/8a8efada-1d6d-4bcc-828e-939af60bb626"
-					(reference "CN1")
-					(unit 1)
-				)
+					(reference "PJ1")
+					(unit 1)
+				)
