File: pcb/v3/io.kicad_sch (KiCad schematic)
At the start: 43 parts, among them U7 STI9287

Commit message: up
Parts:
- added C31: 10uF, Capacitor_SMD:C_0402_1005Metric_Pad0.74x0.62mm_HandSolder, symbol Device:C
- added C32: 0.1uF, Capacitor_SMD:C_0402_1005Metric_Pad0.74x0.62mm_HandSolder, symbol Device:C
- added C33: 1uF, Capacitor_SMD:C_0402_1005Metric_Pad0.74x0.62mm_HandSolder, symbol Device:C
- added J10: Conn_01x05, Connector_PinHeader_2.00mm:PinHeader_1x05_P2.00mm_Vertical, symbol Connector_Generic:Conn_01x05
- added J14: Conn_01x04, Connector_PinHeader_2.00mm:PinHeader_1x04_P2.00mm_Vertical, symbol Connector_Generic:Conn_01x04
- added Q3: PNP, coloryr:SOT-23, symbol Simulation_SPICE:PNP
- added Q4: NPN, coloryr:SOT-23, symbol Simulation_SPICE:NPN
- added R27: 12K, Resistor_SMD:R_0402_1005Metric_Pad0.72x0.64mm_HandSolder, symbol Device:R
- added R34: 5.1K, Resistor_SMD:R_0402_1005Metric_Pad0.72x0.64mm_HandSolder, symbol Device:R
- added R36: 3K, Resistor_SMD:R_0402_1005Metric_Pad0.72x0.64mm_HandSolder, symbol Device:R
- added R37: 100, Resistor_SMD:R_0402_1005Metric_Pad0.72x0.64mm_HandSolder, symbol Device:R
- added R38, R40, R41: 100K, Resistor_SMD:R_0402_1005Metric_Pad0.72x0.64mm_HandSolder, symbol Device:R
- added R39: 10K, Resistor_SMD:R_0402_1005Metric_Pad0.72x0.64mm_HandSolder, symbol Device:R
- added R49, R50, R51: 4.7K, Capacitor_SMD:C_0402_1005Metric_Pad0.74x0.62mm_HandSolder, symbol Device:R
- added U8: CH334R, Package_SO:QSOP-16_3.9x4.9mm_P0.635mm, symbol Interface_USB:CH334R
- added Y1: 12M, Oscillator:Oscillator_SMD_ECS_2520MV-xxx-xx-4Pin_2.5x2.0mm, symbol Oscillator:ECS-2520MV-xxx-xx
- U7: renamed from U6; value ~ -> TCKE812
- renumbered C18 to C26, C19 to C27, C20 to C28, C22 to C29, C21 to C30, C23 to C34, C24 to C35, C25 to C36, C26 to C37, C27 to C38, D6 to D10, D7 to D11, D8 to D12, D9 to D13, D10 to D14, D11 to D15, D12 to D16, D4 to D8, D5 to D9, L2 to L4, R27 to R28, R28 to R29, R29 to R30, R30 to R31, R31 to R32, R32 to R33, R33 to R35, R34 to R42, R35 to R43, R36 to R44, R37 to R45, R38 to R46, R39 to R47, R40 to R48, R41 to R52, R42 to R53, R43 to R54, U7 to U9
Connections:
- net 3.3V: now also C31.2, C32.2, Q3.3 (E), R38.1, R49.1, R50.1, R51.1, U8.13 (VDD33)
- net 5V: now also C33.2, U8.12 (V5)
- net GND: now also C31.1, C32.1, C33.1, J10.1 (Pin_1), J14.1 (Pin_1), Q4.3 (E), R40.2, R41.2, U8.14 (GND), Y1.2 (GND), Y1.4 (VDD)
- net KEY_DOWN: now also J14.2 (Pin_2)
- net KEY_LEFT: now also J14.4 (Pin_4)
- net KEY_RIGHT: now also J14.3 (Pin_3)
- net USB1_DM: now also U8.10 (DMU-); no longer D14.2 (A2), USB2.2 (D-)
- net USB1_DP: now also U8.11 (DPU+); no longer D15.2 (A2), USB2.3 (D+)
- net LCD_X1: no longer names the net of P1.4 (VDD)
- net LCD_X2: no longer names the net of P1.2 (LED+)
- net LCD_Y1: no longer names the net of P1.3 (GND)
- net LCD_Y2: no longer names the net of P1.1 (LED-)
- net RESET renamed TP_RESET
- new net: J10.4 (Pin_4), R34.1, R36.2
- new net: J10.3 (Pin_3), R27.1, R34.2
- new net: Q4.2 (B), R39.2, R41.1
- new net: Q3.2 (B), Q4.1 (C), R38.2
- new net: J10.5 (Pin_5), R36.1, R37.2
- new net: J10.2 (Pin_2), R27.2
- new net: U8.15 (XO), Y1.3 (OUT)
- new net: U8.16 (XI), Y1.1 (Tri-State)
- new net BAT_INT: R51.2
- new net BAT_SCL: R50.2
- new net BAT_SDA: R49.2
- new net RECOVER: R37.1
- new net USBA_DM: D14.2 (A2), U8.7 (DM1-), USB2.2 (D-)
- new net USBA_DP: D15.2 (A2), U8.8 (DP1+), USB2.3 (D+)
- new net USBB_DM: U8.5 (DM2-)
- new net USBB_DP: U8.6 (DP2+)
- new net USB_DET: Q3.1 (C), R40.1
- new net VCC: R39.1
Other:
- note added: "KEY"
- note added: "USB_DET"
- note added: "USB_HUB"
- note added: "编码轮"
- moved on the sheet: C26, C27, C29, C36, C38, D14, D15, R35, U7, USB2
