File: pcb/v3/io.kicad_sch (KiCad schematic)
At the start: 57 parts, among them J12 Conn_01x04, J13 Conn_01x05, P1 LCD_MIPI, P2 LCD_TOUCH, U10 STI9287, U17 CH422E, Y1 24.576M

Commit message: up pcb v3.2
Connections:
- net 3.3V: no longer P1.14 (IOVCC)
- new net VCC_1V8_OUT: P1.14 (IOVCC)
Changed lines of the file:
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@@
 	)
 	(junction
-		(at 260.35 48.26)
-		(diameter 0)
-		(color 0 0 0 0)
-	)
-	(junction
 		(at 59.69 77.47)
 		(diameter 0)
@@
 	(wire
 		(pts
+			(xy 256.54 45.72) (xy 261.62 45.72)
+		)
+		(stroke
+			(width 0)
+			(type default)
+		)
+	)
+	(wire
+		(pts
 			(xy 217.17 33.02) (xy 213.36 33.02)
 		)
@@
 	(wire
 		(pts
-			(xy 260.35 45.72) (xy 260.35 48.26)
-		)
-		(stroke
-			(width 0)
-			(type default)
-		)
-	)
-	(wire
-		(pts
 			(xy 57.15 77.47) (xy 59.69 77.47)
 		)
@@
 	(wire
 		(pts
-			(xy 261.62 45.72) (xy 260.35 45.72)
-		)
-		(stroke
-			(width 0)
-			(type default)
-		)
-	)
-	(wire
-		(pts
 			(xy 224.79 33.02) (xy 227.33 33.02)
 		)
@@
 	(wire
 		(pts
-			(xy 260.35 48.26) (xy 261.62 48.26)
+			(xy 257.81 48.26) (xy 261.62 48.26)
 		)
 		(stroke
@@
 	(wire
 		(pts
-			(xy 257.81 48.26) (xy 260.35 48.26)
-		)
-		(stroke
-			(width 0)
-			(type default)
-		)
-	)
-	(wire
-		(pts
 			(xy 229.87 44.45) (xy 213.36 44.45)
 		)
@@
 	(wire
 		(pts
-			(xy 241.3 35.56) (xy 241.3 43.18)
+			(xy 241.3 35.56) (xy 241.3 36.83)
 		)
 		(stroke
@@
 		)
 	)
+	(global_label "VCC_1V8_OUT"
+		(shape input)
+		(at 256.54 45.72 180)
+		(fields_autoplaced yes)
+		(effects
+			(font
+				(size 1.27 1.27)
+			)
+			(justify right)
+		)
+		(property "Intersheetrefs" "${INTERSHEET_REFS}"
+			(at 240.8548 45.72 0)
+			(effects
+				(font
+					(size 1.27 1.27)
+				)
+				(justify right)
+				(hide yes)
+			)
+		)
+	)
 	(global_label "BAT_STAT"
 		(shape input)
@@
 	(symbol
 		(lib_id "power:GND")
-		(at 241.3 43.18 0)
+		(at 241.3 36.83 0)
 		(unit 1)
 		(exclude_from_sim no)
@@
 		(dnp no)
 		(property "Reference" "#PWR077"
-			(at 241.3 49.53 0)
+			(at 241.3 43.18 0)
 			(effects
 				(font
@@
 		)
 		(property "Value" "GND"
-			(at 239.268 46.99 0)
+			(at 239.268 40.64 0)
 			(effects
 				(font
@@
 		)
 		(property "Footprint" ""
-			(at 241.3 43.18 0)
+			(at 241.3 36.83 0)
 			(effects
 				(font
@@
 		)
 		(property "Datasheet" ""
-			(at 241.3 43.18 0)
+			(at 241.3 36.83 0)
 			(effects
 				(font
@@
 		)
 		(property "Description" "Power symbol creates a global label with name \"GND\" , ground"
-			(at 241.3 43.18 0)
+			(at 241.3 36.83 0)
 			(effects
 				(font

Commit message: up use new driver
Parts:
- added R12, R81: 0, Resistor_SMD:R_0402_1005Metric_Pad0.72x0.64mm_HandSolder, symbol Device:R
Connections:
- net 3.3V: now also R81.2
- net VCC_1V8_OUT: now also R12.2; no longer P1.14 (IOVCC)
- new net LCD_VDDIO: P1.14 (IOVCC), R12.1, R81.1
Other:
- moved on the sheet: C34, R52, R53

Commit message: up
Connections:
- net 3.3V: no longer C79.1, R88.2, U17.10 (VCC)
- net VCC: now also C79.1, R88.2, U17.10 (VCC)
Changed lines of the file:
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@@
 	)
 	(symbol
+		(lib_id "power:VCC")
+		(at 71.12 102.87 0)
+		(unit 1)
+		(exclude_from_sim no)
+		(in_bom yes)
+		(on_board yes)
+		(dnp no)
+		(fields_autoplaced yes)
+		(property "Reference" "#PWR058"
+			(at 71.12 106.68 0)
+			(effects
+				(font
+					(size 1.27 1.27)
+				)
+				(hide yes)
+			)
+		)
+		(property "Value" "VCC"
+			(at 71.12 97.79 0)
+			(effects
+				(font
+					(size 1.27 1.27)
+				)
+			)
+		)
+		(property "Footprint" ""
+			(at 71.12 102.87 0)
+			(effects
+				(font
+					(size 1.27 1.27)
+				)
+				(hide yes)
+			)
+		)
+		(property "Datasheet" ""
+			(at 71.12 102.87 0)
+			(effects
+				(font
+					(size 1.27 1.27)
+				)
+				(hide yes)
+			)
+		)
+		(property "Description" "Power symbol creates a global label with name \"VCC\""
+			(at 71.12 102.87 0)
+			(effects
+				(font
+					(size 1.27 1.27)
+				)
+				(hide yes)
+			)
+		)
+		(pin "1"
+		)
+		(instances
+			(project "coloryr"
+				(path "/9e6d55f4-a9e8-48fa-bb52-b4e4e3117f8b/d9c616e1-2298-455a-b24a-3007b8e9dd7b"
+					(reference "#PWR058")
+					(unit 1)
+				)
+			)
+		)
+	)
+	(symbol
 		(lib_id "Device:R")
 		(at 167.64 77.47 90)
@@
 	)
 	(symbol
-		(lib_id "power:VCC")
-		(at 31.75 105.41 90)
-		(unit 1)
-		(exclude_from_sim no)
-		(in_bom yes)
-		(on_board yes)
-		(dnp no)
-		(fields_autoplaced yes)
-		(property "Reference" "#PWR0133"
-			(at 35.56 105.41 0)
-			(effects
-				(font
-					(size 1.27 1.27)
-				)
-				(hide yes)
-			)
-		)
-		(property "Value" "3.3V"
-			(at 27.94 105.4099 90)
-			(effects
-				(font
-					(size 1.27 1.27)
-				)
-				(justify left)
-			)
-		)
-		(property "Footprint" ""
-			(at 31.75 105.41 0)
-			(effects
-				(font
-					(size 1.27 1.27)
-				)
-				(hide yes)
-			)
-		)
-		(property "Datasheet" ""
-			(at 31.75 105.41 0)
-			(effects
-				(font
-					(size 1.27 1.27)
-				)
-				(hide yes)
-			)
-		)
-		(property "Description" "Power symbol creates a global label with name \"VCC\""
-			(at 31.75 105.41 0)
-			(effects
-				(font
-					(size 1.27 1.27)
-				)
-				(hide yes)
-			)
-		)
-		(pin "1"
-		)
-		(instances
-			(project "coloryr"
-				(path "/9e6d55f4-a9e8-48fa-bb52-b4e4e3117f8b/d9c616e1-2298-455a-b24a-3007b8e9dd7b"
-					(reference "#PWR0133")
-					(unit 1)
-				)
-			)
-		)
-	)
-	(symbol
 		(lib_id "Device:R")
 		(at 241.3 104.14 270)
@@
 	)
 	(symbol
-		(lib_id "power:VCC")
-		(at 71.12 102.87 0)
+		(lib_id "Device:C")
+		(at 130.81 114.3 0)
 		(unit 1)
 		(exclude_from_sim no)
@@
 		(on_board yes)
 		(dnp no)
-		(fields_autoplaced yes)
-		(property "Reference" "#PWR0131"
-			(at 71.12 106.68 0)
+		(property "Reference" "C80"
+			(at 126.238 111.76 0)
 			(effects
 				(font
 					(size 1.27 1.27)
 				)
-				(hide yes)
+				(justify left)
 			)
 		)
-		(property "Value" "3.3V"
-			(at 71.12 97.79 0)
+		(property "Value" "0.1uF"
+			(at 131.826 116.84 0)
 			(effects
 				(font
 					(size 1.27 1.27)
 				)
+				(justify left)
 			)
 		)
-		(property "Footprint" ""
-			(at 71.12 102.87 0)
+		(property "Footprint" "Capacitor_SMD:C_0402_1005Metric_Pad0.74x0.62mm_HandSolder"
+			(at 131.7752 118.11 0)
 			(effects
 				(font
@@
 			)
 		)
-		(property "Datasheet" ""
-			(at 71.12 102.87 0)
+		(property "Datasheet" "~"
+			(at 130.81 114.3 0)
 			(effects
 				(font
@@
 			)
 		)
-		(property "Description" "Power symbol creates a global label with name \"VCC\""
-			(at 71.12 102.87 0)
+		(property "Description" "Unpolarized capacitor"
+			(at 130.81 114.3 0)
 			(effects
 				(font
@@
 			)
 		)
+		(pin "2"
+		)
 		(pin "1"
 		)
@@
 			(project "coloryr"
 				(path "/9e6d55f4-a9e8-48fa-bb52-b4e4e3117f8b/d9c616e1-2298-455a-b24a-3007b8e9dd7b"
-					(reference "#PWR0131")
+					(reference "C80")
 					(unit 1)
 				)
@@
 	)
 	(symbol
-		(lib_id "Device:C")
-		(at 130.81 114.3 0)
+		(lib_id "power:VCC")
+		(at 31.75 105.41 90)
 		(unit 1)
 		(exclude_from_sim no)
@@
 		(on_board yes)
 		(dnp no)
-		(property "Reference" "C80"
-			(at 126.238 111.76 0)
+		(fields_autoplaced yes)
+		(property "Reference" "#PWR061"
+			(at 35.56 105.41 0)
 			(effects
 				(font
 					(size 1.27 1.27)
 				)
-				(justify left)
+				(hide yes)
 			)
 		)
-		(property "Value" "0.1uF"
-			(at 131.826 116.84 0)
+		(property "Value" "VCC"
+			(at 27.94 105.4099 90)
 			(effects
 				(font
@@
 			)
 		)
-		(property "Footprint" "Capacitor_SMD:C_0402_1005Metric_Pad0.74x0.62mm_HandSolder"
-			(at 131.7752 118.11 0)
+		(property "Footprint" ""
+			(at 31.75 105.41 0)
 			(effects
 				(font
@@
 			)
 		)
-		(property "Datasheet" "~"
-			(at 130.81 114.3 0)
+		(property "Datasheet" ""
+			(at 31.75 105.41 0)
 			(effects
 				(font
@@
 			)
 		)
-		(property "Description" "Unpolarized capacitor"
-			(at 130.81 114.3 0)
+		(property "Description" "Power symbol creates a global label with name \"VCC\""
+			(at 31.75 105.41 0)
 			(effects
 				(font
@@
 			)
 		)
-		(pin "2"
-		)
 		(pin "1"
 		)
@@
 			(project "coloryr"
 				(path "/9e6d55f4-a9e8-48fa-bb52-b4e4e3117f8b/d9c616e1-2298-455a-b24a-3007b8e9dd7b"
-					(reference "C80")
+					(reference "#PWR061")
 					(unit 1)
 				)

Commit message: up
Parts:
- removed C79: 0.1uF, Capacitor_SMD:C_0402_1005Metric_Pad0.74x0.62mm_HandSolder, symbol Device:C
- removed R43: 4.7K, Capacitor_SMD:C_0402_1005Metric_Pad0.74x0.62mm_HandSolder, symbol Device:R
- removed R86, R87: 0, Resistor_SMD:R_0402_1005Metric_Pad0.72x0.64mm_HandSolder, symbol Device:R
- removed R88: 10K, Capacitor_SMD:C_0402_1005Metric_Pad0.74x0.62mm_HandSolder, symbol Device:R
- removed U17: CH422E, Package_SO:MSOP-10_3x3mm_P0.5mm, symbol coloryr:CH442E
Other:
- note removed: "USB_BAT_SWITCH"

Commit message: ?
Parts:
- added D4, D5: D, Diode_SMD:D_SOD-323_HandSoldering, symbol Device:D
- added J10: Conn_01x02, Connector_PinHeader_2.00mm:PinHeader_1x02_P2.00mm_Vertical, symbol Connector_Generic:Conn_01x02
- added Q1: NPN, coloryr:SOT-23, symbol Simulation_SPICE:NPN
- added Q2: PMOS, coloryr:SOT-23, symbol Simulation_SPICE:PMOS
- added R18, R19, R22: 10K, Resistor_SMD:R_0402_1005Metric_Pad0.72x0.64mm_HandSolder, symbol Device:R
- added R20: 100K/NC, Resistor_SMD:R_0402_1005Metric_Pad0.72x0.64mm_HandSolder, symbol Device:R
- added R21: 1K, Resistor_SMD:R_0402_1005Metric_Pad0.72x0.64mm_HandSolder, symbol Device:R
Connections:
- net 3.3V: now also R18.1
- net GND: now also J10.1 (Pin_1), Q1.3 (E), R20.1, R22.2
- new net: Q1.2 (B), R20.2, R21.2
- new net: D5.2 (A), Q1.1 (C), Q2.2 (G), R19.2
- new net: D4.1 (K), D5.1 (K), J10.2 (Pin_2)
- new net KEY_POWER: D4.2 (A), R18.2
- new net POWER_EN: Q2.1 (D), R22.1
- new net POWER_ON: R21.1
- new net SYS: Q2.3 (S), R19.1
Other:
- note added: "POWER_SWITCH"

Commit message: up
Parts:
- removed D4, D5: D, Diode_SMD:D_SOD-323_HandSoldering, symbol Device:D
- removed J10: Conn_01x02, Connector_PinHeader_2.00mm:PinHeader_1x02_P2.00mm_Vertical, symbol Connector_Generic:Conn_01x02
- removed Q1: NPN, coloryr:SOT-23, symbol Simulation_SPICE:NPN
- removed Q2: PMOS, coloryr:SOT-23, symbol Simulation_SPICE:PMOS
- removed R18, R19, R22: 10K, Resistor_SMD:R_0402_1005Metric_Pad0.72x0.64mm_HandSolder, symbol Device:R
- removed R20: 100K/NC, Resistor_SMD:R_0402_1005Metric_Pad0.72x0.64mm_HandSolder, symbol Device:R
- removed R21: 1K, Resistor_SMD:R_0402_1005Metric_Pad0.72x0.64mm_HandSolder, symbol Device:R
- added R43: 4.7K, Capacitor_SMD:C_0402_1005Metric_Pad0.74x0.62mm_HandSolder, symbol Device:R
Connections:
- net 3.3V: now also R43.1
- new net BAT_INT: R43.2
Other:
- note removed: "POWER_SWITCH"

Commit message: up
Connections:
- net GND: now also P1.MP, P2.MP
Other:
- moved on the sheet: C32, R12, R81, R91

Commit message: up
Parts:
- removed R89: 0, Resistor_SMD:R_0402_1005Metric_Pad0.72x0.64mm_HandSolder, symbol Device:R
- added C43: 10uF, Capacitor_SMD:C_0402_1005Metric_Pad0.74x0.62mm_HandSolder, symbol Device:C
- added C44: 0.1uF, Capacitor_SMD:C_0402_1005Metric_Pad0.74x0.62mm_HandSolder, symbol Device:C
- added R88, R92: 4.7K, Capacitor_SMD:C_0402_1005Metric_Pad0.74x0.62mm_HandSolder, symbol Device:R
- added U13: TS3A227E, Package_DFN_QFN:QFN-16-1EP_3x3mm_P0.5mm_EP1.675x1.675mm, symbol coloryr:TS3A227E
Connections:
- net 3.3V: now also C43.1, C44.1, R88.1, R92.1, U13.4 (VDD)
- net DAC_SCL: now also U13.9 (SCL)
- net DAC_SDA: now also U13.3 (SDA)
- net GND: now also C43.2, C44.2, U13.1 (GND), U13.11 (GNDA), U13.17 (GND), U13.2 (GND)
- new net HP_CONTROL: U13.6 (MICP)
- new net HP_DET: U13.15 (DET_TRIGGER)
- new net HP_DETECT_IO: R92.2
- new net HP_INT: R88.2, U13.13 (INT)
- new net HP_RING2: U13.12 (RING2), U13.7 (RING2_SENSE)
- new net HP_SLEEVE: U13.10 (SLEEVE), U13.8 (SLEEVE_SENSE)
- new net HP_TIP: U13.14 (TIP)
- new net MIC_GND: U13.5 (GND_SENSE)
Other:
- note added: "HP"
- moved on the sheet: C34, R34, R35, R36, R37, R38, R39, R40, R41, R42, R43, R52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
