File: pcb/v3/io.kicad_sch (KiCad schematic)
At the start: 58 parts, among them J12 Conn_01x04, J13 Conn_01x05, P1 LCD_MIPI, P2 LCD_TOUCH, U10 STI9287, U13 TS3A227E, Y1 24.576M

Commit message: up
Parts:
- removed R92: 4.7K, Capacitor_SMD:C_0402_1005Metric_Pad0.74x0.62mm_HandSolder, symbol Device:R
- added C35, C37: 0.1uF, Capacitor_SMD:C_0402_1005Metric_Pad0.74x0.62mm_HandSolder, symbol Device:C
- added Q3: NMOS, coloryr:SOT-23, symbol Simulation_SPICE:NMOS
- added R44, R93: 330K, Resistor_SMD:R_0402_1005Metric_Pad0.72x0.64mm_HandSolder, symbol Device:R
- added R54, R56: 3.3K, Capacitor_SMD:C_0402_1005Metric_Pad0.74x0.62mm_HandSolder, symbol Device:R
- added U11: TXS0102DCU, Package_SO:VSSOP-8_2.3x2mm_P0.5mm, symbol Logic_LevelTranslator:TXS0102DCU
Connections:
- net 1.8V: now also C35.1, R54.2, R56.2, U11.3 (VCCA), U11.6 (OE)
- net 3.3V: now also C37.1, R44.2, R93.2, U11.7 (VCCB)
- net DAC_SCL: now also U11.1 (B2)
- net DAC_SDA: now also U11.8 (B1)
- net GND: now also C35.2, C37.2, Q3.3 (S), U11.2 (GND)
- net HP_DETECT_IO: now also Q3.2 (G), R93.1
- net HP_DET renamed HP_DETECT1
- net HP_DETECT1: now also Q3.1 (D), R44.1
- new net DAC_SCL_1: R56.1, U11.4 (A2)
- new net DAC_SDA_1: R54.1, U11.5 (A1)
Other:
- note added: "LEVEL_TRANSLATOR"
- moved on the sheet: C80, R85, R90, Y1

Commit message: up
Parts:
- U13: footprint Package_DFN_QFN:QFN-16-1EP_3x3mm_P0.5mm_EP1.675x1.675mm -> Package_DFN_QFN:Texas_RVA_VQFN-16-1EP_3.5x3.5mm_P0.5mm_EP2.14x2.14mm
Changed lines of the file:
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@@
 			)
 		)
-		(property "Footprint" "Package_DFN_QFN:QFN-16-1EP_3x3mm_P0.5mm_EP1.675x1.675mm"
+		(property "Footprint" "Package_DFN_QFN:Texas_RVA_VQFN-16-1EP_3.5x3.5mm_P0.5mm_EP2.14x2.14mm"
 			(at 62.23 130.81 0)
 			(effects

Commit message: 123
Parts:
- added R80: 4.7K, Capacitor_SMD:C_0402_1005Metric_Pad0.74x0.62mm_HandSolder, symbol Device:R
Connections:
- net 3.3V: now also R80.1
- new net HP_DETECT: R80.2
Changed lines of the file:
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@@
 	)
 	(junction
+		(at 196.85 53.34)
+		(diameter 0)
+		(color 0 0 0 0)
+	)
+	(junction
 		(at 196.85 30.48)
 		(diameter 0)
@@
 	(wire
 		(pts
+			(xy 184.15 55.88) (xy 196.85 55.88)
+		)
+		(stroke
+			(width 0)
+			(type default)
+		)
+	)
+	(wire
+		(pts
 			(xy 184.15 27.94) (xy 196.85 27.94)
 		)
@@
 	(wire
 		(pts
+			(xy 167.64 55.88) (xy 176.53 55.88)
+		)
+		(stroke
+			(width 0)
+			(type default)
+		)
+	)
+	(wire
+		(pts
 			(xy 142.24 180.34) (xy 142.24 185.42)
 		)
@@
 	(wire
 		(pts
+			(xy 196.85 55.88) (xy 196.85 53.34)
+		)
+		(stroke
+			(width 0)
+			(type default)
+		)
+	)
+	(wire
+		(pts
 			(xy 64.77 76.2) (xy 64.77 77.47)
 		)
@@
 		)
 	)
+	(global_label "HP_DETECT"
+		(shape input)
+		(at 167.64 55.88 180)
+		(fields_autoplaced yes)
+		(effects
+			(font
+				(size 1.27 1.27)
+			)
+			(justify right)
+		)
+		(property "Intersheetrefs" "${INTERSHEET_REFS}"
+			(at 154.3135 55.88 0)
+			(effects
+				(font
+					(size 1.27 1.27)
+				)
+				(justify right)
+				(hide yes)
+			)
+		)
+	)
 	(global_label "HP_SLEEVE"
 		(shape input)
@@
 					(unit 1)
 				)
+			)
+		)
+	)
+	(symbol
+		(lib_id "Device:R")
+		(at 180.34 55.88 270)
+		(unit 1)
+		(exclude_from_sim no)
+		(in_bom yes)
+		(on_board yes)
+		(dnp no)
+		(property "Reference" "R80"
+			(at 187.452 54.864 90)
+			(effects
+				(font
+					(size 1.27 1.27)
+				)
+				(justify right)
+			)
+		)
+		(property "Value" "4.7K"
+			(at 193.04 54.864 90)
+			(effects
+				(font
+					(size 1.27 1.27)
+				)
+				(justify right)
+			)
+		)
+		(property "Footprint" "Capacitor_SMD:C_0402_1005Metric_Pad0.74x0.62mm_HandSolder"
+			(at 180.34 54.102 90)
+			(effects
+				(font
+					(size 1.27 1.27)
+				)
+				(hide yes)
+			)
+		)
+		(property "Datasheet" "~"
+			(at 180.34 55.88 0)
+			(effects
+				(font
+					(size 1.27 1.27)
+				)
+				(hide yes)
+			)
+		)
+		(property "Description" "Resistor"
+			(at 180.34 55.88 0)
+			(effects
+				(font
+					(size 1.27 1.27)
+				)
+				(hide yes)
+			)
+		)
+		(pin "2"
+		)
+		(pin "1"
+		)
+		(instances
+			(project "coloryr"
+				(path "/9e6d55f4-a9e8-48fa-bb52-b4e4e3117f8b/d9c616e1-2298-455a-b24a-3007b8e9dd7b"
+					(reference "R80")
+					(unit 1)
+				)

Commit message: pcb 3.9
Parts:
- U11: footprint Package_SO:VSSOP-8_2.3x2mm_P0.5mm -> Package_SON:X2SON-8_1.4x1mm_P0.35mm
Changed lines of the file:
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@@
 			)
 		)
-		(property "Footprint" "Package_SO:VSSOP-8_2.3x2mm_P0.5mm"
+		(property "Footprint" "Package_SON:X2SON-8_1.4x1mm_P0.35mm"
 			(at 171.45 140.97 0)
 			(effects

Commit message: pcb
Parts:
- added R100, R99: 4.7K, Capacitor_SMD:C_0402_1005Metric_Pad0.74x0.62mm_HandSolder, symbol Device:R
Connections:
- net 3.3V: now also R100.1, R99.1
- new net DAC_INT_A: R99.2
- new net DAC_INT_B: R100.2
Other:
- moved on the sheet: R34, R35, R36, R37, R38, R39, R40, R41, R42, R43, R80, R88

Commit message: 3.11
Parts:
- U11: footprint Package_SON:X2SON-8_1.4x1mm_P0.35mm -> Package_SO:VSSOP-8_2.3x2mm_P0.5mm
Changed lines of the file:
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@@
 			)
 		)
-		(property "Footprint" "Package_SON:X2SON-8_1.4x1mm_P0.35mm"
+		(property "Footprint" "Package_SO:VSSOP-8_2.3x2mm_P0.5mm"
 			(at 171.45 140.97 0)
 			(effects
