File: pcb/v3/power.kicad_sch (KiCad schematic)
At the start: 73 parts, among them J10 Conn_01x02, J11 TestPoint, J14 TestPoint, J4 Conn_01x02, J5 TestPoint, J6 TestPoint, J7 TestPoint, J8 TestPoint, J9 Conn_01x02, Q1 NPN, Q2 PMOS, U2 TLV6213x, U4 BQ25895RTW, U5 LM27762, U6 LP5907MFX-3.3, U7 TPS61230DRC

Commit message: up
Parts:
- removed R12: 10K, Capacitor_SMD:C_0402_1005Metric_Pad0.74x0.62mm_HandSolder, symbol Device:R
- C23: footprint Capacitor_SMD:C_0402_1005Metric_Pad0.74x0.62mm_HandSolder -> Capacitor_SMD:C_0603_1608Metric_Pad1.08x0.95mm_HandSolder
- R14: value 220K -> 510K
Connections:
- net BAT_STAT: now also U4.24 (DSEL); no longer U4.4 (STAT)
- net GND: now also U5.1 (PGOOD)
- net at R13.2, U5.2 (FB+): now also RV1.3; no longer RV1.1
Other:
- moved on the sheet: RV1
Changed lines of the file:
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@@
 	)
 	(junction
-		(at 35.56 100.33)
-		(diameter 0)
-		(color 0 0 0 0)
-	)
-	(junction
 		(at 82.55 104.14)
 		(diameter 0)
@@
 	(wire
 		(pts
-			(xy 41.91 100.33) (xy 35.56 100.33)
+			(xy 25.4 100.33) (xy 41.91 100.33)
 		)
 		(stroke
@@
 	(wire
 		(pts
-			(xy 35.56 100.33) (xy 25.4 100.33)
-		)
-		(stroke
-			(width 0)
-			(type default)
-		)
-	)
-	(wire
-		(pts
 			(xy 81.28 154.94) (xy 81.28 156.21)
 		)
@@
 	(wire
 		(pts
-			(xy 240.03 72.39) (xy 240.03 69.85)
+			(xy 36.83 105.41) (xy 43.18 105.41)
 		)
 		(stroke
@@
 	(wire
 		(pts
-			(xy 237.49 154.94) (xy 240.03 154.94)
+			(xy 240.03 72.39) (xy 240.03 69.85)
 		)
 		(stroke
@@
 	(wire
 		(pts
-			(xy 262.89 66.04) (xy 262.89 69.85)
+			(xy 237.49 154.94) (xy 240.03 154.94)
 		)
 		(stroke
@@
 	(wire
 		(pts
-			(xy 191.77 26.67) (xy 194.31 26.67)
+			(xy 262.89 66.04) (xy 262.89 69.85)
 		)
 		(stroke
@@
 	(wire
 		(pts
-			(xy 189.23 123.19) (xy 189.23 129.54)
+			(xy 191.77 26.67) (xy 194.31 26.67)
 		)
 		(stroke
@@
 	(wire
 		(pts
-			(xy 177.8 140.97) (xy 185.42 140.97)
+			(xy 189.23 123.19) (xy 189.23 129.54)
 		)
 		(stroke
@@
 	(wire
 		(pts
-			(xy 38.1 111.76) (xy 35.56 111.76)
+			(xy 177.8 140.97) (xy 185.42 140.97)
 		)
 		(stroke
@@
 	(wire
 		(pts
-			(xy 35.56 110.49) (xy 35.56 111.76)
-		)
-		(stroke
-			(width 0)
-			(type default)
-		)
-	)
-	(wire
-		(pts
 			(xy 71.12 64.77) (xy 71.12 66.04)
 		)
@@
 	(wire
 		(pts
-			(xy 43.18 105.41) (xy 38.1 105.41)
-		)
-		(stroke
-			(width 0)
-			(type default)
-		)
-	)
-	(wire
-		(pts
 			(xy 233.68 116.84) (xy 232.41 116.84)
 		)
@@
 	(wire
 		(pts
-			(xy 35.56 100.33) (xy 35.56 102.87)
-		)
-		(stroke
-			(width 0)
-			(type default)
-		)
-	)
-	(wire
-		(pts
 			(xy 237.49 104.14) (xy 240.03 104.14)
 		)
@@
 	(wire
 		(pts
+			(xy 162.56 125.73) (xy 165.1 125.73)
+		)
+		(stroke
+			(width 0)
+			(type default)
+		)
+	)
+	(wire
+		(pts
 			(xy 48.26 181.61) (xy 41.91 181.61)
 		)
@@
 	(wire
 		(pts
-			(xy 38.1 105.41) (xy 38.1 111.76)
+			(xy 49.53 130.81) (xy 53.34 130.81)
 		)
 		(stroke
@@
 	(wire
 		(pts
-			(xy 49.53 130.81) (xy 53.34 130.81)
+			(xy 182.88 49.53) (xy 182.88 52.07)
 		)
 		(stroke
@@
 	(wire
 		(pts
-			(xy 182.88 49.53) (xy 182.88 52.07)
+			(xy 93.98 170.18) (xy 93.98 171.45)
 		)
 		(stroke
@@
 	(wire
 		(pts
-			(xy 93.98 170.18) (xy 93.98 171.45)
+			(xy 71.12 120.65) (xy 66.04 120.65)
 		)
 		(stroke
@@
 	(wire
 		(pts
-			(xy 71.12 120.65) (xy 66.04 120.65)
+			(xy 163.83 129.54) (xy 170.18 129.54)
 		)
 		(stroke
@@
 	(wire
 		(pts
-			(xy 163.83 129.54) (xy 170.18 129.54)
+			(xy 248.92 140.97) (xy 251.46 140.97)
 		)
 		(stroke
@@
 	(wire
 		(pts
-			(xy 248.92 140.97) (xy 251.46 140.97)
+			(xy 107.95 44.45) (xy 115.57 44.45)
 		)
 		(stroke
@@
 	(wire
 		(pts
-			(xy 107.95 44.45) (xy 115.57 44.45)
+			(xy 162.56 133.35) (xy 161.29 133.35)
 		)
 		(stroke
@@
 	(wire
 		(pts
-			(xy 137.16 123.19) (xy 140.97 123.19)
-		)
-		(stroke
-			(width 0)
-			(type default)
-		)
-	)
-	(wire
-		(pts
 			(xy 191.77 110.49) (xy 185.42 110.49)
 		)
@@
 	(wire
 		(pts
+			(xy 162.56 125.73) (xy 162.56 133.35)
+		)
+		(stroke
+			(width 0)
+			(type default)
+		)
+	)
+	(wire
+		(pts
 			(xy 153.67 52.07) (xy 176.53 52.07)
 		)
@@
 		)
 	)
-	(global_label "BAT_STAT"
-		(shape input)
-		(at 137.16 123.19 180)
-		(fields_autoplaced yes)
-		(effects
-			(font
-				(size 1.27 1.27)
-			)
-			(justify right)
-		)
-		(property "Intersheetrefs" "${INTERSHEET_REFS}"
-			(at 125.6477 123.19 0)
-			(effects
-				(font
-					(size 1.27 1.27)
-				)
-				(justify right)
-				(hide yes)
-			)
-		)
-	)
 	(global_label "OP+"
 		(shape input)
@@
 		)
 	)
+	(global_label "BAT_STAT"
+		(shape input)
+		(at 165.1 125.73 0)
+		(fields_autoplaced yes)
+		(effects
+			(font
+				(size 1.27 1.27)
+			)
+			(justify left)
+		)
+		(property "Intersheetrefs" "${INTERSHEET_REFS}"
+			(at 176.6123 125.73 0)
+			(effects
+				(font
+					(size 1.27 1.27)
+				)
+				(justify left)
+				(hide yes)
+			)
+		)
+	)
 	(global_label "DAC_3V3"
 		(shape input)
@@
 			)
 		)
-		(property "Value" "220K"
+		(property "Value" "510K"
 			(at 77.47 96.266 90)
 			(effects
@@
 			)
 		)
-		(property "Footprint" "Capacitor_SMD:C_0402_1005Metric_Pad0.74x0.62mm_HandSolder"
+		(property "Footprint" "Capacitor_SMD:C_0603_1608Metric_Pad1.08x0.95mm_HandSolder"
 			(at 42.8752 180.34 0)
 			(effects
@@
 	)
 	(symbol
+		(lib_id "power:GND")
+		(at 36.83 105.41 270)
+		(unit 1)
+		(exclude_from_sim no)
+		(in_bom yes)
+		(on_board yes)
+		(dnp no)
+		(fields_autoplaced yes)
+		(property "Reference" "#PWR053"
+			(at 30.48 105.41 0)
+			(effects
+				(font
+					(size 1.27 1.27)
+				)
+				(hide yes)
+			)
+		)
+		(property "Value" "GND"
+			(at 33.02 105.4099 90)
+			(effects
+				(font
+					(size 1.27 1.27)
+				)
+				(justify right)
+			)
+		)
+		(property "Footprint" ""
+			(at 36.83 105.41 0)
+			(effects
+				(font
+					(size 1.27 1.27)
+				)
+				(hide yes)
+			)
+		)
+		(property "Datasheet" ""
+			(at 36.83 105.41 0)
+			(effects
+				(font
+					(size 1.27 1.27)
+				)
+				(hide yes)
+			)
+		)
+		(property "Description" "Power symbol creates a global label with name \"GND\" , ground"
+			(at 36.83 105.41 0)
+			(effects
+				(font
+					(size 1.27 1.27)
+				)
+				(hide yes)
+			)
+		)
+		(pin "1"
+		)
+		(instances
+			(project "coloryr"
+				(path "/9e6d55f4-a9e8-48fa-bb52-b4e4e3117f8b/45b885e8-026d-42f0-9271-c60672108a75"
+					(reference "#PWR053")
+					(unit 1)
+				)
+			)
+		)
+	)
+	(symbol
 		(lib_id "Device:R")
 		(at 81.28 168.91 0)
@@
 	)
 	(symbol
-		(lib_id "Device:R")
-		(at 35.56 106.68 0)
-		(unit 1)
-		(exclude_from_sim no)
-		(in_bom yes)
-		(on_board yes)
-		(dnp no)
-		(property "Reference" "R12"
-			(at 33.274 106.934 90)
-			(effects
-				(font
-					(size 1.27 1.27)
-				)
-				(justify right)
-			)
-		)
-		(property "Value" "10K"
-			(at 33.274 101.6 90)
-			(effects
-				(font
-					(size 1.27 1.27)
-				)
-				(justify right)
-			)
-		)
-		(property "Footprint" "Capacitor_SMD:C_0402_1005Metric_Pad0.74x0.62mm_HandSolder"
-			(at 33.782 106.68 90)
-			(effects
-				(font
-					(size 1.27 1.27)
-				)
-				(hide yes)
-			)
-		)
-		(property "Datasheet" "~"
-			(at 35.56 106.68 0)
-			(effects
-				(font
-					(size 1.27 1.27)
-				)
-				(hide yes)
-			)
-		)
-		(property "Description" "Resistor"
-			(at 35.56 106.68 0)
-			(effects
-				(font
-					(size 1.27 1.27)
-				)
-				(hide yes)
-			)
-		)
-		(pin "2"
-		)
-		(pin "1"
-		)
-		(instances
-			(project "coloryr"
-				(path "/9e6d55f4-a9e8-48fa-bb52-b4e4e3117f8b/45b885e8-026d-42f0-9271-c60672108a75"
-					(reference "R12")
-					(unit 1)
-				)
-			)
-		)
-	)
-	(symbol
 		(lib_id "Connector_Generic:Conn_01x01")
 		(at 266.7 31.75 0)
@@
 	(symbol
 		(lib_id "Device:R_Potentiometer")
-		(at 72.39 105.41 90)
+		(at 72.39 105.41 270)
+		(mirror x)
 		(unit 1)
 		(exclude_from_sim no)

Commit message: up
Parts:
- U3: footprint Package_TO_SOT_SMD:SOT-23-5_HandSoldering -> Package_TO_SOT_SMD:SOT-23-5
Changed lines of the file:
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@@
 			)
 		)
-		(property "Footprint" "Package_TO_SOT_SMD:SOT-23-5_HandSoldering"
+		(property "Footprint" "Package_TO_SOT_SMD:SOT-23-5"
 			(at 233.68 40.386 0)
 			(effects

Commit message: up uac
Parts:
- added R82, R83: 5.1K, Capacitor_SMD:C_0402_1005Metric_Pad0.74x0.62mm_HandSolder, symbol Device:R
Connections:
- net GND: now also J9.1 (Pin_1), R82.1, R83.1; no longer J9.2 (Pin_2)
- net at USB1.A5 (CC): now also R82.2
- net at USB1.B5 (VCONN): now also R83.2
- net at C18.1, U4.13 (BAT), U4.14 (BAT): now also J9.2 (Pin_2); no longer J9.1 (Pin_1)
Other:
- moved on the sheet: J4

Commit message: up
Parts:
- removed R82, R83: 5.1K, Capacitor_SMD:C_0402_1005Metric_Pad0.74x0.62mm_HandSolder, symbol Device:R
- removed U4: BQ25895RTW, Package_DFN_QFN:Texas_RTW_WQFN-24-1EP_4x4mm_P0.5mm_EP2.7x2.7mm_ThermalVias, symbol Battery_Management:BQ25895RTW
- added C40: 10uF, Capacitor_SMD:C_0402_1005Metric_Pad0.74x0.62mm_HandSolder, symbol Device:C
- added D14: D, Diode_SMD:D_SOD-323_HandSoldering, symbol Device:D
- added Q3: NPN, coloryr:SOT-23, symbol Simulation_SPICE:NPN
- added R43: 10K, Resistor_SMD:R_0402_1005Metric_Pad0.72x0.64mm_HandSolder, symbol Device:R
- added U4: IP2315, Package_DFN_QFN:QFN-32-1EP_5x5mm_P0.5mm_EP3.3x3.3mm_ThermalVias, symbol coloryr:IP2315
- C15: value 1uF -> 22uF; footprint Capacitor_SMD:C_0402_1005Metric_Pad0.74x0.62mm_HandSolder -> Capacitor_SMD:C_0603_1608Metric_Pad1.08x0.95mm_HandSolder
- C16: value 47nF -> 22uF; footprint Capacitor_SMD:C_0402_1005Metric_Pad0.74x0.62mm_HandSolder -> Capacitor_SMD:C_0603_1608Metric_Pad1.08x0.95mm_HandSolder
- C17: value 4.7uF -> 22uF; footprint Capacitor_SMD:C_0402_1005Metric_Pad0.74x0.62mm_HandSolder -> Capacitor_SMD:C_0603_1608Metric_Pad1.08x0.95mm_HandSolder
- C18: value 10uF -> 22uF; footprint Capacitor_SMD:C_0402_1005Metric_Pad0.74x0.62mm_HandSolder -> Capacitor_SMD:C_0603_1608Metric_Pad1.08x0.95mm_HandSolder
- C19, C20: value 10uF -> 0.1uF
- R15: value 260 -> 51K
- R16: value 10K -> 100K
- R17: footprint Capacitor_SMD:C_0402_1005Metric_Pad0.74x0.62mm_HandSolder -> Resistor_SMD:R_0402_1005Metric_Pad0.72x0.64mm_HandSolder
Connections:
- net 3.3V: now also R43.1
- net BAT_SCL: now also U4.8 (LED1/SCK)
- net BAT_SDA: now also U4.9 (LED2/SDA)
- net GND: now also C15.1, C16.1, C18.1, R15.1, R16.1, C40.2, D14.2 (A), Q3.3 (E), U4.17 (GND), U4.31 (GND), U4.33 (GND); no longer C15.2, C18.2, C19.2, R15.2, R17.2
- net SYS: now also J9.2 (Pin_2), C40.1, U4.22 (BAT); no longer C19.1
- net VCC: now also U4.20 (VIN), U4.21 (VIN); no longer C15.1
- net CC2: now reaches USB1.B5 (VCONN)
- net CC2: now also U4.3 (CC2)
- net at L2.1: now also C19.1, D14.1 (K), U4.11 (LX), U4.12 (LX), U4.13 (LX), U4.14 (LX); no longer C16.2
- net CC1: now reaches USB1.A5 (CC)
- net CC1: now also U4.2 (CC1)
- net VSYS: now reaches C17.2
- net VSYS: now also C15.2, C16.2, C18.2, U4.18 (VSYS), U4.19 (VSYS), U4.6 (VSYS), U4.7 (VSYS); no longer R16.1
- net at R16.2: now also U4.27 (ICHGSET); no longer R17.1
- net USB_DM renamed USB0_DM
- net USB_DP renamed USB0_DP
- new net: C19.2, U4.15 (BST)
- new net: R15.2, U4.26 (NTC)
- new net: Q3.2 (B), R17.1
- new net HCHAG: Q3.1 (C), R43.2
- new net HLED: R17.2, U4.16 (HLED)

Commit message: ?
Parts:
- removed D14, D4, D5: D, Diode_SMD:D_SOD-323_HandSoldering, symbol Device:D
- removed J10: Conn_01x02, Connector_PinHeader_2.00mm:PinHeader_1x02_P2.00mm_Vertical, symbol Connector_Generic:Conn_01x02
- removed Q1, Q3: NPN, coloryr:SOT-23, symbol Simulation_SPICE:NPN
- removed Q2: PMOS, coloryr:SOT-23, symbol Simulation_SPICE:PMOS
- removed R18, R19, R22: 10K, Resistor_SMD:R_0402_1005Metric_Pad0.72x0.64mm_HandSolder, symbol Device:R
- removed R20: 100K/NC, Resistor_SMD:R_0402_1005Metric_Pad0.72x0.64mm_HandSolder, symbol Device:R
- removed R21: 1K, Resistor_SMD:R_0402_1005Metric_Pad0.72x0.64mm_HandSolder, symbol Device:R
- removed U4: IP2315, Package_DFN_QFN:QFN-32-1EP_5x5mm_P0.5mm_EP3.3x3.3mm_ThermalVias, symbol coloryr:IP2315
- added C43, C44: 22uF, Capacitor_SMD:C_0603_1608Metric_Pad1.08x0.95mm_HandSolder, symbol Device:C
- added C79: 0.1uF, Capacitor_SMD:C_0402_1005Metric_Pad0.74x0.62mm_HandSolder, symbol Device:C
- added R84: 5.24K, Capacitor_SMD:C_0402_1005Metric_Pad0.74x0.62mm_HandSolder, symbol Device:R
- added U4: BQ25792RQMR, coloryr:bq25792, symbol coloryr:BQ25792RQMR
- C15, C16: value 22uF -> 47nF; footprint Capacitor_SMD:C_0603_1608Metric_Pad1.08x0.95mm_HandSolder -> Capacitor_SMD:C_0402_1005Metric_Pad0.74x0.62mm_HandSolder
- C17: value 22uF -> 4.7uF; footprint Capacitor_SMD:C_0603_1608Metric_Pad1.08x0.95mm_HandSolder -> Capacitor_SMD:C_0402_1005Metric_Pad0.74x0.62mm_HandSolder
- C18: value 22uF -> 10uF; footprint Capacitor_SMD:C_0603_1608Metric_Pad1.08x0.95mm_HandSolder -> Capacitor_SMD:C_0402_1005Metric_Pad0.74x0.62mm_HandSolder
- C19: value 0.1uF -> 10uF
- C40: value 10uF -> 1nF
- R15: value 51K -> 3K
- R16: value 100K -> 127K
- R17: value 10K -> 100K; footprint Resistor_SMD:R_0402_1005Metric_Pad0.72x0.64mm_HandSolder -> Capacitor_SMD:C_0402_1005Metric_Pad0.74x0.62mm_HandSolder
- R43: value 10K -> 30.31K; footprint Resistor_SMD:R_0402_1005Metric_Pad0.72x0.64mm_HandSolder -> Capacitor_SMD:C_0402_1005Metric_Pad0.74x0.62mm_HandSolder
Connections:
- net HLED is gone; now on an unnamed net: R17.2
- net 3.3V: no longer R43.1
- net BAT_SCL: now also U4.14 (SCL)
- net BAT_SDA: now also U4.15 (SDA)
- net GND: now also C17.2, C19.1, C20.1, R17.1, R43.1, C43.2, C44.2, C79.2, U4.10 (ACDRV2), U4.11 (ACDRV1), U4.13 (CE#), U4.27 (GND); no longer C15.1, C16.1, C17.1, C20.2, R16.1
- net SYS: now also C43.1, C44.1, C79.1, U4.25 (SYS); no longer C20.1, C40.1, J9.2 (Pin_2), L2.2
- net VCC: now also C18.2, C19.2, C20.2, U4.2 (VBUS), U4.3 (VBUS)
- net at L2.1: now also C15.1, U4.28 (SW1); no longer C19.1
- net at R15.2: now also U4.20 (PROG)
- net at R16.2: now also U4.17 (ILIM_HIZ)
- net HCHAG: no longer names the net of R43.2
- net HCHAG: now also R84.2, U4.16 (TS)
- removed net VSYS: C15.2, C16.2, C17.2, C18.2
- new net: C17.1, R16.1, R84.1, U4.5 (REGN)
- new net: C40.1, U4.24 (SDRV)
- new net: J9.2 (Pin_2), U4.18 (BATP), U4.22 (BAT), U4.23 (BAT)
- new net: C16.1, U4.19 (BTST2)
- new net: C16.2, L2.2, U4.26 (SW2)
- new net: C15.2, U4.4 (BTST1)
- new net: U4.8 (VAC2), U4.9 (VAC1)
- new net BAT_INT: U4.21 (INT#)
- new net BAT_QON: U4.12 (QON#)
Other:
- note removed: "POWER_SWITCH"
- moved on the sheet: C21, C22, J14, J9, U6

Commit message: up
Parts:
- removed C40: 1nF, Capacitor_SMD:C_0402_1005Metric_Pad0.74x0.62mm_HandSolder, symbol Device:C
- removed C43, C44: 22uF, Capacitor_SMD:C_0603_1608Metric_Pad1.08x0.95mm_HandSolder, symbol Device:C
- removed C79: 0.1uF, Capacitor_SMD:C_0402_1005Metric_Pad0.74x0.62mm_HandSolder, symbol Device:C
- removed R43: 30.31K, Capacitor_SMD:C_0402_1005Metric_Pad0.74x0.62mm_HandSolder, symbol Device:R
- removed R84: 5.24K, Capacitor_SMD:C_0402_1005Metric_Pad0.74x0.62mm_HandSolder, symbol Device:R
- removed U4: BQ25792RQMR, coloryr:bq25792, symbol coloryr:BQ25792RQMR
- added D4, D5: D, Diode_SMD:D_SOD-323_HandSoldering, symbol Device:D
- added J10: Conn_01x02, Connector_PinHeader_2.00mm:PinHeader_1x02_P2.00mm_Vertical, symbol Connector_Generic:Conn_01x02
- added Q1: NPN, coloryr:SOT-23, symbol Simulation_SPICE:NPN
- added Q2: PMOS, coloryr:SOT-23, symbol Simulation_SPICE:PMOS
- added R18, R19, R22: 10K, Resistor_SMD:R_0402_1005Metric_Pad0.72x0.64mm_HandSolder, symbol Device:R
- added R20: 100K/NC, Resistor_SMD:R_0402_1005Metric_Pad0.72x0.64mm_HandSolder, symbol Device:R
- added R21: 1K, Resistor_SMD:R_0402_1005Metric_Pad0.72x0.64mm_HandSolder, symbol Device:R
- added R82, R83: 5.1K, Capacitor_SMD:C_0402_1005Metric_Pad0.74x0.62mm_HandSolder, symbol Device:R
- added U4: BQ25895RTW, Package_DFN_QFN:Texas_RTW_WQFN-24-1EP_4x4mm_P0.5mm_EP2.7x2.7mm_ThermalVias, symbol Battery_Management:BQ25895RTW
- C15: value 47nF -> 1uF
- C20: value 0.1uF -> 10uF
- R15: value 3K -> 260
- R16: value 127K -> 10K
- R17: value 100K -> 10K
Connections:
- net 3.3V: now also R18.1
- net BAT_INT: now also U4.7 (INT)
- net BAT_SCL: now also U4.5 (SCL)
- net BAT_SDA: now also U4.6 (SDA)
- net GND: now also C15.2, C17.1, C18.2, C19.2, C20.2, R15.2, R17.2, J10.1 (Pin_1), Q1.3 (E), R20.1, R22.2, R82.1, R83.1, U4.17 (PGND), U4.18 (PGND), U4.25 (PGND), U4.9 (~{CE}); no longer C17.2, C18.1, C19.1, C20.1, R15.1, R17.1
- net POWER_EN: now also Q2.1 (D), R22.1
- net SYS: now also C19.1, C20.1, L2.2, Q2.3 (S), R19.1, U4.15 (SYS), U4.16 (SYS)
- net VCC: now also C15.1, U4.1 (VBUS); no longer C18.2, C19.2, C20.2
- net at R16.2: now also R17.1, U4.11 (TS); no longer R17.2
- net at R16.1: now also C17.2, U4.22 (REGN); no longer C17.1
- net at J9.2 (Pin_2): now also C18.1, U4.13 (BAT), U4.14 (BAT)
- net at C16.1: now also U4.21 (BTST)
- net at C16.2: now also L2.1, U4.19 (SW), U4.20 (SW); no longer L2.2
- net CC1: no longer names the net of USB1.A5 (CC)
- net CC1: now also R82.2
- net CC2: no longer names the net of USB1.B5 (VCONN)
- net CC2: now also R83.2
- new net: Q1.2 (B), R20.2, R21.2
- new net: R15.1, U4.10 (ILIM)
- new net: D5.2 (A), Q1.1 (C), Q2.2 (G), R19.2
- new net: D4.1 (K), D5.1 (K), J10.2 (Pin_2)
- new net KEY_POWER: D4.2 (A), R18.2
- new net POWER_ON: R21.1
Other:
- note added: "POWER_SWITCH"
- moved on the sheet: C21, C22, J14, U6

Commit message: up
Parts:
- added C40: 100nF, Capacitor_SMD:C_0402_1005Metric_Pad0.74x0.62mm_HandSolder, symbol Device:C
- R20: value 100K/NC -> 10K
- RV1, RV2: footprint Potentiometer_THT:Potentiometer_Bourns_3266W_Vertical -> Potentiometer_SMD:Potentiometer_Bourns_TC33X_Vertical
Connections:
- net GND: no longer R22.2
- net SYS: now also C40.2; no longer C23.1, L3.1, U7.10 (VIN)
- net at Q2.2 (G), R19.2: now also R22.1, C40.1; no longer D5.2 (A), Q1.1 (C)
- net POWER_EN renamed POWER
- net POWER: now also C23.1, L3.1, U7.10 (VIN); no longer R22.1
- new net: D5.2 (A), Q1.1 (C), R22.2
Other:
- moved on the sheet: D4, D5, J10, Q1, Q2, R19

Commit message: 123
Parts:
- added R75: 10K, Resistor_SMD:R_0402_1005Metric_Pad0.72x0.64mm_HandSolder, symbol Device:R
Connections:
- net GND: now also R75.1
- net at D4.1 (K), D5.1 (K), J10.2 (Pin_2): now also R75.2
Changed lines of the file:
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@@
 	(wire
 		(pts
-			(xy 245.11 154.94) (xy 245.11 153.67)
-		)
-		(stroke
-			(width 0)
-			(type default)
-		)
-	)
-	(wire
-		(pts
 			(xy 49.53 151.13) (xy 49.53 161.29)
 		)
@@
 	(wire
 		(pts
-			(xy 236.22 154.94) (xy 245.11 154.94)
+			(xy 236.22 154.94) (xy 248.92 154.94)
 		)
 		(stroke
@@
 	(wire
 		(pts
-			(xy 248.92 153.67) (xy 248.92 152.4)
+			(xy 248.92 154.94) (xy 248.92 152.4)
 		)
 		(stroke
@@
 	(wire
 		(pts
-			(xy 245.11 153.67) (xy 248.92 153.67)
+			(xy 170.18 149.86) (xy 170.18 151.13)
 		)
 		(stroke
@@
 	(wire
 		(pts
-			(xy 170.18 149.86) (xy 170.18 151.13)
+			(xy 48.26 181.61) (xy 41.91 181.61)
 		)
 		(stroke
@@
 	(wire
 		(pts
-			(xy 48.26 181.61) (xy 41.91 181.61)
+			(xy 189.23 123.19) (xy 185.42 123.19)
 		)
 		(stroke
@@
 	(wire
 		(pts
-			(xy 189.23 123.19) (xy 185.42 123.19)
+			(xy 99.06 170.18) (xy 99.06 171.45)
 		)
 		(stroke
@@
 	(wire
 		(pts
-			(xy 99.06 170.18) (xy 99.06 171.45)
+			(xy 88.9 161.29) (xy 88.9 162.56)
 		)
 		(stroke
@@
 	(wire
 		(pts
-			(xy 88.9 161.29) (xy 88.9 162.56)
+			(xy 120.65 118.11) (xy 130.81 118.11)
 		)
 		(stroke
@@
 	(wire
 		(pts
-			(xy 120.65 118.11) (xy 130.81 118.11)
+			(xy 232.41 81.28) (xy 232.41 82.55)
 		)
 		(stroke
@@
 	(wire
 		(pts
-			(xy 232.41 81.28) (xy 232.41 82.55)
+			(xy 236.22 114.3) (xy 242.57 114.3)
 		)
 		(stroke
@@
 	(wire
 		(pts
+			(xy 250.19 114.3) (xy 254 114.3)
+		)
+		(stroke
+			(width 0)
+			(type default)
+		)
+	)
+	(wire
+		(pts
 			(xy 49.53 130.81) (xy 53.34 130.81)
 		)
@@
 	(symbol
 		(lib_id "Device:R")
+		(at 246.38 114.3 270)
+		(unit 1)
+		(exclude_from_sim no)
+		(in_bom yes)
+		(on_board yes)
+		(dnp no)
+		(property "Reference" "R75"
+			(at 248.412 116.586 90)
+			(effects
+				(font
+					(size 1.27 1.27)
+				)
+			)
+		)
+		(property "Value" "10K"
+			(at 243.586 116.586 90)
+			(effects
+				(font
+					(size 1.27 1.27)
+				)
+			)
+		)
+		(property "Footprint" "Resistor_SMD:R_0402_1005Metric_Pad0.72x0.64mm_HandSolder"
+			(at 246.38 112.522 90)
+			(effects
+				(font
+					(size 1.27 1.27)
+				)
+				(hide yes)
+			)
+		)
+		(property "Datasheet" "~"
+			(at 246.38 114.3 0)
+			(effects
+				(font
+					(size 1.27 1.27)
+				)
+				(hide yes)
+			)
+		)
+		(property "Description" "Resistor"
+			(at 246.38 114.3 0)
+			(effects
+				(font
+					(size 1.27 1.27)
+				)
+				(hide yes)
+			)
+		)
+		(pin "2"
+		)
+		(pin "1"
+		)
+		(instances
+			(project "coloryr"
+				(path "/9e6d55f4-a9e8-48fa-bb52-b4e4e3117f8b/45b885e8-026d-42f0-9271-c60672108a75"
+					(reference "R75")
+					(unit 1)
+				)
+			)
+		)
+	)
+	(symbol
+		(lib_id "Device:R")
 		(at 139.7 185.42 90)
 		(unit 1)
@@
 					(unit 1)
 				)
+			)
+		)
+	)
+	(symbol
+		(lib_id "power:GND")
+		(at 254 114.3 90)
+		(unit 1)
+		(exclude_from_sim no)
+		(in_bom yes)
+		(on_board yes)
+		(dnp no)
+		(property "Reference" "#PWR082"
+			(at 260.35 114.3 0)
+			(effects
+				(font
+					(size 1.27 1.27)
+				)
+				(hide yes)
+			)
+		)
+		(property "Value" "GND"
+			(at 258.064 116.332 0)
+			(effects
+				(font
+					(size 1.27 1.27)
+				)
+				(justify left)
+			)
+		)
+		(property "Footprint" ""
+			(at 254 114.3 0)
+			(effects
+				(font
+					(size 1.27 1.27)
+				)
+				(hide yes)
+			)
+		)
+		(property "Datasheet" ""
+			(at 254 114.3 0)
+			(effects
+				(font
+					(size 1.27 1.27)
+				)
+				(hide yes)
+			)
+		)
+		(property "Description" "Power symbol creates a global label with name \"GND\" , ground"
+			(at 254 114.3 0)
+			(effects
+				(font
+					(size 1.27 1.27)
+				)
+				(hide yes)
+			)
+		)
+		(pin "1"
+		)
+		(instances
+			(project "coloryr"
+				(path "/9e6d55f4-a9e8-48fa-bb52-b4e4e3117f8b/45b885e8-026d-42f0-9271-c60672108a75"
+					(reference "#PWR082")
+					(unit 1)
+				)
