File: pcb/v3/power.kicad_sch (KiCad schematic)
At the start: 76 parts, among them J10 Conn_01x02, J11 TestPoint, J14 TestPoint, J4 Conn_01x02, J5 TestPoint, J6 TestPoint, J7 TestPoint, J8 TestPoint, J9 Conn_01x02, Q1 NPN, Q2 PMOS, U2 TLV6213x, U4 BQ25895RTW, U5 LM27762, U6 LP5907MFX-3.3, U7 TPS61230DRC

Commit message: pcb 3.9
Parts:
- C40: value 100nF -> 0.1uF
- U3: value ~ -> RT9013
Changed lines of the file:
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@@
 		(dnp no)
 		(property "Reference" "U3"
-			(at 236.22 25.146 0)
-			(effects
-				(font
-					(size 1.27 1.27)
-				)
-			)
-		)
-		(property "Value" "~"
-			(at 238.76 25.4 0)
+			(at 238.506 25.146 0)
+			(effects
+				(font
+					(size 1.27 1.27)
+				)
+			)
+		)
+		(property "Value" "RT9013"
+			(at 238.506 27.686 0)
 			(effects
 				(font
@@
 					(size 1.27 1.27)
 				)
+				(hide yes)
 			)
 		)
@@
 			)
 		)
-		(property "Value" "100nF"
+		(property "Value" "0.1uF"
 			(at 257.048 133.35 0)
 			(effects

Commit message: 3.11
Parts:
- removed C7, C8: 22uF, Capacitor_SMD:C_0603_1608Metric_Pad1.08x0.95mm_HandSolder, symbol Device:C
- removed J11, J14, J5, J6: TestPoint, TestPoint:TestPoint_Pad_D1.0mm, symbol Connector_Generic:Conn_01x01
- removed L1: 2,2uH, Inductor_SMD:L_1008_2520Metric_Pad1.43x2.20mm_HandSolder, symbol Device:L
- removed R10: 750K, Capacitor_SMD:C_0402_1005Metric_Pad0.74x0.62mm_HandSolder, symbol Device:R
- removed R11: 240K, Capacitor_SMD:C_0402_1005Metric_Pad0.74x0.62mm_HandSolder, symbol Device:R
- removed U2: TLV6213x, Package_DFN_QFN:VQFN-16-1EP_3x3mm_P0.5mm_EP1.68x1.68mm_ThermalVias, symbol coloryr:TLV62130x
- added U2: LP5912-3.3DRV, Package_SON:WSON-6-1EP_2x2mm_P0.65mm_EP1x1.6mm_ThermalVias, symbol Regulator_Linear:LP5912-3.3DRV
- C6: value 0.1uF -> 10uF
- R9: value 100K -> 10K
Connections:
- net 3.3V: now also C6.1, U2.1 (OUT)
- net 5V: now also U2.4 (EN), U2.6 (IN); no longer C6.1
- net GND: now also C6.2, U2.5 (GND), U2.7 (EP)
- net at R9.2: now also U2.3 (PG)
Other:
- note added: "SYS 3.3V"
- note removed: "DC-DC 3.3V"
- moved on the sheet: C5, C6
