File: pcb/v3/wifi.kicad_sch (KiCad schematic)
At the start: 20 parts, among them U8 AP6256, Y1 37.4M, Y2 32.768K

Commit message: up
Parts:
- removed C28, C29, C31, C38: 10pF, Capacitor_SMD:C_0402_1005Metric_Pad0.74x0.62mm_HandSolder, symbol Device:C
- removed C30, C36: 0.1uF, Capacitor_SMD:C_0402_1005Metric_Pad0.74x0.62mm_HandSolder, symbol Device:C
- removed C32: 5.6pF, Capacitor_SMD:C_0402_1005Metric_Pad0.74x0.62mm_HandSolder, symbol Device:C
- removed C33, C34, C35: 4.7uF, Capacitor_SMD:C_0402_1005Metric_Pad0.74x0.62mm_HandSolder, symbol Device:C
- removed L3: 4.7uH, Inductor_SMD:L_Murata_LQH2MCNxxxx02_2.0x1.6mm, symbol Device:L
- removed R44, R45: 0, Resistor_SMD:R_0402_1005Metric_Pad0.72x0.64mm_HandSolder, symbol Device:R
- removed R46: 0, Resistor_SMD:R_1206_3216Metric_Pad1.30x1.75mm_HandSolder, symbol Device:R
- removed U8: AP6256, coloryr:AP6256, symbol coloryr:AP6256
- removed Y1: 37.4M, Oscillator:Oscillator_SMD_ECS_2520MV-xxx-xx-4Pin_2.5x2.0mm, symbol Oscillator:ECS-2520MV-xxx-xx
- removed Y2: 32.768K, Oscillator:Oscillator_SMD_ECS_2520MV-xxx-xx-4Pin_2.5x2.0mm, symbol Oscillator:ECS-2520MV-xxx-xx
- added C39: 4.7uF, Capacitor_SMD:C_0402_1005Metric_Pad0.74x0.62mm_HandSolder, symbol Device:C
- added C40, C41: 0.1uF, Capacitor_SMD:C_0402_1005Metric_Pad0.74x0.62mm_HandSolder, symbol Device:C
- added C42: 10uF, Capacitor_SMD:C_0402_1005Metric_Pad0.74x0.62mm_HandSolder, symbol Device:C
- added R55: 10K, Resistor_SMD:R_0402_1005Metric_Pad0.72x0.64mm_HandSolder, symbol Device:R
- added R56: 0, Resistor_SMD:R_0402_1005Metric_Pad0.72x0.64mm_HandSolder, symbol Device:R
- added U10: AIC8800, coloryr:AIC8800模组, symbol coloryr:AIC8800模组
- renumbered C37 to C43, C39 to C44
Connections:
- net 3.3V: now also C39.2, C40.2, C41.2, C42.2, R55.1, U10.22 (VDDIO), U10.9 (VCC3V3)
- net GND: now also C39.1, C40.1, C41.1, C42.1, U10.1 (GND), U10.20 (GND), U10.3 (GND), U10.31 (GND), U10.33 (GND), U10.36 (GND)
- net at C43.1: now also R56.2, U10.2 (WL-BT-ANT)
- net at C44.1, P3.1 (ANT): now also R56.1
- new net: R55.2, U10.12 (WIFI_POWER)
- new net USBB_DM: U10.10 (USB_DM)
- new net USBB_DP: U10.11 (USB_DP)
Other:
- moved on the sheet: C43, C44, P3
