File: pcb/v3/wifi.kicad_sch (KiCad schematic)
At the start: 12 parts, among them U11 TXS0102DCU, U12 TXS0102DCU, U8 M8800DU6

Commit message: up
Parts:
- added C39: 4.7uF, Capacitor_SMD:C_0402_1005Metric_Pad0.74x0.62mm_HandSolder, symbol Device:C
- added R44: 3.3K, Capacitor_SMD:C_0402_1005Metric_Pad0.74x0.62mm_HandSolder, symbol Device:R
- added R57: 10K, Capacitor_SMD:C_0402_1005Metric_Pad0.74x0.62mm_HandSolder, symbol Device:R
- added R58: 5K, Capacitor_SMD:C_0402_1005Metric_Pad0.74x0.62mm_HandSolder, symbol Device:R
- added U9: ME1502AM5G, Package_TO_SOT_SMD:SOT-23-5, symbol coloryr:ETA6280S2F
Connections:
- net 1.8V: now also R44.2
- net 3.3V: now also C39.1, R57.2, U9.5 (IN); no longer C41.2, C42.2, U8.3 (VDD33)
- net GND: now also C39.2, R58.2, U9.2 (GND)
- net DAC_INT_B: now reaches U12.1 (B2)
- net DAC_INT_2: now reaches U12.4 (A2)
- net DAC_INT_2: now also R44.1
- net DAC_INT renamed DAC_INT_A
- new net: C41.2, C42.2, U8.3 (VDD33), U9.1 (VOUT)
- new net: R58.1, U9.3 (OCB)
- new net WIFI_POWER: R57.1, U9.4 (EN)

Commit message: up
Parts:
- added C40: 0.1uF, Capacitor_SMD:C_0402_1005Metric_Pad0.74x0.62mm_HandSolder, symbol Device:C
- added R84, R92: 15K, Resistor_SMD:R_0402_1005Metric_Pad0.72x0.64mm_HandSolder, symbol Device:R
- added U13: CH422E, Package_SO:MSOP-10_3x3mm_P0.5mm, symbol coloryr:CH442E
Connections:
- net GND: now also C40.2, R84.2, R92.1, U13.5 (GND), U13.9 (EN)
- net USB1_DM: now also U13.6 (DC); no longer U8.4 (USB_DM)
- net USB1_DP: now also U13.4 (DB); no longer U8.5 (USB_DP)
- net WIFI_POWER: now also U13.1 (IN)
- new net: R92.2, U13.2 (S1B)
- new net: R84.1, U13.8 (S1C)
- new net USB1_DM_: U13.7 (S2C), U8.4 (USB_DM)
- new net USB1_DP_: U13.3 (S2B), U8.5 (USB_DP)
- new net VCC: C40.1, U13.10 (VCC)

Commit message: up
Parts:
- added R94, R96: 15K, Capacitor_SMD:C_0402_1005Metric_Pad0.74x0.62mm_HandSolder, symbol Device:R
Connections:
- net GND: now also R94.1, R96.1
- net USB1_DM: now also U8.4 (USB_DM), R94.2
- net USB1_DM_: no longer U8.4 (USB_DM)
- net USB1_DP: now also U8.5 (USB_DP), R96.2
- net USB1_DP_: no longer U8.5 (USB_DP)

Commit message: up pcb
Parts:
- removed C40: 0.1uF, Capacitor_SMD:C_0402_1005Metric_Pad0.74x0.62mm_HandSolder, symbol Device:C
- removed R84, R92: 15K, Resistor_SMD:R_0402_1005Metric_Pad0.72x0.64mm_HandSolder, symbol Device:R
- removed R94, R96: 15K, Capacitor_SMD:C_0402_1005Metric_Pad0.74x0.62mm_HandSolder, symbol Device:R
- removed U13: CH422E, Package_SO:MSOP-10_3x3mm_P0.5mm, symbol coloryr:CH442E

Commit message: up
Changed lines of the file:
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@@
 	(rectangle
 		(start 120.65 20.32)
-		(end 266.065 104.775)
+		(end 266.065 72.39)
 		(stroke
 			(width 0)
@@
 		)
 		(property "Value" "4.7uF"
-			(at 252.73 34.798 90)
+			(at 253.492 34.798 90)
 			(effects
 				(font

Commit message: up
Changed lines of the file:
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@@
 	(rectangle
 		(start 120.65 20.32)
-		(end 266.065 72.39)
+		(end 266.065 104.775)
 		(stroke
 			(width 0)
@@
 		)
 		(property "Value" "4.7uF"
-			(at 253.492 34.798 90)
+			(at 252.73 34.798 90)
 			(effects
 				(font

Commit message: up
Parts:
- R58: value 5K -> 30K
Changed lines of the file:
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@@
 			)
 		)
-		(property "Value" "5K"
+		(property "Value" "30K"
 			(at 221.234 50.038 0)
 			(effects

Commit message: up
Parts:
- U9: value ME1502AM5G -> SY6280
Connections:
- net 3.3V: no longer R57.2
- net GND: now also R57.2
Changed lines of the file:
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@@
-	)
-	(symbol
-		(lib_id "power:VCC")
-		(at 243.84 54.61 180)
-		(unit 1)
-		(exclude_from_sim no)
-		(in_bom yes)
-		(on_board yes)
-		(dnp no)
-		(fields_autoplaced yes)
-		(property "Reference" "#PWR048"
-			(at 243.84 50.8 0)
-			(effects
-				(font
-					(size 1.27 1.27)
-				)
-				(hide yes)
-			)
-		)
-		(property "Value" "3.3V"
-			(at 243.84 59.69 0)
-			(effects
-				(font
-					(size 1.27 1.27)
-				)
-			)
-		)
-		(property "Footprint" ""
-			(at 243.84 54.61 0)
-			(effects
-				(font
-					(size 1.27 1.27)
-				)
-				(hide yes)
-			)
-		)
-		(property "Datasheet" ""
-			(at 243.84 54.61 0)
-			(effects
-				(font
-					(size 1.27 1.27)
-				)
-				(hide yes)
-			)
-		)
-		(property "Description" "Power symbol creates a global label with name \"VCC\""
-			(at 243.84 54.61 0)
-			(effects
-				(font
-					(size 1.27 1.27)
-				)
-				(hide yes)
-			)
-		)
-		(pin "1"
-		)
-		(instances
-			(project "coloryr"
-				(path "/9e6d55f4-a9e8-48fa-bb52-b4e4e3117f8b/948902b6-b2f7-4c71-911b-e81cfbf71b50"
-					(reference "#PWR048")
-					(unit 1)
-				)
-			)
-		)
 	)
 	(symbol
@@
 			)
 		)
-		(property "Value" "ME1502AM5G"
+		(property "Value" "SY6280"
 			(at 228.6 33.02 0)
 			(effects
@@
 					(unit 1)
 				)
+			)
+		)
+	)
+	(symbol
+		(lib_id "power:GND")
+		(at 243.84 54.61 0)
+		(unit 1)
+		(exclude_from_sim no)
+		(in_bom yes)
+		(on_board yes)
+		(dnp no)
+		(fields_autoplaced yes)
+		(property "Reference" "#PWR048"
+			(at 243.84 60.96 0)
+			(effects
+				(font
+					(size 1.27 1.27)
+				)
+				(hide yes)
+			)
+		)
+		(property "Value" "GND"
+			(at 246.38 55.8799 0)
+			(effects
+				(font
+					(size 1.27 1.27)
+				)
+				(justify left)
+			)
+		)
+		(property "Footprint" ""
+			(at 243.84 54.61 0)
+			(effects
+				(font
+					(size 1.27 1.27)
+				)
+				(hide yes)
+			)
+		)
+		(property "Datasheet" ""
+			(at 243.84 54.61 0)
+			(effects
+				(font
+					(size 1.27 1.27)
+				)
+				(hide yes)
+			)
+		)
+		(property "Description" "Power symbol creates a global label with name \"GND\" , ground"
+			(at 243.84 54.61 0)
+			(effects
+				(font
+					(size 1.27 1.27)
+				)
+				(hide yes)
+			)
+		)
+		(pin "1"
+		)
+		(instances
+			(project "coloryr"
+				(path "/9e6d55f4-a9e8-48fa-bb52-b4e4e3117f8b/948902b6-b2f7-4c71-911b-e81cfbf71b50"
+					(reference "#PWR048")
+					(unit 1)
+				)
