File: pcb/v3/coloryr.kicad_pcb (KiCad board)
At the start: 2 copper layers, 43.4 x 75.3 mm, 227 parts, among them J1 TestPoint, J10 Conn_01x02, J11 TestPoint, J12 Conn_01x04, J13 Conn_01x05, J14 TestPoint, J15 TestPoint, J2 Conn_01x03, J3 TestPoint, J4 Conn_01x02, J5 TestPoint, J6 TestPoint, J7 TestPoint, J8 TestPoint, J9 Conn_01x02, P1 LCD_MIPI, P2 LCD_TOUCH, Q1 NPN, Q2 PMOS, U1 SOM3562_18, U10 STI9287, U11 TXS0102DCU, U12 TXS0102DCU, U14 CS43198, U15 CS43198, U16 OPA1622, U17 CH422E, U2 TLV6213x, U4 BQ25895RTW, U5 LM27762, U6 LP5907MFX-3.3, U7 TPS61230DRC, U8 M8800DU6, U9 ME1502AM5G, Y1 24.576M

Commit message: up
Parts:
- added R82: 12.7K, Resistor_SMD:R_0402_1005Metric_Pad0.72x0.64mm_HandSolder, F.Cu at (128.2, 91.9)
- added R83: 22.6K, Resistor_SMD:R_0402_1005Metric_Pad0.72x0.64mm_HandSolder, F.Cu at (128.2, 93.0)
Connections:
- U16 pad 8: OP+ -> Net-(U16A-EN)
Routing:
- net Net-(U16A-EN): track 0.00 -> 8.74 mm, vias 0 -> 2
- net OP+: track 35.5 -> 39.0 mm
- net GND: vias 147 -> 148

Commit message: up
Connections:
- C79 pad 1: 3.3V -> VCC
- R88 pad 2: 3.3V -> VCC
- U17 pad 10: 3.3V -> VCC
Routing:
- net VCC: track 25.8 -> 36.2 mm, vias 3 -> 4
- net 3.3V: track 184.0 -> 180.4 mm, vias 20 -> 18
- net GND: track 96.5 -> 96.1 mm, vias 148 -> 151
Other:
- board text added: "V3.5 By:Coloryr"
- board text removed: "V3.4 By:Coloryr"

Commit message: up
Parts:
- moved R42 33.6 mm to (144.6, 115.9), turned to 0 degrees
- moved R41 33.0 mm to (144.6, 114.7), turned to 0 degrees
- moved R43 31.6 mm to (144.6, 117.0), turned to 0 degrees
- moved C20 4.23 mm to (129.6, 151.6), turned to 0 degrees
- moved C19 4.20 mm to (129.6, 152.6), turned to 0 degrees
- moved J9 3.88 mm to (127.1, 154.6), turned to -90 degrees
Connections:
- U8 pad 4: USB1_DM -> USB1_DM_
- U8 pad 5: USB1_DP -> USB1_DP_
Routing:
- net 3.3V: track 180.4 -> 190.6 mm, vias 18 -> 19
- net Net-(J9-Pin_1): track 0.00 -> 8.15 mm
- net POWER_EN: track 75.5 -> 71.6 mm, vias 4 -> 2
- net BAT_SCL: track 51.4 -> 48.8 mm, vias 2 -> 3
- net SYS: track 36.1 -> 38.5 mm
- net BAT_SDA: track 48.9 -> 49.5 mm, vias 2 -> 3
- net BAT_INT: track 47.0 -> 47.5 mm
- net USB1_DP: vias 1 -> 0
- net USB1_DM: vias 1 -> 0
- net GND: vias 151 -> 152

Commit message: up
Parts:
- removed R82: 12.7K, Resistor_SMD:R_0402_1005Metric_Pad0.72x0.64mm_HandSolder
- removed R83: 22.6K, Resistor_SMD:R_0402_1005Metric_Pad0.72x0.64mm_HandSolder
- added R94: 15K, Capacitor_SMD:C_0402_1005Metric_Pad0.74x0.62mm_HandSolder, F.Cu at (120.9, 126.5)
- added R96: 15K, Capacitor_SMD:C_0402_1005Metric_Pad0.74x0.62mm_HandSolder, F.Cu at (120.9, 125.5)
- moved R87 0.24 mm to (110.1, 148.4)
Connections:
- U1 pad 28: unconnected-(U1-RM_IO11/SAI1_SDI/GPIO0_B3_d-Pad28) -> OUT_EN
- U16 pad 8: Net-(U16A-EN) -> OUT_EN
- U8 pad 4: USB1_DM_ -> USB1_DM
- U8 pad 5: USB1_DP_ -> USB1_DP
Routing:
- net OUT_EN: track 0.00 -> 18.0 mm, vias 0 -> 1
- net OP+: track 39.0 -> 28.5 mm, vias 3 -> 2
- net Net-(U16A-EN): track 8.64 -> 0.00 mm, vias 2 -> 0
- net USB1_DM: track 18.0 -> 22.4 mm, vias 0 -> 1
- net USB1_DP: track 18.1 -> 21.1 mm, vias 0 -> 1
- net 3.3V: track 190.6 -> 188.1 mm, vias 19 -> 17
- net DAC_SCLK: track 48.4 -> 50.0 mm
- net Net-(R7-Pad2): track 2.63 -> 4.10 mm
- net VCC: track 36.2 -> 34.8 mm
- net (no net): track 0.00 -> 1.04 mm
- net GND: vias 152 -> 151

Commit message: up
Routing:
- net (no net): track 1.04 -> 0.00 mm
Changed lines of the file:
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@@
 		(tags "Diode SOD523")
 		(property "Reference" "D3"
-			(at 4.28 -0.17 0)
+			(at 4.5 -0.07 0)
 			(layer "F.SilkS")
 			(effects
@@
 		(tags "capacitor handsolder")
 		(property "Reference" "R8"
-			(at 3.59 -0.13 0)
+			(at 3.81 -0.03 0)
 			(layer "F.SilkS")
 			(effects
@@
 		(tags "Diode SOD523")
 		(property "Reference" "D2"
-			(at 4.2775 0.08 0)
+			(at 4.4975 0.18 0)
 			(layer "F.SilkS")
 			(effects
@@
 		(tags "capacitor handsolder")
 		(property "Reference" "R7"
-			(at 3.58 0.02 0)
+			(at 3.8 0.12 0)
 			(layer "F.SilkS")
 			(effects
@@
 		)
 	)
-	(segment
-		(start 128.76 92.96)
-		(end 128.76 91.92)
-		(width 0.12)
-		(layer "F.Cu")
-		(net 0)
-	)
 	(via

Commit message: up uac
Parts:
- added R82: 5.1K, Capacitor_SMD:C_0402_1005Metric_Pad0.74x0.62mm_HandSolder, F.Cu at (118.1, 146.0)
- added R83: 5.1K, Capacitor_SMD:C_0402_1005Metric_Pad0.74x0.62mm_HandSolder, F.Cu at (117.1, 146.0)
- moved J9 2.54 mm to (124.6, 154.6), turned to 90 degrees
Connections:
- C18 pad 1: Net-(J9-Pin_1) -> Net-(J9-Pin_2)
- J9 pad 1: Net-(J9-Pin_1) -> GND
- J9 pad 2: GND -> Net-(J9-Pin_2)
- U4 pad 13: Net-(J9-Pin_1) -> Net-(J9-Pin_2)
- U4 pad 14: Net-(J9-Pin_1) -> Net-(J9-Pin_2)
- USB1 pad A5: unconnected-(USB1-CC-PadA5) -> Net-(USB1-CC)
- USB1 pad B5: unconnected-(USB1-VCONN-PadB5) -> Net-(USB1-VCONN)
Routing:
- net Net-(USB1-CC): track 0.00 -> 11.0 mm, vias 0 -> 3
- net Net-(J9-Pin_2): track 0.00 -> 8.20 mm
- net Net-(J9-Pin_1): track 8.20 -> 0.00 mm
- net Net-(USB1-VCONN): track 0.00 -> 5.44 mm, vias 0 -> 3
- net VCC: track 34.8 -> 35.8 mm
