File: pcb/v3/coloryr.kicad_pcb (KiCad board)
At the start: 2 copper layers, 43.4 x 75.3 mm, 227 parts, among them J1 TestPoint, J10 Conn_01x02, J11 TestPoint, J12 Conn_01x04, J13 Conn_01x05, J14 TestPoint, J15 TestPoint, J2 Conn_01x03, J3 TestPoint, J4 Conn_01x02, J5 TestPoint, J6 TestPoint, J7 TestPoint, J8 TestPoint, J9 Conn_01x02, P1 LCD_MIPI, P2 LCD_TOUCH, Q1 NPN, Q2 PMOS, Q3 NPN, U1 SOM3562_18, U10 STI9287, U11 TXS0102DCU, U12 TXS0102DCU, U14 CS43198, U15 CS43198, U16 OPA1622, U2 TLV6213x, U4 IP2315, U5 LM27762, U6 LP5907MFX-3.3, U7 TPS61230DRC, U8 M8800DU6, U9 ME1502AM5G, Y1 24.576M

Commit message: up
Parts:
- removed C40: 10uF, Capacitor_SMD:C_0402_1005Metric_Pad0.74x0.62mm_HandSolder
- removed D14: D, Diode_SMD:D_SOD-323_HandSoldering
- removed Q3: NPN, coloryr:SOT-23
- added R84: 22.6K, Capacitor_SMD:C_0402_1005Metric_Pad0.74x0.62mm_HandSolder, F.Cu at (128.2, 91.8)
- added R86: 12.7K, Capacitor_SMD:C_0402_1005Metric_Pad0.74x0.62mm_HandSolder, F.Cu at (128.2, 93.0)
- C15: value 22uF -> 1uF; footprint Capacitor_SMD:C_0603_1608Metric_Pad1.08x0.95mm_HandSolder -> Capacitor_SMD:C_0402_1005Metric_Pad0.74x0.62mm_HandSolder
- C16: value 22uF -> 47nF; footprint Capacitor_SMD:C_0603_1608Metric_Pad1.08x0.95mm_HandSolder -> Capacitor_SMD:C_0402_1005Metric_Pad0.74x0.62mm_HandSolder
- C17: value 22uF -> 4.7uF; footprint Capacitor_SMD:C_0603_1608Metric_Pad1.08x0.95mm_HandSolder -> Capacitor_SMD:C_0402_1005Metric_Pad0.74x0.62mm_HandSolder
- C18: value 22uF -> 10uF; footprint Capacitor_SMD:C_0603_1608Metric_Pad1.08x0.95mm_HandSolder -> Capacitor_SMD:C_0402_1005Metric_Pad0.74x0.62mm_HandSolder
- C19: value 0.1uF -> 10uF; moved to B.Cu
- C20: value 0.1uF -> 10uF
- R15: value 51K -> 260
- R16: value 100K -> 10K
- R17: footprint Resistor_SMD:R_0402_1005Metric_Pad0.72x0.64mm_HandSolder -> Capacitor_SMD:C_0402_1005Metric_Pad0.74x0.62mm_HandSolder; moved to B.Cu
- R43: value 10K -> 4.7K; footprint Resistor_SMD:R_0402_1005Metric_Pad0.72x0.64mm_HandSolder -> Capacitor_SMD:C_0402_1005Metric_Pad0.74x0.62mm_HandSolder
- R82: value 22.6K -> 5.1K; footprint Resistor_SMD:R_0402_1005Metric_Pad0.72x0.64mm_HandSolder -> Capacitor_SMD:C_0402_1005Metric_Pad0.74x0.62mm_HandSolder
- R83: value 12.7K -> 5.1K; footprint Resistor_SMD:R_0402_1005Metric_Pad0.72x0.64mm_HandSolder -> Capacitor_SMD:C_0402_1005Metric_Pad0.74x0.62mm_HandSolder
- U4: value IP2315 -> BQ25895RTW; footprint Package_DFN_QFN:QFN-32-1EP_5x5mm_P0.5mm_EP3.3x3.3mm_ThermalVias -> Package_DFN_QFN:Texas_RTW_WQFN-24-1EP_4x4mm_P0.5mm_EP2.7x2.7mm_ThermalVias
- moved R82 63.2 mm to (110.1, 152.4)
- moved R83 58.3 mm to (110.1, 148.4)
- moved R43 39.3 mm to (144.6, 117.0), turned to 0 degrees
- moved R17 15.9 mm to (132.9, 148.4), turned to 90 degrees
- moved C17 9.31 mm to (123.1, 147.7), turned to 0 degrees
- moved C15 9.09 mm to (126.4, 143.9), turned to 0 degrees
- moved R15 7.44 mm to (131.2, 147.8)
- moved R16 6.42 mm to (131.2, 148.8)
- moved C16 4.17 mm to (123.1, 148.8), turned to 0 degrees
- moved C19 2.67 mm to (129.0, 151.6), turned to 90 degrees
- moved L2 2.33 mm to (125.8, 151.9)
- moved C18 1.92 mm to (131.2, 149.9), turned to 0 degrees
- moved R41 1.12 mm to (144.6, 114.7)
- moved R42 1.08 mm to (144.6, 115.8)
- moved C20 0.80 mm to (130.0, 151.6)
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Connections:
- C15 pad 1: GND -> VCC
- C15 pad 2: VSYS -> GND
- C16 pad 1: GND -> Net-(U4-BTST)
- C16 pad 2: VSYS -> Net-(C16-Pad2)
- C17 pad 2: VSYS -> Net-(U4-REGN)
- C18 pad 1: GND -> Net-(J9-Pin_2)
- C18 pad 2: VSYS -> GND
- C19 pad 1: Net-(D14-K) -> SYS
- C19 pad 2: Net-(U4-BST) -> GND
- J9 pad 2: SYS -> Net-(J9-Pin_2)
- L2 pad 1: Net-(D14-K) -> Net-(C16-Pad2)
- R15 pad 1: GND -> Net-(U4-ILIM)
- R15 pad 2: Net-(U4-NTC) -> GND
- R16 pad 1: GND -> Net-(U4-REGN)
- R16 pad 2: Net-(U4-ICHGSET) -> Net-(U4-TS)
- R17 pad 1: Net-(Q3-B) -> Net-(U4-TS)
- R17 pad 2: HLED -> GND
- R43 pad 2: HCHAG -> BAT_INT
- R82 pad 1: OP+ -> GND
- R82 pad 2: OUT_EN -> Net-(USB1-CC)
- R83 pad 2: OUT_EN -> Net-(USB1-VCONN)
- U1 pad 111: HCHAG -> unconnected-(U1-FLEXBUS1_D4/DSMC_D1/VO_LCDC_D23/GPIO1_A4_d-Pad111)
- U1 pad 41: BAT_SCL -> BAT_SDA
- U1 pad 42: BAT_SDA -> BAT_SCL
- U1 pad 43: unconnected-(U1-RM_IO0/SAI0_LRCK/GPIO0_A0_u-Pad43) -> BAT_INT
- U4 pad 1: (no net) -> VCC
- U4 pad 10: unconnected-(U4-LED3/VSET-Pad10) -> Net-(U4-ILIM)
- U4 pad 11: Net-(D14-K) -> Net-(U4-TS)
- U4 pad 12: Net-(D14-K) -> unconnected-(U4-~{QON}-Pad12)
- U4 pad 13: Net-(D14-K) -> Net-(J9-Pin_2)
- U4 pad 14: Net-(D14-K) -> Net-(J9-Pin_2)
- U4 pad 15: Net-(U4-BST) -> SYS
- U4 pad 16: HLED -> SYS
- U4 pad 18: VSYS -> GND
- U4 pad 19: VSYS -> Net-(C16-Pad2)
- U4 pad 2: CC1 -> unconnected-(U4-D+-Pad2)
- U4 pad 20: VCC -> Net-(C16-Pad2)
- U4 pad 21: VCC -> Net-(U4-BTST)
- U4 pad 22: SYS -> Net-(U4-REGN)
- U4 pad 25: (no net) -> GND
- U4 pad 3: CC2 -> unconnected-(U4-D--Pad3)
- U4 pad 4: (no net) -> unconnected-(U4-STAT-Pad4)
- U4 pad 5: (no net) -> BAT_SCL
- U4 pad 6: VSYS -> BAT_SDA
- U4 pad 7: VSYS -> BAT_INT
- U4 pad 8: BAT_SCL -> unconnected-(U4-OTG-Pad8)
- U4 pad 9: BAT_SDA -> GND
- USB1 pad A5: CC1 -> Net-(USB1-CC)
- USB1 pad B5: CC2 -> Net-(USB1-VCONN)
Routing:
- net BAT_INT: track 0.00 -> 47.3 mm, vias 0 -> 2
- net HCHAG: track 29.0 -> 0.00 mm, vias 2 -> 0
- net CC1: track 25.7 -> 0.00 mm, vias 2 -> 0
- net CC2: track 21.6 -> 0.00 mm, vias 2 -> 0
- net Net-(U4-REGN): track 0.00 -> 12.8 mm, vias 0 -> 2
- net SYS: track 41.8 -> 29.9 mm
- net 3.3V: track 152.0 -> 142.3 mm, vias 19 -> 17
- net HLED: track 9.55 -> 0.00 mm, vias 3 -> 0
- net Net-(J9-Pin_2): track 0.00 -> 4.74 mm, vias 0 -> 2
- net Net-(U4-TS): track 0.00 -> 4.32 mm
- net BAT_SCL: track 53.4 -> 49.3 mm
- net BAT_SDA: track 53.1 -> 49.7 mm
- net Net-(D14-K): track 3.19 -> 0.00 mm, vias 2 -> 0
- net Net-(U4-BTST): track 0.00 -> 2.99 mm
- net VCC: track 23.1 -> 25.8 mm
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Other:
- board text added: "V3.6 By:Coloryr"
- board text removed: "V3.5 By:Coloryr"

Commit message: up
Routing:
- net GND: track 88.6 -> 86.8 mm
- net Net-(U4-REGN): track 12.8 -> 11.1 mm
Changed lines of the file:
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@@
 	)
 	(segment
-		(start 121.5075 91.99)
-		(end 121.5075 93.7925)
-		(width 0.5)
-		(layer "F.Cu")
-		(net 2)
-	)
-	(segment
 		(start 141.1575 107.43)
 		(end 139.72 107.43)
@@
 	)
 	(segment
+		(start 115.941112 118.7635)
+		(end 115.6435 118.465888)
+		(width 0.5)
+		(layer "F.Cu")
+		(net 5)
+	)
+	(segment
 		(start 125.1 128.2025)
 		(end 126.2225 127.08)
@@
 	)
 	(segment
-		(start 115.6435 118.448322)
-		(end 114.63 117.434822)
-		(width 0.5)
-		(layer "F.Cu")
-		(net 5)
-	)
-	(segment
 		(start 126.2225 127.08)
 		(end 126.2225 126.0875)
@@
 	)
 	(segment
-		(start 114.63 117.434822)
-		(end 114.63 116.91)
-		(width 0.5)
-		(layer "F.Cu")
-		(net 5)
-	)
-	(segment
 		(start 109.525 118.74)
 		(end 109.515 118.75)
@@
 	)
 	(segment
+		(start 115.6435 118.465888)
+		(end 115.6435 118.448322)
+		(width 0.5)
+		(layer "F.Cu")
+		(net 5)
+	)
+	(segment
 		(start 123.82 117.94)
 		(end 123.425 118.335)
@@
 	)
 	(segment
-		(start 116.763806 119.586194)
-		(end 115.6435 118.465888)
-		(width 0.5)
-		(layer "F.Cu")
-		(net 5)
-	)
-	(segment
 		(start 126.3 126.13)
 		(end 126.24 126.07)
@@
 	)
 	(segment
-		(start 115.6435 118.465888)
-		(end 115.6435 118.448322)
-		(width 0.5)
+		(start 115.08 138.13)
+		(end 114.58 138.13)
+		(width 0.3)
 		(layer "F.Cu")
 		(net 5)
 	)
 	(segment
-		(start 115.08 138.13)
-		(end 114.58 138.13)
-		(width 0.3)
+		(start 116.763806 119.568628)
+		(end 115.958678 118.7635)
+		(width 0.5)
 		(layer "F.Cu")
 		(net 5)
@@
 	)
 	(segment
+		(start 115.958678 118.7635)
+		(end 115.941112 118.7635)
+		(width 0.5)
+		(layer "F.Cu")
+		(net 5)
+	)
+	(segment
 		(start 113.72599 139.93401)
 		(end 114.58 139.08)
@@
 	)
 	(segment
+		(start 114.63 117.434822)
+		(end 114.63 116.91)
+		(width 0.5)
+		(layer "F.Cu")
+		(net 5)
+	)
+	(segment
+		(start 116.763806 119.586194)
+		(end 116.763806 119.568628)
+		(width 0.5)
+		(layer "F.Cu")
+		(net 5)
+	)
+	(segment
+		(start 115.6435 118.448322)
+		(end 114.63 117.434822)
+		(width 0.5)
+		(layer "F.Cu")
+		(net 5)
+	)
+	(segment
 		(start 133.7615 133.761)
 		(end 133.099 133.761)
@@
 	)
 	(segment
-		(start 124.921 103.911)
-		(end 126.106667 105.096667)
+		(start 124.489 102.014678)
+		(end 124.921 102.446678)
 		(width 0.2)
 		(layer "F.Cu")
@@
 	)
 	(segment
-		(start 126.106667 105.096667)
-		(end 126.106667 106.009167)
+		(start 124.489 97.63)
+		(end 124.489 102.014678)
 		(width 0.2)
 		(layer "F.Cu")
@@
 	)
 	(segment
-		(start 124.688 102.213678)
-		(end 124.921 102.446678)
-		(width 0.2)
-		(layer "F.Cu")
-		(net 124)
-	)
-	(segment
-		(start 124.688 99.578)
-		(end 124.688 102.213678)
-		(width 0.2)
-		(layer "F.Cu")
-		(net 124)
-	)
-	(segment
 		(start 124.489 97.579322)
 		(end 126.221 95.847322)
@@
 	)
 	(segment
-		(start 124.921 102.446678)
-		(end 124.921 103.911)
+		(start 138.12 104.949738)
+		(end 137.010262 103.84)
 		(width 0.2)
 		(layer "F.Cu")
@@
 	)
 	(segment
-		(start 138.12 104.949738)
-		(end 137.010262 103.84)
+		(start 124.921 102.446678)
+		(end 124.921 103.911)
 		(width 0.2)
 		(layer "F.Cu")
@@
 	)
 	(segment
-		(start 124.489 97.63)
-		(end 124.489 99.379)
+		(start 126.221 93.231)
+		(end 124.98 91.99)
 		(width 0.2)
 		(layer "F.Cu")
@@
 	)
 	(segment
-		(start 126.221 93.231)
-		(end 124.98 91.99)
+		(start 124.921 103.911)
+		(end 126.106667 105.096667)
 		(width 0.2)
 		(layer "F.Cu")
@@
 	)
 	(segment
-		(start 124.489 99.379)
-		(end 124.688 99.578)
+		(start 126.106667 105.096667)
+		(end 126.106667 106.009167)
 		(width 0.2)
 		(layer "F.Cu")
@@
 	)
 	(segment
-		(start 128.332 149.44)
-		(end 127.15 149.44)
+		(start 129.339 146.109)
+		(end 125.591 146.109)
 		(width 0.12)
 		(layer "F.Cu")
@@
 	)
 	(segment
-		(start 130.17 147.602)
-		(end 128.332 149.44)
-		(width 0.12)
-		(layer "F.Cu")
-		(net 225)
-	)
-	(segment
-		(start 125.928 149.44)
-		(end 124.34 147.852)
+		(start 125.591 146.109)
+		(end 124.34 147.36)
 		(width 0.12)
 		(layer "F.Cu")
@@
 	(segment
 		(start 130.17 146.94)
-		(end 130.17 147.602)
-		(width 0.12)
-		(layer "F.Cu")
-		(net 225)
-	)
-	(segment
-		(start 127.15 149.44)
-		(end 125.928 149.44)
-		(width 0.12)
-		(layer "F.Cu")
-		(net 225)
-	)
-	(segment
-		(start 124.34 147.852)
-		(end 124.34 147.36)
+		(end 129.339 146.109)
 		(width 0.12)
 		(layer "F.Cu")
@@
 		(polygon
 			(pts
-				(xy 104.49 93.42) (xy 124.47 93.42) (xy 124.47 85.69) (xy 147.94 85.69) (xy 147.94 156.06) (xy 104.49 156.06)
+				(xy 104.49 93.42) (xy 120.72 93.42) (xy 120.72 85.69) (xy 147.94 85.69) (xy 147.94 156.06) (xy 104.49 156.06)
 			)
 		)

Commit message: up
Parts:
- moved R2 1.96 mm to (127.8, 140.4)
- moved R95 1.89 mm to (127.8, 139.3)
Routing:
- net Net-(U1-USB20_OTG0_ID): track 12.3 -> 14.4 mm
- net RESET: track 60.4 -> 58.4 mm
- net VCC_1V8_OUT: track 35.4 -> 33.7 mm
- net HP_CONTROL: track 105.4 -> 106.9 mm, vias 4 -> 3
- net 3.3V: track 142.3 -> 141.3 mm
- net TP_SDA: track 46.7 -> 47.3 mm
- net VCC_3V3_OUT: track 69.0 -> 69.4 mm, vias 1 -> 3
- net GND: vias 144 -> 147

Commit message: up
Parts:
- moved R41 1.34 mm to (144.6, 113.4)
- moved R42 1.18 mm to (144.6, 114.7)
- moved R43 0.98 mm to (144.6, 116.0)
Routing:
- net BAT_SDA: track 49.7 -> 51.7 mm
- net BAT_SCL: track 49.3 -> 50.9 mm
- net BAT_INT: track 47.3 -> 48.8 mm
- net 3.3V: track 141.3 -> 142.7 mm

Commit message: up
Parts:
- R58: value 5K -> 30K
Connections:
- P1 pad MP: (no net) -> GND
- P2 pad MP: (no net) -> GND
Routing:
- net POWER_ON: track 19.5 -> 18.8 mm
- net Net-(U1-USB20_OTG0_ID): track 14.4 -> 13.8 mm

Commit message: up
Routing:
- net POWER_ON: track 18.8 -> 19.5 mm
Changed lines of the file:
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@@
+	)
+	(segment
+		(start 111.079001 141.049)
+		(end 109.269 139.239)
+		(width 0.12)
+		(layer "F.Cu")
+		(net 87)
+	)
+	(segment
+		(start 118.139047 139.749)
+		(end 116.839047 141.049)
+		(width 0.12)
+		(layer "F.Cu")
+		(net 87)
+	)
+	(segment
+		(start 125.248 139.749)
+		(end 118.139047 139.749)
+		(width 0.12)
+		(layer "F.Cu")
+		(net 87)
+	)
+	(segment
+		(start 116.839047 141.049)
+		(end 111.079001 141.049)
+		(width 0.12)
+		(layer "F.Cu")
+		(net 87)
 	)
 	(segment
@@
 	)
 	(segment
-		(start 115.21 114.09)
-		(end 113.5475 114.09)
-		(width 0.12)
-		(layer "F.Cu")
-		(net 87)
-	)
-	(segment
 		(start 126.23 140.731)
 		(end 125.248 139.749)
-		(width 0.12)
-		(layer "F.Cu")
-		(net 87)
-	)
-	(segment
-		(start 113.579 128.410999)
-		(end 113.579 116.854522)
 		(width 0.12)
 		(layer "F.Cu")
@@
 	)
 	(segment
-		(start 119.161 139.749)
-		(end 117.861 141.049)
-		(width 0.12)
-		(layer "F.Cu")
-		(net 87)
-	)
-	(segment
-		(start 125.248 139.749)
-		(end 119.161 139.749)
-		(width 0.12)
-		(layer "F.Cu")
-		(net 87)
-	)
-	(segment
 		(start 142.5475 142.39)
 		(end 142.0665 142.871)
@@
 	)
 	(segment
+		(start 116.21 115.09)
+		(end 115.21 114.09)
+		(width 0.12)
+		(layer "F.Cu")
+		(net 87)
+	)
+	(segment
 		(start 116.21 116.03)
 		(end 116.21 115.09)
@@
 		(start 138.075191 140.271)
 		(end 129.499 140.271)
-		(width 0.12)
-		(layer "F.Cu")
-		(net 87)
-	)
-	(segment
-		(start 114.033522 116.4)
-		(end 115.84 116.4)
-		(width 0.12)
-		(layer "F.Cu")
-		(net 87)
-	)
-	(segment
-		(start 117.861 141.049)
-		(end 111.079001 141.049)
 		(width 0.12)
 		(layer "F.Cu")
@@
 	)
 	(segment
+		(start 114.033522 116.4)
+		(end 115.84 116.4)
+		(width 0.12)
+		(layer "F.Cu")
+		(net 87)
+	)
+	(segment
+		(start 109.269 132.721)
+		(end 113.579 128.410999)
+		(width 0.12)
+		(layer "F.Cu")
+		(net 87)
+	)
+	(segment
 		(start 142.0665 142.871)
 		(end 140.675191 142.871)
@@
 	)
 	(segment
-		(start 111.079001 141.049)
-		(end 109.269 139.239)
+		(start 113.579 128.410999)
+		(end 113.579 116.854522)
 		(width 0.12)
 		(layer "F.Cu")
@@
 	)
 	(segment
-		(start 116.21 115.09)
-		(end 115.21 114.09)
-		(width 0.12)
-		(layer "F.Cu")
-		(net 87)
-	)
-	(segment
 		(start 129.499 140.271)
 		(end 129.218 139.99)
@@
 	)
 	(segment
-		(start 109.269 132.721)
-		(end 113.579 128.410999)
+		(start 115.21 114.09)
+		(end 113.5475 114.09)
 		(width 0.12)
 		(layer "F.Cu")
@@
 	)
 	(segment
-		(start 108.827 139.422082)
-		(end 108.827 130.487)
+		(start 108.04 139.418)
+		(end 108.04 129.7)
 		(width 0.12)
 		(layer "F.Cu")
@@
 	)
 	(segment
-		(start 113.124918 143.72)
-		(end 108.827 139.422082)
+		(start 115.08 143.72)
+		(end 111.86 143.72)
 		(width 0.12)
 		(layer "F.Cu")
@@
 	)
 	(segment
-		(start 108.827 130.487)
-		(end 108.04 129.7)
+		(start 108.741 140.601)
+		(end 108.741 140.119)
 		(width 0.12)
 		(layer "F.Cu")
@@
 	)
 	(segment
-		(start 115.08 143.72)
-		(end 113.124918 143.72)
+		(start 108.741 140.119)
+		(end 108.04 139.418)
+		(width 0.12)
+		(layer "F.Cu")
+		(net 99)
+	)
+	(segment
+		(start 111.86 143.72)
+		(end 108.741 140.601)
 		(width 0.12)
 		(layer "F.Cu")
@@
 	)
 	(segment
+		(start 115.07 115.301831)
+		(end 114.877169 115.109)
+		(width 0.12)
+		(layer "F.Cu")
+		(net 110)
+	)
+	(segment
+		(start 113.358 128.319458)
+		(end 113.358 116.76298)
+		(width 0.12)
+		(layer "F.Cu")
+		(net 110)
+	)
+	(segment
+		(start 112.96 114.318396)
+		(end 112.96 112.08)
+		(width 0.12)
+		(layer "F.Cu")
+		(net 110)
+	)
+	(segment
+		(start 113.358 116.76298)
+		(end 113.941981 116.179)
+		(width 0.12)
+		(layer "F.Cu")
+		(net 110)
+	)
+	(segment
+		(start 113.941981 116.179)
+		(end 114.821 116.179)
+		(width 0.12)
+		(layer "F.Cu")
+		(net 110)
+	)
+	(segment
+		(start 109.048 132.629458)
+		(end 113.358 128.319458)
+		(width 0.12)
+		(layer "F.Cu")
+		(net 110)
+	)
+	(segment
+		(start 114.877169 115.109)
+		(end 113.750604 115.109)
+		(width 0.12)
+		(layer "F.Cu")
+		(net 110)
+	)
+	(segment
+		(start 109.6 108.72)
+		(end 109.401953 108.72)
+		(width 0.12)
+		(layer "F.Cu")
+		(net 110)
+	)
+	(segment
+		(start 117.95 141.27)
+		(end 110.987459 141.27)
+		(width 0.12)
+		(layer "F.Cu")
+		(net 110)
+	)
+	(segment
+		(start 113.750604 115.109)
+		(end 112.96 114.318396)
+		(width 0.12)
+		(layer "F.Cu")
+		(net 110)
+	)
+	(segment
 		(start 112.96 112.08)
 		(end 109.6 108.72)
@@
 	)
 	(segment
-		(start 114.877169 115.109)
-		(end 113.750604 115.109)
-		(width 0.12)
-		(layer "F.Cu")
-		(net 110)
-	)
-	(segment
 		(start 109.048 139.330541)
 		(end 109.048 132.629458)
@@
 	)
 	(segment
-		(start 112.96 114.318396)
-		(end 112.96 112.08)
-		(width 0.12)
-		(layer "F.Cu")
-		(net 110)
-	)
-	(segment
-		(start 115.07 115.301831)
-		(end 114.877169 115.109)
-		(width 0.12)
-		(layer "F.Cu")
-		(net 110)
-	)
-	(segment
-		(start 113.941981 116.179)
-		(end 114.821 116.179)
+		(start 114.821 116.179)
+		(end 115.07 115.93)
+		(width 0.12)
+		(layer "F.Cu")
+		(net 110)
+	)
+	(segment
+		(start 110.987459 141.27)
+		(end 109.048 139.330541)
 		(width 0.12)
 		(layer "F.Cu")
@@
 		(net 110)
 	)
-	(segment
-		(start 114.821 116.179)
-		(end 115.07 115.93)
-		(width 0.12)
-		(layer "F.Cu")
-		(net 110)
-	)
-	(segment
-		(start 113.358 116.76298)
-		(end 113.941981 116.179)
-		(width 0.12)
-		(layer "F.Cu")
-		(net 110)
-	)
-	(segment
-		(start 113.358 128.319458)
-		(end 113.358 116.76298)
-		(width 0.12)
-		(layer "F.Cu")
-		(net 110)
-	)
-	(segment
-		(start 109.6 108.72)
-		(end 109.401953 108.72)
-		(width 0.12)
-		(layer "F.Cu")
-		(net 110)
-	)
-	(segment
-		(start 109.048 132.629458)
-		(end 113.358 128.319458)
-		(width 0.12)
-		(layer "F.Cu")
-		(net 110)
-	)
-	(segment
-		(start 113.750604 115.109)
-		(end 112.96 114.318396)
-		(width 0.12)
-		(layer "F.Cu")
-		(net 110)
-	)
-	(segment
-		(start 118.4 141.27)
-		(end 110.987459 141.27)
-		(width 0.12)
-		(layer "F.Cu")
-		(net 110)
-	)
-	(segment
-		(start 110.987459 141.27)
-		(end 109.048 139.330541)
-		(width 0.12)
-		(layer "F.Cu")
-		(net 110)
-	)
-	(via
-		(at 118.4 141.27)
-		(size 0.6)
-		(drill 0.3)
-		(layers "F.Cu" "B.Cu")
+	(via
+		(at 117.95 141.27)
+		(size 0.6)
+		(drill 0.3)
+		(layers "F.Cu" "B.Cu")
+		(net 110)
+	)
+	(segment
+		(start 120.96118 141.75118)
+		(end 120.96118 142.988262)
+		(width 0.12)
+		(layer "B.Cu")
+		(net 110)
+	)
+	(segment
+		(start 120.96118 142.988262)
+		(end 121.248918 143.276)
+		(width 0.12)
+		(layer "B.Cu")
+		(net 110)
+	)
+	(segment
+		(start 122.67 143.073319)
+		(end 122.67 142.48)
+		(width 0.12)
+		(layer "B.Cu")
+		(net 110)
+	)
+	(segment
+		(start 117.95 141.27)
+		(end 120.48 141.27)
+		(width 0.12)
+		(layer "B.Cu")
+		(net 110)
+	)
+	(segment
+		(start 121.248918 143.276)
+		(end 122.467319 143.276)
+		(width 0.12)
+		(layer "B.Cu")
+		(net 110)
+	)
+	(segment
+		(start 120.48 141.27)
+		(end 120.96118 141.75118)
+		(width 0.12)
+		(layer "B.Cu")
 		(net 110)
 	)
@@
 		(width 0.12)
 		(layer "B.Cu")
-		(net 110)
-	)
-	(segment
-		(start 120.96118 142.988262)
-		(end 121.248918 143.276)
-		(width 0.12)
-		(layer "B.Cu")
-		(net 110)
-	)
-	(segment
-		(start 121.248918 143.276)
-		(end 122.467319 143.276)
-		(width 0.12)
-		(layer "B.Cu")
-		(net 110)
-	)
-	(segment
-		(start 118.4 141.27)
-		(end 120.48 141.27)
-		(width 0.12)
-		(layer "B.Cu")
-		(net 110)
-	)
-	(segment
-		(start 120.96118 141.75118)
-		(end 120.96118 142.988262)
-		(width 0.12)
-		(layer "B.Cu")
-		(net 110)
-	)
-	(segment
-		(start 120.48 141.27)
-		(end 120.96118 141.75118)
-		(width 0.12)
-		(layer "B.Cu")
-		(net 110)
-	)
-	(segment
-		(start 122.67 143.073319)
-		(end 122.67 142.48)
-		(width 0.12)
-		(layer "B.Cu")
