File: pcb/v3/coloryr.kicad_pcb (KiCad board)
At the start: 2 copper layers, 43.4 x 75.3 mm, 226 parts, among them J1 TestPoint, J10 Conn_01x02, J11 TestPoint, J12 Conn_01x04, J13 Conn_01x05, J14 TestPoint, J15 TestPoint, J2 Conn_01x03, J3 TestPoint, J4 Conn_01x02, J5 TestPoint, J6 TestPoint, J7 TestPoint, J8 TestPoint, J9 Conn_01x02, P1 LCD_MIPI, P2 LCD_TOUCH, Q1 NPN, Q2 PMOS, U1 SOM3562_18, U10 STI9287, U11 TXS0102DCU, U12 TXS0102DCU, U14 CS43198, U15 CS43198, U16 OPA1622, U2 TLV6213x, U4 BQ25895RTW, U5 LM27762, U6 LP5907MFX-3.3, U7 TPS61230DRC, U8 M8800DU6, U9 ME1502AM5G, Y1 24.576M

Commit message: up
Parts:
- U9: value ME1502AM5G -> SY6280
- moved C39 0.14 mm to (116.4, 117.5)
Connections:
- R57 pad 2: 3.3V -> GND
Routing:
- net HP_DETECT1: track 10.5 -> 12.3 mm
- net 3.3V: track 142.7 -> 141.3 mm
- net +INA: track 18.8 -> 17.5 mm, vias 2 -> 3
- net REF_B: track 35.3 -> 36.0 mm
- net GND: vias 147 -> 153
Other:
- board text added: "V3.7 By:Coloryr"
- board text removed: "V3.6 By:Coloryr"

Commit message: up
Parts:
- removed R93: 0, Resistor_SMD:R_0805_2012Metric
- added C40: 100nF, Capacitor_SMD:C_0402_1005Metric_Pad0.74x0.62mm_HandSolder, B.Cu at (123.1, 146.7)
- added C43: 10uF, Capacitor_SMD:C_0402_1005Metric_Pad0.74x0.62mm_HandSolder, F.Cu at (141.1, 89.9)
- added C44: 0.1uF, Capacitor_SMD:C_0402_1005Metric_Pad0.74x0.62mm_HandSolder, F.Cu at (141.1, 88.8)
- added R87: 10K, Capacitor_SMD:C_0402_1005Metric_Pad0.74x0.62mm_HandSolder, F.Cu at (144.3, 85.2)
- added R88: 4.7K, Capacitor_SMD:C_0402_1005Metric_Pad0.74x0.62mm_HandSolder, F.Cu at (145.4, 85.2)
- added R92: 4.7K, Capacitor_SMD:C_0402_1005Metric_Pad0.74x0.62mm_HandSolder, F.Cu at (142.2, 94.6)
- added RF1: 6GHz, coloryr:IPEX-SMD_BWIPX-3-001E-1, B.Cu at (106.2, 127.6)
- added U13: TS3A227E, Package_DFN_QFN:QFN-16-1EP_3x3mm_P0.5mm_EP1.675x1.675mm, F.Cu at (144.6, 89.0)
- R20: value 100K/NC -> 10K
- R89: value 0 -> 10K; footprint Resistor_SMD:R_0402_1005Metric_Pad0.72x0.64mm_HandSolder -> Capacitor_SMD:C_0402_1005Metric_Pad0.74x0.62mm_HandSolder
- RV1, RV2: footprint Potentiometer_THT:Potentiometer_Bourns_3266W_Vertical -> Potentiometer_SMD:Potentiometer_Bourns_TC33X_Vertical
- moved R89 22.4 mm to (128.2, 94.2), turned to 180 degrees
- moved R22 14.1 mm to (121.4, 146.1), turned to -90 degrees
- moved J11 6.71 mm to (131.5, 155.2)
- moved R19 6.63 mm to (123.1, 145.6)
- moved C5 4.78 mm to (135.3, 144.5), turned to 180 degrees
- moved C15 3.36 mm to (123.1, 144.5), turned to 180 degrees
- moved Q1 3.25 mm to (118.9, 145.8), turned to 0 degrees
- moved C6 2.95 mm to (135.3, 145.6)
- moved RV2 2.25 mm to (107.5, 100.7)
- moved RV1 1.57 mm to (113.6, 100.7)
- moved R43 1.56 mm to (144.6, 114.4)
- moved R42 1.31 mm to (144.6, 113.3)
- moved R95 1.15 mm to (127.8, 140.5)
- moved R41 1.09 mm to (144.6, 112.3)
- moved R9 1.08 mm to (135.2, 148.7)
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Connections:
- net Net-(CN1-Pad3) renamed HP_TIP
- net Net-(PJ1-Pad4) renamed HP_DET
- C23 pad 1: SYS -> POWER
- CN1 pad 6: unconnected-(CN1-Pad6) -> HP_DETECT_IO
- L3 pad 1: SYS -> POWER
- PJ1 pad 1: GND -> HP_SLEEVE
- PJ1 pad 5: Net-(PJ1-Pad5) -> HP_RING2
- Q2 pad 1: POWER_EN -> POWER
- Q2 pad 2: Net-(D5-A) -> Net-(Q2-G)
- R19 pad 2: Net-(D5-A) -> Net-(Q2-G)
- R22 pad 1: POWER_EN -> Net-(Q2-G)
- R22 pad 2: GND -> Net-(D5-A)
- R26 pad 1: POWER_EN -> POWER
- R89 pad 1: DAC_MCLK_1 -> Net-(CN1-3-Pad4)
- R89 pad 2: DAC_PWM -> GND
- U1 pad 29: LED_STATE -> HP_INT
- U1 pad 30: DAC_SDA -> HP_DETECT_IO
- U1 pad 31: DAC_SCL -> LED_STATE
- U1 pad 36: DAC_PWM -> DAC_SDA
- U1 pad 37: TP_SCL -> DAC_SCL
- U1 pad 38: TP_SDA -> BAT_SDA
- U1 pad 39: LCD_LED -> BAT_SCL
- U1 pad 40: unconnected-(U1-RM_IO3/SAI0_SDO/GPIO0_A3_d-Pad40) -> BAT_INT
- U1 pad 41: BAT_SDA -> TP_SCL
- U1 pad 42: BAT_SCL -> TP_SDA
- U1 pad 43: BAT_INT -> LCD_LED
- U1 pad 88: unconnected-(U1-ACODEC_ADC_INP-Pad88) -> HP_CONTROL
- U1 pad 89: unconnected-(U1-ACODEC_ADC_INN-Pad89) -> MIC_GND
- U7 pad 10: SYS -> POWER
- U7 pad 9: POWER_EN -> POWER
- U8 pad 2: unconnected-(U8-ANT0-Pad2) -> Net-(U8-ANT0)
Routing:
- net MIC_GND: track 0.00 -> 111.3 mm, vias 0 -> 3
- net POWER: track 0.00 -> 74.0 mm, vias 0 -> 8
- net POWER_EN: track 71.1 -> 0.00 mm, vias 2 -> 0
- net HP_DETECT_IO: track 0.00 -> 60.0 mm, vias 0 -> 3
- net 3.3V: track 141.3 -> 178.3 mm, vias 17 -> 19
- net DAC_PWM: track 31.0 -> 0.00 mm, vias 1 -> 0
- net HP_INT: track 0.00 -> 25.8 mm, vias 0 -> 1
- net SYS: track 29.9 -> 6.70 mm, vias 7 -> 8
- net GND: track 86.8 -> 69.2 mm, vias 153 -> 178
- net DAC_SDA: track 40.2 -> 57.3 mm, vias 3 -> 4
- net DAC_SCL: track 39.1 -> 56.0 mm, vias 3 -> 4
- net HP_CONTROL: track 106.9 -> 122.7 mm, vias 3 -> 4
- net HP_SLEEVE: track 0.00 -> 14.3 mm, vias 0 -> 1
- net HP_DET: track 3.15 -> 16.4 mm, vias 0 -> 1
- net Net-(D5-A): track 26.7 -> 14.1 mm
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
Commit message: up
Parts:
- removed C36, C38: 0.1uF, Capacitor_SMD:C_0402_1005Metric_Pad0.74x0.62mm_HandSolder
- removed R55: 3.3K, Capacitor_SMD:C_0402_1005Metric_Pad0.74x0.62mm_HandSolder
- removed R75, R80: 0, Resistor_SMD:R_0805_2012Metric
- removed R89: 10K, Capacitor_SMD:C_0402_1005Metric_Pad0.74x0.62mm_HandSolder
- removed R92: 4.7K, Capacitor_SMD:C_0402_1005Metric_Pad0.74x0.62mm_HandSolder
- removed U12: TXS0102DCU, Package_SO:VSSOP-8_2.3x2mm_P0.5mm
- added C79: 10uF, Capacitor_SMD:C_0603_1608Metric_Pad1.08x0.95mm_HandSolder, B.Cu at (137.1, 82.2)
- added Q3: NMOS, coloryr:SOT-23, F.Cu at (145.1, 85.0)
- added R93: 330K, Resistor_SMD:R_0402_1005Metric_Pad0.72x0.64mm_HandSolder, F.Cu at (141.1, 86.6)
- R44: value 3.3K -> 330K; footprint Capacitor_SMD:C_0402_1005Metric_Pad0.74x0.62mm_HandSolder -> Resistor_SMD:R_0402_1005Metric_Pad0.72x0.64mm_HandSolder
- moved R44 32.0 mm to (141.1, 87.7), turned to 180 degrees
- moved R88 4.31 mm to (141.2, 84.1), turned to 0 degrees
- moved R87 3.14 mm to (141.2, 85.1), turned to 180 degrees
Connections:
- CN1 pad 3: HP_TIP -> Net-(C79-Pad1)
- CN1 pad 4: Net-(CN1-3-Pad4) -> unconnected-(CN1-3-Pad4)
- CN1 pad 6: HP_DETECT_IO -> HP_DETECT
- PJ1 pad 4: HP_DET -> HP_DETECT_IO
- R44 pad 1: DAC_INT_2 -> HP_DETECT1
- R44 pad 2: 1.8V -> 3.3V
- R76 pad 1: HP_TIP -> Net-(C79-Pad1)
- R87 pad 1: HP_DET -> HP_DETECT_IO
- U1 pad 27: unconnected-(U1-RM_IO12/SAI1_SDO0/GPIO0_B4_d-Pad27) -> OUT_EN
- U1 pad 28: OUT_EN -> HP_DETECT
- U1 pad 29: HP_INT -> HP_DETECT1
- U1 pad 30: HP_DETECT_IO -> HP_INT
- U13 pad 15: HP_DET -> HP_DETECT1
- U14 pad 22: HP_DETECT -> unconnected-(U14-HP_DETECT-Pad22)
- U14 pad 27: DAC_INT_1 -> unconnected-(U14-INT-Pad27)
- U15 pad 22: HP_DETECT1 -> unconnected-(U15-HP_DETECT-Pad22)
- U15 pad 27: DAC_INT_2 -> unconnected-(U15-INT-Pad27)
Routing:
- net HP_DETECT: track 12.9 -> 62.3 mm, vias 2 -> 1
- net HP_DETECT_IO: track 60.0 -> 18.5 mm, vias 3 -> 1
- net DAC_INT_A: track 23.6 -> 0.00 mm, vias 1 -> 0
- net DAC_INT_B: track 20.4 -> 0.00 mm, vias 1 -> 0
- net HP_TIP: track 34.9 -> 17.4 mm
- net Net-(C79-Pad1): track 0.00 -> 16.9 mm
- net HP_DET: track 16.4 -> 0.00 mm, vias 1 -> 0
- net DAC_INT_2: track 14.8 -> 0.00 mm, vias 2 -> 0
- net DAC_INT_1: track 11.4 -> 0.00 mm, vias 2 -> 0
- net HP_DETECT1: track 12.2 -> 22.4 mm
- net 1.8V: track 102.4 -> 92.5 mm
- net 3.3V: track 178.3 -> 169.9 mm, vias 19 -> 18
- net Net-(CN1-3-Pad4): track 4.29 -> 0.00 mm
- net HP_INT: track 25.8 -> 29.3 mm
- net OUT_EN: track 24.6 -> 23.8 mm
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Other:
- board text added: "V3.8 By:Coloryr"
- board text removed: "V3.7 By:Coloryr"

Commit message: up
Parts:
- added C36: 10uF, Capacitor_SMD:C_0603_1608Metric_Pad1.08x0.95mm_HandSolder, F.Cu at (130.7, 88.1)
- added R55: 10K, Capacitor_SMD:C_0402_1005Metric_Pad0.74x0.62mm_HandSolder, F.Cu at (131.0, 86.7)
- turned C79 to 180 degrees
Connections:
- C79 pad 1: Net-(C79-Pad1) -> HP_TIP
- C79 pad 2: HP_TIP -> Net-(C79-Pad2)
- CN1 pad 2: Net-(CN1-Pad2) -> Net-(C36-Pad2)
- CN1 pad 3: Net-(C79-Pad1) -> Net-(C79-Pad2)
- PJ1 pad 2: Net-(CN1-Pad2) -> Net-(C36-Pad1)
- R76 pad 1: Net-(C79-Pad1) -> Net-(C79-Pad2)
- R77 pad 1: Net-(CN1-Pad2) -> Net-(C36-Pad2)
- R87 pad 1: HP_DETECT_IO -> HP_TIP
Routing:
- net Net-(CN1-Pad2): track 32.4 -> 0.00 mm
- net Net-(C36-Pad2): track 0.00 -> 24.4 mm
- net Net-(C79-Pad2): track 0.00 -> 16.9 mm
- net Net-(C79-Pad1): track 16.9 -> 0.00 mm
- net Net-(C36-Pad1): track 0.00 -> 8.55 mm, vias 0 -> 1
- net HP_DETECT_IO: track 18.5 -> 17.1 mm
- net HP_TIP: vias 1 -> 2

Commit message: up
Parts:
- C79: moved to F.Cu
- moved C79 1.79 mm to (138.8, 82.0)
Routing:
- net HP_TIP: track 17.4 -> 15.2 mm, vias 2 -> 3
- net Net-(C36-Pad2): track 24.4 -> 22.4 mm
- net Net-(C79-Pad2): track 16.9 -> 18.2 mm, vias 0 -> 1
- net GND: vias 178 -> 180

Commit message: up
Parts:
- U13: footprint Package_DFN_QFN:QFN-16-1EP_3x3mm_P0.5mm_EP1.675x1.675mm -> Package_DFN_QFN:Texas_RVA_VQFN-16-1EP_3.5x3.5mm_P0.5mm_EP2.14x2.14mm
- moved C43 3.86 mm to (144.1, 92.3), turned to 0 degrees
- moved C44 0.97 mm to (141.1, 89.8)
- moved R44 0.64 mm to (141.0, 88.3)
