File: pcb/v2/coloryr.kicad_sch (KiCad schematic)
At the start: 0 parts

Commit message: up fix lcd pcb
Changed lines of the file:
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@@
 	)
 	(sheet
-		(at 40.64 66.04)
+		(at 91.44 72.39)
 		(size 25.4 21.59)
 		(exclude_from_sim no)
@@
 		)
 		(property "Sheetname" "DAC"
-			(at 40.64 65.3284 0)
+			(at 91.44 71.6784 0)
 			(effects
 				(font
@@
 		)
 		(property "Sheetfile" "dac.kicad_sch"
-			(at 40.64 88.2146 0)
+			(at 91.44 94.5646 0)
 			(effects
 				(font
@@
 	)
 	(sheet
-		(at 158.75 29.21)
+		(at 59.69 72.39)
 		(size 24.13 21.59)
 		(exclude_from_sim no)
@@
 		)
 		(property "Sheetname" "WIFI"
-			(at 158.75 28.4984 0)
+			(at 59.69 71.6784 0)
 			(effects
 				(font
@@
 		)
 		(property "Sheetfile" "wifi.kicad_sch"
-			(at 158.75 51.3846 0)
+			(at 59.69 94.5646 0)
 			(effects
 				(font
@@
 	)
 	(sheet
-		(at 125.73 25.4)
+		(at 26.67 68.58)
 		(size 25.4 25.4)
 		(exclude_from_sim no)
@@
 		)
 		(property "Sheetname" "IO"
-			(at 125.73 24.6884 0)
+			(at 26.67 67.8684 0)
 			(effects
 				(font
@@
 		)
 		(property "Sheetfile" "io.kicad_sch"
-			(at 125.73 51.3846 0)
+			(at 26.67 94.5646 0)
 			(effects
 				(font
