File: pcb/v2/coloryr.kicad_pcb (KiCad board)
At the start: 2 copper layers, 118 x 67 mm, 217 parts, among them J1 Conn_01x02, J10 Conn_01x05, J14 Conn_01x04, J15 Conn_01x02, J16 TestPoint, J17 TestPoint, J2 Conn_01x03, J3 Conn_01x02, J4 Conn_01x02, J5 TestPoint, J6 TestPoint, J7 Conn_01x02, J8 Conn_01x02, J9 TestPoint, Q1 NPN, Q2 PNP, Q3 PNP, Q4 NPN, U1 SOM3562_18, U10 AIC8800, U11 1, U12 1, U13 OPA1622, U2 TPS61230DRC, U3 LM27762, U4 TLV6213x, U5 BQ25895RTW, U7 TCKE812, U8 CH334R, U9 STI9287, Y1 12M

Commit message: up
Parts:
- removed J15: Conn_01x02, Connector_PinHeader_2.54mm:PinHeader_1x02_P2.54mm_Vertical
- added R14: 10K, Resistor_SMD:R_0402_1005Metric_Pad0.72x0.64mm_HandSolder, F.Cu at (182.9, 118.6)
- Q2, Q3: value PNP -> PMOS
- R17: value 100K -> 260
- R24, R38: value 100K -> 10K
- U11, U12: value 1 -> CS43198
- moved USB1 0.47 mm to (190.7, 114.3)
Connections:
- U5 pad 23: Net-(J15-Pin_1) -> unconnected-(U5-PMID-Pad23)
Routing:
- net SYS: track 72.8 -> 75.7 mm
- net POWER_EN: track 117.2 -> 119.2 mm
- net GND: track 48.3 -> 49.5 mm
- net Net-(R7-Pad2): track 4.77 -> 5.27 mm
- net Net-(J15-Pin_1): vias 1 -> 0
Other:
- board text added: "ColorAudio v2.1"
- board text removed: "ColorAudio v2.0"

Commit message: up
Parts:
- added C80: 1uF, Capacitor_SMD:C_0402_1005Metric_Pad0.74x0.62mm_HandSolder, F.Cu at (122.0, 110.5)
- added C81: 1uF, Capacitor_SMD:C_0402_1005Metric_Pad0.74x0.62mm_HandSolder, F.Cu at (119.7, 115.1)
- added C82: 0.1uF, Capacitor_SMD:C_0402_1005Metric_Pad0.74x0.62mm_HandSolder, F.Cu at (127.3, 96.5)
- added C83: 0.1uF, Capacitor_SMD:C_0402_1005Metric_Pad0.74x0.62mm_HandSolder, F.Cu at (123.0, 97.0)
- added C84: 0.1uF, Capacitor_SMD:C_0402_1005Metric_Pad0.74x0.62mm_HandSolder, F.Cu at (125.1, 85.1)
- added C85: 0.1uF, Capacitor_SMD:C_0402_1005Metric_Pad0.74x0.62mm_HandSolder, F.Cu at (127.3, 88.6)
- added R79: 3.3K, Capacitor_SMD:C_0402_1005Metric_Pad0.74x0.62mm_HandSolder, F.Cu at (124.4, 93.2)
- added R80: 3.3K, Capacitor_SMD:C_0402_1005Metric_Pad0.74x0.62mm_HandSolder, F.Cu at (124.4, 101.0)
- added R81: 3.3K, Capacitor_SMD:C_0402_1005Metric_Pad0.74x0.62mm_HandSolder, F.Cu at (122.9, 90.6)
- added R82: 402K, Capacitor_SMD:C_0402_1005Metric_Pad0.74x0.62mm_HandSolder, F.Cu at (133.0, 129.8)
- added U14: TXS0102DCU, Package_SO:VSSOP-8_2.3x2mm_P0.5mm, F.Cu at (125.2, 97.0)
- added U15: LP5907MFX-3.3, Package_TO_SOT_SMD:SOT-23-5, F.Cu at (120.2, 112.7)
- added U16: TXS0102DCU, Package_SO:VSSOP-8_2.3x2mm_P0.5mm, F.Cu at (125.1, 88.5)
- moved R10 1.03 mm to (131.9, 129.8)
- moved C8 1.03 mm to (130.9, 129.8)
- moved R47 0.44 mm to (127.2, 101.0)
- moved R48 0.44 mm to (126.2, 101.0)
- moved J9 0.41 mm to (113.2, 116.8)
Connections:
- C55 pad 2: Net-(U11-VP) -> DAC_3V3
- C56 pad 1: Net-(U11-VP) -> DAC_3V3
- C62 pad 2: Net-(U12-VP) -> DAC_3V3
- C63 pad 1: Net-(U12-VP) -> DAC_3V3
- R9 pad 1: 5V -> Net-(R82-Pad2)
- U11 pad 1: DAC_SCL -> DAC_SCL_1
- U11 pad 26: Net-(U11-VP) -> DAC_3V3
- U11 pad 36: unconnected-(U11-XTO-Pad36) -> GND
- U11 pad 39: DAC_SDA -> DAC_SDA_1
- U12 pad 1: DAC_SCL -> DAC_SCL_1
- U12 pad 26: Net-(U12-VP) -> DAC_3V3
- U12 pad 27: DAC_INT -> DAC_INT_1
- U12 pad 36: unconnected-(U12-XTO-Pad36) -> GND
- U12 pad 39: DAC_SDA -> DAC_SDA_1
Routing:
- net DAC_INT_1: track 0.00 -> 48.7 mm
- net DAC_SCL_1: track 0.00 -> 46.0 mm, vias 0 -> 2
- net DAC_SDA: track 102.2 -> 56.8 mm, vias 4 -> 2
- net DAC_3V3: track 0.00 -> 44.1 mm, vias 0 -> 2
- net DAC_SDA_1: track 0.00 -> 41.9 mm, vias 0 -> 2
- net DAC_SCL: track 95.6 -> 59.6 mm, vias 4 -> 3
- net 1.8V: track 65.1 -> 97.5 mm
- net DAC_INT: track 76.7 -> 54.0 mm
- net SYS: track 75.7 -> 64.4 mm, vias 12 -> 13
- net Net-(U12-VP): track 4.00 -> 0.00 mm
- net 5V: track 220.5 -> 224.4 mm
- net Net-(U11-VP): track 3.48 -> 0.00 mm
- net 3.3V: track 285.4 -> 287.6 mm, vias 19 -> 21
- net Net-(R82-Pad2): track 0.00 -> 1.58 mm
- net DAC_RESET: track 72.2 -> 70.8 mm
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
Commit message: up fix lcd pcb
Parts:
- removed C38: 0.1uF, Capacitor_SMD:C_0402_1005Metric_Pad0.74x0.62mm_HandSolder
- R82: value 402K -> 12K
- R9: value 402K -> 390K
- moved C37 14.0 mm to (172.7, 120.9)
Connections:
- P1 pad 10: LCD_CLK -> LCD_EN
- P1 pad 11: GND -> LCD_CLK
- P1 pad 12: LCD_D7 -> GND
- P1 pad 13: LCD_D6 -> LCD_D7
- P1 pad 14: LCD_D5 -> LCD_D6
- P1 pad 15: LCD_D4 -> LCD_D5
- P1 pad 16: LCD_D3 -> LCD_D4
- P1 pad 17: LCD_D2 -> LCD_D3
- P1 pad 18: LCD_D1 -> LCD_D2
- P1 pad 19: LCD_D0 -> LCD_D1
- P1 pad 20: LCD_D15 -> LCD_D0
- P1 pad 21: LCD_D14 -> LCD_D15
- P1 pad 22: LCD_D13 -> LCD_D14
- P1 pad 23: LCD_D12 -> LCD_D13
- P1 pad 24: LCD_D11 -> LCD_D12
- P1 pad 25: LCD_D10 -> LCD_D11
- P1 pad 26: LCD_D9 -> LCD_D10
- P1 pad 27: LCD_D8 -> LCD_D9
- P1 pad 28: LCD_D23 -> LCD_D8
- P1 pad 29: LCD_D22 -> LCD_D23
- P1 pad 30: LCD_D21 -> LCD_D22
- P1 pad 31: LCD_D20 -> LCD_D21
- P1 pad 32: LCD_D19 -> LCD_D20
- P1 pad 33: LCD_D18 -> LCD_D19
- P1 pad 34: LCD_D17 -> LCD_D18
- P1 pad 35: (no net) -> LCD_D17
- P1 pad 6: LCD_DE -> unconnected-(P1-NC-Pad6)
- P1 pad 7: LCD_VSYNC -> LCD_DE
- P1 pad 8: LCD_HSYNC -> LCD_VSYNC
- P1 pad 9: 3.3V -> LCD_HSYNC
- U1 pad 62: unconnected-(U1-SAI3_SDI/DSM_AUD_LN_M1/ETH_RMII0_MDC/GPIO2_B6_d-Pad62) -> LCD_EN
Routing:
- net LCD_EN: track 0.00 -> 56.8 mm, vias 0 -> 4
- net LCD_D17: track 21.8 -> 19.4 mm
- net LCD_D15: track 14.4 -> 12.0 mm
- net LCD_D14: track 14.4 -> 12.3 mm
- net LCD_D18: track 21.8 -> 19.8 mm
- net LCD_D13: track 14.4 -> 12.5 mm
- net LCD_D19: track 21.8 -> 20.0 mm
- net 3.3V: track 287.6 -> 285.8 mm, vias 21 -> 20
- net LCD_D12: track 14.4 -> 12.8 mm
- net LCD_D11: track 14.4 -> 13.5 mm
- net LCD_D10: track 14.4 -> 13.7 mm
- net 1.8V: track 97.5 -> 98.1 mm
Other:
- board text added: "ColorAudio v2.3"
- board text removed: "ColorAudio v2.1"

Commit message: up
Parts:
- removed Q3: PMOS, coloryr:SOT-23
- removed Q4: NPN, coloryr:SOT-23
- removed R38: 10K, Resistor_SMD:R_0402_1005Metric_Pad0.72x0.64mm_HandSolder
- removed R41: 100K, Resistor_SMD:R_0402_1005Metric_Pad0.72x0.64mm_HandSolder
- added C38: 0.1uF, Capacitor_SMD:C_0402_1005Metric_Pad0.74x0.62mm_HandSolder, F.Cu at (135.0, 104.3)
- R25: value 100K -> 100K/NC
- R39: value 10K -> 100K
- R40: value 100K -> 150K
- moved R39 4.21 mm to (182.9, 114.3)
- turned R40 to 180 degrees
Connections:
- P1 pad 1: unconnected-(P1-Y2-Pad1) -> LCD_Y2
- P1 pad 2: unconnected-(P1-X2-Pad2) -> LCD_X2
- P1 pad 3: unconnected-(P1-Y1-Pad3) -> LCD_Y1
- P1 pad 4: unconnected-(P1-X1-Pad4) -> LCD_X1
- R39 pad 2: Net-(Q4-B) -> USB_DET
Routing:
- net Net-(Q3-G): track 9.66 -> 0.00 mm
- net Net-(Q4-B): track 8.22 -> 0.00 mm
- net LCD_D16: track 19.3 -> 22.0 mm
- net LCD_D17: track 19.4 -> 22.0 mm
- net USB0_DP: track 53.0 -> 50.6 mm
- net USB0_DM: track 52.9 -> 50.6 mm
- net USB_DET: track 52.4 -> 54.6 mm
- net LCD_D18: track 19.8 -> 22.0 mm
- net LCD_D15: track 12.0 -> 14.2 mm
- net LCD_D19: track 20.0 -> 22.0 mm
- net LCD_D14: track 12.3 -> 14.2 mm
- net LCD_D13: track 12.5 -> 14.2 mm
- net 1.8V: track 98.1 -> 96.6 mm
- net LCD_D1: track 27.3 -> 28.8 mm
- net LCD_D12: track 12.8 -> 14.2 mm
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
Commit message: up
Parts:
- removed the C32 at (130.0, 114.7)
- C34: renamed from C31; value 10uF -> 1uF
- C44: renamed from C41; value 0.1uF -> 4.7uF
- C45: renamed from C42; value 10uF -> 0.1uF
- C47: renamed from C39; value 4.7uF -> 10uF
- C69: renamed from C56; value 10uF -> 0.1uF
- C70: renamed from C55; value 0.1uF -> 10uF
- C82: renamed from C78; value 10uF -> 1.0uF
- C83: renamed from C77; value 1.0uF -> 10uF
- R28, R29: value 10K -> 4.7K
- R30, R31, R32, R33: value 47K -> 4.7K
- moved J4 3.47 mm to (197.6, 121.9), turned to 180 degrees
- moved C33 1.00 mm to (128.8, 114.2)
- moved C34 1.00 mm to (129.9, 114.2)
- moved USB1 0.74 mm to (190.6, 115.0)
- turned C69 to 90 degrees
- turned C70 to -90 degrees
- renumbered C5 to C10, C7 to C11, C9 to C12, C11 to C13, C13 to C14, C17 to C15, C18 to C16, C19 to C17, C21 to C18, C24 to C19, C22 to C20, C81 to C21, C80 to C22, C6 to C23, C8 to C24, C10 to C25, C12 to C26, C14 to C27, C30 to C29, C26 to C30, C27 to C31, C29 to C32, C34 to C35, C35 to C36, C36 to C37, C37 to C38, C38 to C39, C83 to C40, C84 to C41, C82 to C42, C85 to C43, C40 to C46, C43 to C48, C44 to C49, C15 to C5, C47 to C50, C48 to C51, C50 to C52, C62 to C55, C63 to C56, C64 to C57, C65 to C58, C66 to C59, C16 to C6, C67 to C60, C68 to C61, C71 to C62, C72 to C63, C45 to C64, C46 to C65, C49 to C66, C51 to C67, C52 to C68, C23 to C7, C57 to C71, C58 to C72, C59 to C73, C60 to C74, C61 to C75, C69 to C76, C70 to C77, C73 to C78, C74 to C79, C20 to C8, C75 to C80, C76 to C81, C79 to C84, C25 to C9, D6 to D4, D7 to D5, D4 to D6, D5 to D7, J8 to J10, J5 to J11, J14 to J12, J10 to J13, J6 to J5, J9 to J6, J16 to J7, J17 to J8, J7 to J9, L2 to L1, L3 to L2, L1 to L3, R21 to R10, R22 to R11, R78 to R12, R12 to R13, R13 to R14, R17 to R15, R19 to R16, R20 to R17, R23 to R18, R24 to R19, R6 to R2, R25 to R20, R26 to R21, R14 to R22, R82 to R23, R9 to R24, R10 to R25, R15 to R26, R16 to R27, R2 to R3, R42 to R34, R43 to R35, R44 to R36, R45 to R37, R46 to R38, R47 to R39, R3 to R4, R48 to R40, R49 to R41, R50 to R42, R51 to R43, R35 to R44, R52 to R45, R53 to R46, R54 to R47, R27 to R48, R34 to R49, R4 to R5, R36 to R50, R37 to R51, R39 to R52, R40 to R53, R80 to R54, R81 to R55, R79 to R56, R55 to R57, R56 to R58, R5 to R6, R63 to R61, R64 to R62, R57 to R63, R58 to R64, R61 to R65, R62 to R66, R65 to R67, R66 to R68, R67 to R69, R68 to R70, R76 to R71, R77 to R72, R69 to R73, R70 to R74, R71 to R75, R72 to R76, R73 to R77, R74 to R78, R75 to R79, R11 to R80, R18 to R9, U9 to U10, U14 to U11, U16 to U12, U10 to U13, U12 to U14, U11 to U15, U13 to U16, U4 to U2, U6 to U3, U5 to U4, U3 to U5, U15 to U6, U2 to U7, U7 to U8, U8 to U9
Connections:
- C33 pad 2: 5V -> 3.3V
- C69 pad 1: DAC_3V3 -> GND
- C69 pad 2: GND -> DAC_3V3
- C70 pad 1: GND -> DAC_3V3
- C70 pad 2: DAC_3V3 -> GND
- U9 pad 12: 5V -> 3.3V
Routing:
- net 5V: track 224.3 -> 212.4 mm, vias 25 -> 24
- net 3.3V: track 285.0 -> 286.3 mm
