File: pcb/v2/coloryr.kicad_pcb (KiCad board)
At the start: 2 copper layers, 118 x 67 mm, 225 parts, among them J1 Conn_01x02, J10 Conn_01x02, J11 TestPoint, J12 Conn_01x04, J13 Conn_01x05, J2 Conn_01x03, J3 Conn_01x02, J4 Conn_01x02, J5 TestPoint, J6 TestPoint, J7 TestPoint, J8 TestPoint, J9 Conn_01x02, Q1 NPN, Q2 PMOS, U1 SOM3562_18, U10 STI9287, U11 TXS0102DCU, U12 TXS0102DCU, U13 AIC8800, U14 CS43198, U15 CS43198, U16 OPA1622, U2 TLV6213x, U4 BQ25895RTW, U5 LM27762, U6 LP5907MFX-3.3, U7 TPS61230DRC, U8 TCKE812, U9 CH334R, Y1 12M

Commit message: up pcb
Parts:
- added C85: 0.1uF, Capacitor_SMD:C_0402_1005Metric_Pad0.74x0.62mm_HandSolder, F.Cu at (178.3, 106.5)
- added R81: 4.7K, Capacitor_SMD:C_0402_1005Metric_Pad0.74x0.62mm_HandSolder, F.Cu at (135.1, 81.5)
- added R82: 4.7K, Capacitor_SMD:C_0402_1005Metric_Pad0.74x0.62mm_HandSolder, F.Cu at (135.1, 80.4)
- added R83: 4.7K, Capacitor_SMD:C_0402_1005Metric_Pad0.74x0.62mm_HandSolder, F.Cu at (151.8, 113.8)
- added R84: 4.7K, Capacitor_SMD:C_0402_1005Metric_Pad0.74x0.62mm_HandSolder, F.Cu at (140.8, 71.3)
- added R85: 4.7K, Capacitor_SMD:C_0402_1005Metric_Pad0.74x0.62mm_HandSolder, F.Cu at (139.7, 71.3)
- added R86: 0, Resistor_SMD:R_0402_1005Metric_Pad0.72x0.64mm_HandSolder, F.Cu at (180.1, 107.2)
- added R87: 0, Resistor_SMD:R_0402_1005Metric_Pad0.72x0.64mm_HandSolder, F.Cu at (180.1, 115.0)
- added R88: 10K, Capacitor_SMD:C_0402_1005Metric_Pad0.74x0.62mm_HandSolder, F.Cu at (178.2, 115.6)
- added U17: CH422E, Package_SO:MSOP-10_3x3mm_P0.5mm, F.Cu at (179.7, 111.1)
Connections:
- D2 pad 2: USB0_DP -> USB_DP
- D3 pad 2: USB0_DM -> USB_DM
- R7 pad 1: USB0_DM -> USB_DM
- R8 pad 1: USB0_DP -> USB_DP
- U4 pad 2: unconnected-(U4-D+-Pad2) -> BAT_DP
- U4 pad 3: unconnected-(U4-D--Pad3) -> BAT_DM
- U4 pad 4: unconnected-(U4-STAT-Pad4) -> BAT_STAT
Routing:
- net BAT_DM: track 0.00 -> 28.0 mm, vias 0 -> 4
- net 1.8V: track 96.6 -> 122.3 mm, vias 10 -> 12
- net BAT_STAT: track 0.00 -> 20.0 mm, vias 0 -> 2
- net BAT_DP: track 0.00 -> 18.1 mm, vias 0 -> 2
- net 3.3V: track 286.3 -> 297.1 mm, vias 18 -> 21
- net USB_DP: track 0.00 -> 9.30 mm
- net USB_DM: track 0.00 -> 8.96 mm
- net VCC_3V3_OUT: track 13.4 -> 18.3 mm
- net USB0_DM: track 50.6 -> 47.1 mm
- net USB0_DP: track 50.6 -> 47.8 mm
- net DAC_SCLK: track 46.3 -> 48.6 mm
- net DAC_MCLK: track 52.3 -> 54.5 mm
- net DAC_SDIN: track 55.0 -> 57.2 mm
- net BAT_SCL: track 40.6 -> 41.8 mm
- net DAC_LRCK: track 46.1 -> 47.0 mm
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Other:
- board text added: "ColorAudio v2.4"
- board text removed: "ColorAudio v2.3"

Commit message: up
Parts:
- added C86: 0.1uF, Capacitor_SMD:C_0402_1005Metric_Pad0.74x0.62mm_HandSolder, F.Cu at (130.5, 92.8)
- added R89: 0, Resistor_SMD:R_0402_1005Metric_Pad0.72x0.64mm_HandSolder, F.Cu at (132.3, 87.1)
- added R90: 0, Resistor_SMD:R_0402_1005Metric_Pad0.72x0.64mm_HandSolder, F.Cu at (131.1, 87.1)
- added Y2: 24.576M, Oscillator:Oscillator_SMD_ECS_2520MV-xxx-xx-4Pin_2.5x2.0mm, F.Cu at (130.5, 90.3)
- R85: value 4.7K -> 0; footprint Capacitor_SMD:C_0402_1005Metric_Pad0.74x0.62mm_HandSolder -> Resistor_SMD:R_0402_1005Metric_Pad0.72x0.64mm_HandSolder
- moved R85 18.6 mm to (129.8, 87.1)
Connections:
- R85 pad 1: 1.8V -> DAC_MCLK_1
- U1 pad 31: unconnected-(U1-RM_IO8/SPI1_CLK/SAI1_MCLK/GPIO0_B0_d-Pad31) -> DAC_PWM
- U14 pad 37: DAC_MCLK -> DAC_MCLK_1
- U15 pad 37: DAC_MCLK -> DAC_MCLK_1
Routing:
- net DAC_PWM: track 0.00 -> 55.9 mm, vias 0 -> 4
- net DAC_MCLK_1: track 0.00 -> 38.6 mm, vias 0 -> 4
- net DAC_MCLK: track 54.5 -> 18.2 mm, vias 4 -> 2
- net 1.8V: track 122.3 -> 138.6 mm, vias 12 -> 14
- net Net-(Y2-OUT): track 0.00 -> 2.24 mm
- net TP_INT: track 88.5 -> 89.8 mm
- net TP_RESET: track 86.5 -> 87.8 mm
- net RECOVER: track 57.3 -> 58.2 mm
- net GND: vias 186 -> 187

Commit message: up
Parts:
- added J14: TestPoint, TestPoint:TestPoint_Pad_D2.0mm, F.Cu at (124.5, 109.0)
Connections:
- R2 pad 1: GND -> VCC_1V8_OUT
- R57 pad 2: Net-(U13-WIFI_POWER) -> WIFI_PWR
- U1 pad 30: unconnected-(U1-RM_IO9/SPI1_MOSI/SAI1_SCLK/GPIO0_B1_d-Pad30) -> WIFI_PWR
- U13 pad 12: Net-(U13-WIFI_POWER) -> WIFI_PWR
Routing:
- net WIFI_PWR: track 0.00 -> 68.2 mm, vias 0 -> 2
- net VCC_1V8_OUT: track 0.00 -> 34.7 mm, vias 0 -> 2
- net SD_DET: track 43.3 -> 52.0 mm, vias 0 -> 2
- net VCC_3V3_OUT: track 18.3 -> 14.0 mm
- net DAC_3V3: track 44.0 -> 47.7 mm
- net Net-(U13-WIFI_POWER): track 2.87 -> 0.00 mm
- net +INB: track 19.6 -> 20.3 mm
- net TP_SDA: track 94.4 -> 93.8 mm
