File: pcb/v2/io.kicad_sch (KiCad schematic)
At the start: 63 parts, among them J10 Conn_01x05, J14 Conn_01x04, Q3 PNP, Q4 NPN, U7 TCKE812, U8 CH334R, U9 STI9287, Y1 12M

Commit message: up
Parts:
- removed Q3: PNP, coloryr:SOT-23, symbol Simulation_SPICE:PNP
- added Q3: PMOS, coloryr:SOT-23, symbol Simulation_SPICE:PMOS
- R38: value 100K -> 10K
Connections:
- net 3.3V: now also Q3.3 (S)
- net USB_DET: now also Q3.1 (D)
- net at Q4.1 (C), R38.2: now also Q3.2 (G)
Changed lines of the file:
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@@
 	)
 	(symbol
-		(lib_id "Simulation_SPICE:PNP")
-		(at 133.35 182.88 270)
-		(unit 1)
-		(exclude_from_sim no)
-		(in_bom yes)
-		(on_board yes)
-		(dnp no)
-		(property "Reference" "Q3"
-			(at 127.508 180.848 90)
-			(effects
-				(font
-					(size 1.27 1.27)
-				)
-				(justify left)
-			)
-		)
-		(property "Value" "PNP"
-			(at 134.366 180.594 90)
-			(effects
-				(font
-					(size 1.27 1.27)
-				)
-				(justify left)
-			)
-		)
-		(property "Footprint" "coloryr:SOT-23"
-			(at 133.35 218.44 0)
-			(effects
-				(font
-					(size 1.27 1.27)
-				)
-				(hide yes)
-			)
-		)
-		(property "Datasheet" "https://ngspice.sourceforge.io/docs/ngspice-html-manual/manual.xhtml#cha_BJTs"
-			(at 133.35 218.44 0)
-			(effects
-				(font
-					(size 1.27 1.27)
-				)
-				(hide yes)
-			)
-		)
-		(property "Description" "Bipolar transistor symbol for simulation only, substrate tied to the emitter"
-			(at 133.35 182.88 0)
-			(effects
-				(font
-					(size 1.27 1.27)
-				)
-				(hide yes)
-			)
-		)
-		(property "Sim.Device" "PNP"
-			(at 133.35 182.88 0)
-			(effects
-				(font
-					(size 1.27 1.27)
-				)
-				(hide yes)
-			)
-		)
-		(property "Sim.Type" "GUMMELPOON"
-			(at 133.35 182.88 0)
-			(effects
-				(font
-					(size 1.27 1.27)
-				)
-				(hide yes)
-			)
-		)
-		(property "Sim.Pins" "1=C 2=B 3=E"
-			(at 133.35 182.88 0)
-			(effects
-				(font
-					(size 1.27 1.27)
-				)
-				(hide yes)
-			)
-		)
-		(pin "2"
-		)
-		(pin "1"
-		)
-		(pin "3"
-		)
-		(instances
-			(project "coloryr"
-				(path "/9e6d55f4-a9e8-48fa-bb52-b4e4e3117f8b/d9c616e1-2298-455a-b24a-3007b8e9dd7b"
-					(reference "Q3")
-					(unit 1)
-				)
-			)
-		)
-	)
-	(symbol
 		(lib_id "Device:R")
 		(at 236.22 78.74 0)
@@
 	)
 	(symbol
+		(lib_id "Simulation_SPICE:PMOS")
+		(at 133.35 182.88 270)
+		(unit 1)
+		(exclude_from_sim no)
+		(in_bom yes)
+		(on_board yes)
+		(dnp no)
+		(fields_autoplaced yes)
+		(property "Reference" "Q3"
+			(at 133.35 189.23 90)
+			(effects
+				(font
+					(size 1.27 1.27)
+				)
+			)
+		)
+		(property "Value" "PMOS"
+			(at 133.35 191.77 90)
+			(effects
+				(font
+					(size 1.27 1.27)
+				)
+			)
+		)
+		(property "Footprint" "coloryr:SOT-23"
+			(at 135.89 187.96 0)
+			(effects
+				(font
+					(size 1.27 1.27)
+				)
+				(hide yes)
+			)
+		)
+		(property "Datasheet" "https://ngspice.sourceforge.io/docs/ngspice-html-manual/manual.xhtml#cha_MOSFETs"
+			(at 120.65 182.88 0)
+			(effects
+				(font
+					(size 1.27 1.27)
+				)
+				(hide yes)
+			)
+		)
+		(property "Description" "P-MOSFET transistor, drain/source/gate"
+			(at 133.35 182.88 0)
+			(effects
+				(font
+					(size 1.27 1.27)
+				)
+				(hide yes)
+			)
+		)
+		(property "Sim.Device" "PMOS"
+			(at 116.205 182.88 0)
+			(effects
+				(font
+					(size 1.27 1.27)
+				)
+				(hide yes)
+			)
+		)
+		(property "Sim.Type" "VDMOS"
+			(at 114.3 182.88 0)
+			(effects
+				(font
+					(size 1.27 1.27)
+				)
+				(hide yes)
+			)
+		)
+		(property "Sim.Pins" "1=D 2=G 3=S"
+			(at 118.11 182.88 0)
+			(effects
+				(font
+					(size 1.27 1.27)
+				)
+				(hide yes)
+			)
+		)
+		(pin "3"
+		)
+		(pin "1"
+		)
+		(pin "2"
+		)
+		(instances
+			(project "coloryr"
+				(path "/9e6d55f4-a9e8-48fa-bb52-b4e4e3117f8b/d9c616e1-2298-455a-b24a-3007b8e9dd7b"
+					(reference "Q3")
+					(unit 1)
+				)
+			)
+		)
+	)
+	(symbol
 		(lib_id "Device:R")
 		(at 180.34 30.48 270)
@@
 			)
 		)
-		(property "Value" "100K"
+		(property "Value" "10K"
 			(at 128.524 174.244 90)
 			(effects

Commit message: up
Other:
- note added: "ADC_KEY"
- note removed: "KEY"
- moved on the sheet: R36, R37
Changed lines of the file:
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@@
 	(rectangle
 		(start 16.51 160.02)
-		(end 102.87 193.04)
+		(end 101.6 193.04)
 		(stroke
 			(width 0)
@@
 		)
 	)
-	(text "KEY"
+	(text "ADC_KEY"
 		(exclude_from_sim no)
-		(at 19.812 162.814 0)
+		(at 22.352 162.814 0)
 		(effects
 			(font
@@
 	)
 	(junction
+		(at 69.85 172.72)
+		(diameter 0)
+		(color 0 0 0 0)
+	)
+	(junction
 		(at 81.28 125.73)
 		(diameter 0)
@@
 	)
 	(junction
-		(at 72.39 172.72)
-		(diameter 0)
-		(color 0 0 0 0)
-	)
-	(junction
 		(at 62.23 77.47)
 		(diameter 0)
@@
 	)
 	(junction
-		(at 86.36 180.34)
+		(at 82.55 180.34)
 		(diameter 0)
 		(color 0 0 0 0)
@@
 	(wire
 		(pts
-			(xy 85.09 181.61) (xy 85.09 180.34)
+			(xy 82.55 181.61) (xy 82.55 180.34)
 		)
 		(stroke
@@
 	(wire
 		(pts
-			(xy 67.31 172.72) (xy 72.39 172.72)
+			(xy 67.31 172.72) (xy 69.85 172.72)
 		)
 		(stroke
@@
 	(wire
 		(pts
-			(xy 72.39 172.72) (xy 76.2 172.72)
-		)
-		(stroke
-			(width 0)
-			(type default)
-		)
-	)
-	(wire
-		(pts
 			(xy 80.01 123.19) (xy 86.36 123.19)
 		)
@@
 	(wire
 		(pts
-			(xy 30.48 172.72) (xy 43.18 172.72)
+			(xy 30.48 172.72) (xy 39.37 172.72)
 		)
 		(stroke
@@
 	(wire
 		(pts
-			(xy 97.79 180.34) (xy 96.52 180.34)
+			(xy 93.98 180.34) (xy 92.71 180.34)
 		)
 		(stroke
@@
 	(wire
 		(pts
-			(xy 83.82 172.72) (xy 86.36 172.72)
+			(xy 80.01 172.72) (xy 82.55 172.72)
 		)
 		(stroke
@@
 	(wire
 		(pts
-			(xy 43.18 181.61) (xy 85.09 181.61)
+			(xy 39.37 181.61) (xy 82.55 181.61)
 		)
 		(stroke
@@
 	(wire
 		(pts
-			(xy 43.18 172.72) (xy 43.18 181.61)
+			(xy 39.37 172.72) (xy 39.37 181.61)
 		)
 		(stroke
@@
 	(wire
 		(pts
-			(xy 86.36 180.34) (xy 88.9 180.34)
+			(xy 82.55 180.34) (xy 85.09 180.34)
 		)
 		(stroke
@@
 	(wire
 		(pts
-			(xy 30.48 175.26) (xy 72.39 175.26)
+			(xy 30.48 175.26) (xy 69.85 175.26)
 		)
 		(stroke
@@
 	(wire
 		(pts
+			(xy 69.85 172.72) (xy 72.39 172.72)
+		)
+		(stroke
+			(width 0)
+			(type default)
+		)
+	)
+	(wire
+		(pts
 			(xy 231.14 49.53) (xy 231.14 48.26)
 		)
@@
 	(wire
 		(pts
-			(xy 85.09 180.34) (xy 86.36 180.34)
-		)
-		(stroke
-			(width 0)
-			(type default)
-		)
-	)
-	(wire
-		(pts
 			(xy 80.01 125.73) (xy 81.28 125.73)
 		)
@@
 	(wire
 		(pts
-			(xy 97.79 173.99) (xy 97.79 180.34)
+			(xy 93.98 173.99) (xy 93.98 180.34)
 		)
 		(stroke
@@
 	(wire
 		(pts
-			(xy 72.39 172.72) (xy 72.39 175.26)
+			(xy 69.85 172.72) (xy 69.85 175.26)
 		)
 		(stroke
@@
 	(wire
 		(pts
-			(xy 86.36 172.72) (xy 86.36 180.34)
+			(xy 82.55 172.72) (xy 82.55 180.34)
 		)
 		(stroke
@@
 	(global_label "RECOVER"
 		(shape input)
-		(at 97.79 173.99 90)
+		(at 93.98 173.99 90)
 		(fields_autoplaced yes)
 		(effects
@@
 		)
 		(property "Intersheetrefs" "${INTERSHEET_REFS}"
-			(at 97.79 162.4777 90)
+			(at 93.98 162.4777 90)
 			(effects
 				(font
@@
 	(symbol
 		(lib_id "Device:R")
-		(at 80.01 172.72 270)
+		(at 76.2 172.72 270)
 		(unit 1)
 		(exclude_from_sim no)
@@
 		(dnp no)
 		(property "Reference" "R36"
-			(at 82.042 175.006 90)
+			(at 78.232 175.006 90)
 			(effects
 				(font
@@
 		)
 		(property "Value" "3K"
-			(at 77.216 175.006 90)
+			(at 73.406 175.006 90)
 			(effects
 				(font
@@
 		)
 		(property "Footprint" "Resistor_SMD:R_0402_1005Metric_Pad0.72x0.64mm_HandSolder"
-			(at 80.01 170.942 90)
+			(at 76.2 170.942 90)
 			(effects
 				(font
@@
 		)
 		(property "Datasheet" "~"
-			(at 80.01 172.72 0)
+			(at 76.2 172.72 0)
 			(effects
 				(font
@@
 		)
 		(property "Description" "Resistor"
-			(at 80.01 172.72 0)
+			(at 76.2 172.72 0)
 			(effects
 				(font
@@
 	(symbol
 		(lib_id "Device:R")
-		(at 92.71 180.34 270)
+		(at 88.9 180.34 270)
 		(unit 1)
 		(exclude_from_sim no)
@@
 		(dnp no)
 		(property "Reference" "R37"
-			(at 94.742 182.626 90)
+			(at 90.932 182.626 90)
 			(effects
 				(font
@@
 		)
 		(property "Value" "100"
-			(at 89.916 182.626 90)
+			(at 86.106 182.626 90)
 			(effects
 				(font
@@
 		)
 		(property "Footprint" "Resistor_SMD:R_0402_1005Metric_Pad0.72x0.64mm_HandSolder"
-			(at 92.71 178.562 90)
+			(at 88.9 178.562 90)
 			(effects
 				(font
@@
 		)
 		(property "Datasheet" "~"
-			(at 92.71 180.34 0)
+			(at 88.9 180.34 0)
 			(effects
 				(font
@@
 		)
 		(property "Description" "Resistor"
-			(at 92.71 180.34 0)
+			(at 88.9 180.34 0)
 			(effects
 				(font

Commit message: up fix lcd pcb
Parts:
- removed C38: 0.1uF, Capacitor_SMD:C_0402_1005Metric_Pad0.74x0.62mm_HandSolder, symbol Device:C
Connections:
- net 3.3V: no longer P1.9 (R4)
- net GND: now also P1.12 (GND); no longer P1.11 (R6)
- net LCD_CLK: now also P1.11 (DCLK); no longer P1.10 (R5)
- net LCD_D0: now also P1.20 (B0); no longer P1.19 (G6)
- net LCD_D1: now also P1.19 (B1); no longer P1.18 (G5)
- net LCD_D10: now also P1.26 (G2); no longer P1.25 (B4)
- net LCD_D11: now also P1.25 (G3); no longer P1.24 (B3)
- net LCD_D12: now also P1.24 (G4); no longer P1.23 (B2)
- net LCD_D13: now also P1.23 (G5); no longer P1.22 (B1)
- net LCD_D14: now also P1.22 (G6); no longer P1.21 (B0)
- net LCD_D15: now also P1.21 (G7); no longer P1.20 (G7)
- net LCD_D17: now also P1.35 (R1); no longer P1.34 (DE)
- net LCD_D18: now also P1.34 (R2); no longer P1.33 (VSYNC)
- net LCD_D19: now also P1.33 (R3); no longer P1.32 (HSYNC)
- net LCD_D2: now also P1.18 (B2); no longer P1.17 (G4)
- net LCD_D20: now also P1.32 (R4); no longer P1.31 (DISP)
- net LCD_D21: now also P1.31 (R5); no longer P1.30 (DCLK)
- net LCD_D22: now also P1.30 (R6); no longer P1.29 (GND)
- net LCD_D23: now also P1.29 (R7); no longer P1.28 (B7)
- net LCD_D3: now also P1.17 (B3); no longer P1.16 (G3)
- net LCD_D4: now also P1.16 (B4); no longer P1.15 (G2)
- net LCD_D5: now also P1.15 (B5); no longer P1.14 (G1)
- net LCD_D6: now also P1.14 (B6); no longer P1.13 (G0)
- net LCD_D7: now also P1.13 (B7); no longer P1.12 (R7)
- net LCD_D8: now also P1.28 (G0); no longer P1.27 (B6)
- net LCD_D9: now also P1.27 (G1); no longer P1.26 (B5)
- net LCD_DE: now also P1.7 (DE); no longer P1.6 (R1)
- net LCD_HSYNC: now also P1.9 (HSYNC); no longer P1.8 (R3)
- net LCD_VSYNC: now also P1.8 (VSYNC); no longer P1.7 (R2)
- new net LCD_EN: P1.10 (DISP)
Other:
- moved on the sheet: R27, R37

Commit message: up
Parts:
- removed Q3: PMOS, coloryr:SOT-23, symbol Simulation_SPICE:PMOS
- removed Q4: NPN, coloryr:SOT-23, symbol Simulation_SPICE:NPN
- removed R38: 10K, Resistor_SMD:R_0402_1005Metric_Pad0.72x0.64mm_HandSolder, symbol Device:R
- removed R41: 100K, Resistor_SMD:R_0402_1005Metric_Pad0.72x0.64mm_HandSolder, symbol Device:R
- added C38: 0.1uF, Capacitor_SMD:C_0402_1005Metric_Pad0.74x0.62mm_HandSolder, symbol Device:C
- R39: value 10K -> 100K
- R40: value 100K -> 150K
Connections:
- net GND: now also C38.2
- net USB_DET: now also R39.2, C38.1
- net LCD_Y2: now reaches P1.1 (Y2)
- net LCD_X2: now reaches P1.2 (X2)
- net LCD_Y1: now reaches P1.3 (Y1)
- net LCD_X1: now reaches P1.4 (X1)
Other:
- note added: "USB_HOST"
- note added: "VCC_RES"
- note removed: "USB-TypeA"
- moved on the sheet: R39, R40

Commit message: up
Parts:
- removed C32: 0.1uF, Capacitor_SMD:C_0402_1005Metric_Pad0.74x0.62mm_HandSolder, symbol Device:C
- C33: renamed from C31; value 10uF -> 1uF
- R28, R29: value 10K -> 4.7K
- R30, R31, R32, R33: value 47K -> 4.7K
- renumbered C30 to C29, C26 to C30, C27 to C31, C29 to C32, C33 to C34, C34 to C35, C35 to C36, C36 to C37, C37 to C38, C38 to C39, J14 to J12, J10 to J13, R42 to R34, R43 to R35, R44 to R36, R45 to R37, R46 to R38, R47 to R39, R48 to R40, R49 to R41, R50 to R42, R51 to R43, R35 to R44, R52 to R45, R53 to R46, R54 to R47, R27 to R48, R34 to R49, R36 to R50, R37 to R51, R39 to R52, R40 to R53, U9 to U10, U7 to U8, U8 to U9
Connections:
- net 3.3V: now also C34.2, U9.12 (V5)
- net 5V: no longer C34.2, U9.12 (V5)
Other:
- moved on the sheet: C33

Commit message: up pcb
Parts:
- added R83: 4.7K, Capacitor_SMD:C_0402_1005Metric_Pad0.74x0.62mm_HandSolder, symbol Device:R
Connections:
- net 3.3V: now also R83.1
- net LCD_EN: now also R83.2
Other:
- moved on the sheet: R34, R35, R36, R37, R38, R39, R40, R41, R42, R43
