File: pcb/v2/dac.kicad_sch (KiCad schematic)
At the start: 61 parts, among them U11 CS43198, U12 CS43198, U13 OPA1622

Commit message: up
Connections:
- net 3.3V: now reaches C55.2, C56.1, U11.26 (VP)
- net 3.3V: now also C62.2, C63.1, U12.26 (VP)
Changed lines of the file:
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@@
 	)
 	(junction
+		(at 142.24 29.21)
+		(diameter 0)
+		(color 0 0 0 0)
+	)
+	(junction
 		(at 224.79 118.11)
 		(diameter 0)
@@
 	)
 	(junction
+		(at 142.24 116.84)
+		(diameter 0)
+		(color 0 0 0 0)
+	)
+	(junction
 		(at 242.57 48.26)
 		(diameter 0)
@@
 	(wire
 		(pts
-			(xy 135.89 29.21) (xy 153.67 29.21)
+			(xy 135.89 29.21) (xy 142.24 29.21)
 		)
 		(stroke
@@
 	(wire
 		(pts
+			(xy 143.51 20.32) (xy 142.24 20.32)
+		)
+		(stroke
+			(width 0)
+			(type default)
+		)
+	)
+	(wire
+		(pts
 			(xy 209.55 40.64) (xy 215.9 40.64)
 		)
@@
 	(wire
 		(pts
+			(xy 142.24 20.32) (xy 142.24 29.21)
+		)
+		(stroke
+			(width 0)
+			(type default)
+		)
+	)
+	(wire
+		(pts
 			(xy 242.57 55.88) (xy 242.57 48.26)
 		)
@@
 	(wire
 		(pts
+			(xy 142.24 106.68) (xy 142.24 116.84)
+		)
+		(stroke
+			(width 0)
+			(type default)
+		)
+	)
+	(wire
+		(pts
 			(xy 76.2 168.91) (xy 86.36 168.91)
 		)
@@
 	(wire
 		(pts
+			(xy 142.24 116.84) (xy 152.4 116.84)
+		)
+		(stroke
+			(width 0)
+			(type default)
+		)
+	)
+	(wire
+		(pts
 			(xy 134.62 140.97) (xy 149.86 140.97)
 		)
@@
 	(wire
 		(pts
-			(xy 134.62 116.84) (xy 152.4 116.84)
+			(xy 134.62 116.84) (xy 142.24 116.84)
 		)
 		(stroke
@@
 	(wire
 		(pts
+			(xy 142.24 29.21) (xy 153.67 29.21)
+		)
+		(stroke
+			(width 0)
+			(type default)
+		)
+	)
+	(wire
+		(pts
 			(xy 240.03 26.67) (xy 240.03 43.18)
 		)
@@
 	(wire
 		(pts
+			(xy 143.51 106.68) (xy 142.24 106.68)
+		)
+		(stroke
+			(width 0)
+			(type default)
+		)
+	)
+	(wire
+		(pts
 			(xy 83.82 29.21) (xy 87.63 29.21)
 		)
@@
 	)
 	(symbol
+		(lib_id "power:VCC")
+		(at 143.51 20.32 270)
+		(unit 1)
+		(exclude_from_sim no)
+		(in_bom yes)
+		(on_board yes)
+		(dnp no)
+		(fields_autoplaced yes)
+		(property "Reference" "#PWR045"
+			(at 139.7 20.32 0)
+			(effects
+				(font
+					(size 1.27 1.27)
+				)
+				(hide yes)
+			)
+		)
+		(property "Value" "3.3V"
+			(at 147.32 20.3199 90)
+			(effects
+				(font
+					(size 1.27 1.27)
+				)
+				(justify left)
+			)
+		)
+		(property "Footprint" ""
+			(at 143.51 20.32 0)
+			(effects
+				(font
+					(size 1.27 1.27)
+				)
+				(hide yes)
+			)
+		)
+		(property "Datasheet" ""
+			(at 143.51 20.32 0)
+			(effects
+				(font
+					(size 1.27 1.27)
+				)
+				(hide yes)
+			)
+		)
+		(property "Description" "Power symbol creates a global label with name \"VCC\""
+			(at 143.51 20.32 0)
+			(effects
+				(font
+					(size 1.27 1.27)
+				)
+				(hide yes)
+			)
+		)
+		(pin "1"
+		)
+		(instances
+			(project "coloryr"
+				(path "/9e6d55f4-a9e8-48fa-bb52-b4e4e3117f8b/8a8efada-1d6d-4bcc-828e-939af60bb626"
+					(reference "#PWR045")
+					(unit 1)
+				)
+			)
+		)
+	)
+	(symbol
 		(lib_id "Device:C")
 		(at 160.02 142.24 270)
@@
 					(unit 1)
 				)
+			)
+		)
+	)
+	(symbol
+		(lib_id "power:VCC")
+		(at 143.51 106.68 270)
+		(unit 1)
+		(exclude_from_sim no)
+		(in_bom yes)
+		(on_board yes)
+		(dnp no)
+		(fields_autoplaced yes)
+		(property "Reference" "#PWR057"
+			(at 139.7 106.68 0)
+			(effects
+				(font
+					(size 1.27 1.27)
+				)
+				(hide yes)
+			)
+		)
+		(property "Value" "3.3V"
+			(at 147.32 106.6799 90)
+			(effects
+				(font
+					(size 1.27 1.27)
+				)
+				(justify left)
+			)
+		)
+		(property "Footprint" ""
+			(at 143.51 106.68 0)
+			(effects
+				(font
+					(size 1.27 1.27)
+				)
+				(hide yes)
+			)
+		)
+		(property "Datasheet" ""
+			(at 143.51 106.68 0)
+			(effects
+				(font
+					(size 1.27 1.27)
+				)
+				(hide yes)
+			)
+		)
+		(property "Description" "Power symbol creates a global label with name \"VCC\""
+			(at 143.51 106.68 0)
+			(effects
+				(font
+					(size 1.27 1.27)
+				)
+				(hide yes)
+			)
+		)
+		(pin "1"
+		)
+		(instances
+			(project "coloryr"
+				(path "/9e6d55f4-a9e8-48fa-bb52-b4e4e3117f8b/8a8efada-1d6d-4bcc-828e-939af60bb626"
+					(reference "#PWR057")
+					(unit 1)
+				)

Commit message: up
Connections:
- net GND: now also U11.36 (XTO), U12.36 (XTO)
- net 3.3V renamed DAC_3V3
- net DAC_INT renamed DAC_INT_1
- net DAC_SCL renamed DAC_SCL_1
- net DAC_SDA renamed DAC_SDA_1

Commit message: up
Parts:
- renumbered C47 to C50, C48 to C51, C50 to C52, C62 to C55, C63 to C56, C64 to C57, C65 to C58, C66 to C59, C67 to C60, C68 to C61, C71 to C62, C72 to C63, C45 to C64, C46 to C65, C49 to C66, C51 to C67, C52 to C68, C55 to C69, C56 to C70, C57 to C71, C58 to C72, C59 to C73, C60 to C74, C61 to C75, C69 to C76, C70 to C77, C73 to C78, C74 to C79, C75 to C80, C76 to C81, C77 to C82, C78 to C83, C79 to C84, R63 to R61, R64 to R62, R57 to R63, R58 to R64, R61 to R65, R62 to R66, R65 to R67, R66 to R68, R67 to R69, R68 to R70, R76 to R71, R77 to R72, R69 to R73, R70 to R74, R71 to R75, R72 to R76, R73 to R77, R74 to R78, R75 to R79, R11 to R80, U12 to U14, U11 to U15, U13 to U16

Commit message: up
Connections:
- net DAC_MCLK renamed DAC_MCLK_1
Changed lines of the file:
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@@
 		)
 	)
-	(global_label "DAC_MCLK"
+	(global_label "DAC_MCLK_1"
 		(shape input)
 		(at 76.2 137.16 180)
@@
 		)
 		(property "Intersheetrefs" "${INTERSHEET_REFS}"
-			(at 63.5991 137.16 0)
+			(at 61.422 137.16 0)
 			(effects
 				(font
@@
 		)
 	)
-	(global_label "DAC_MCLK"
+	(global_label "DAC_MCLK_1"
 		(shape input)
 		(at 77.47 49.53 180)
@@
 		)
 		(property "Intersheetrefs" "${INTERSHEET_REFS}"
-			(at 64.8691 49.53 0)
-			(effects
-				(font
+			(at 62.692 49.53 0)
+			(effects
+				(font
