File: pcb/v2/power.kicad_sch (KiCad schematic)
At the start: 67 parts, among them J16 TestPoint, J17 TestPoint, J4 Conn_01x02, J5 TestPoint, J6 TestPoint, J7 Conn_01x02, J8 Conn_01x02, J9 TestPoint, Q1 NPN, Q2 PNP, U2 TPS61230DRC, U3 LM27762, U4 TLV6213x, U5 BQ25895RTW

Commit message: up
Parts:
- removed Q2: PNP, coloryr:SOT-23, symbol Simulation_SPICE:PNP
- added Q2: PMOS, coloryr:SOT-23, symbol Simulation_SPICE:PMOS
- added R14: 10K, Resistor_SMD:R_0402_1005Metric_Pad0.72x0.64mm_HandSolder, symbol Device:R
- R17: value 100K -> 260
- R24: value 100K -> 10K
Connections:
- net GND: now also R14.2
- net POWER_EN: now also Q2.1 (D), R14.1
- net SYS: now also Q2.3 (S)
- net at D7.2 (A), Q1.1 (C), R24.2: now also Q2.2 (G)
Other:
- moved on the sheet: C10, C12, C14, C6, C8, L1, R10, R9, U2

Commit message: up
Parts:
- added R82: 402K, Capacitor_SMD:C_0402_1005Metric_Pad0.74x0.62mm_HandSolder, symbol Device:R
Connections:
- net 5V: now also R82.1; no longer R9.1
- new net: R82.2, R9.1
Changed lines of the file:
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@@
 	)
 	(junction
+		(at 88.9 161.29)
+		(diameter 0)
+		(color 0 0 0 0)
+	)
+	(junction
 		(at 78.74 107.95)
 		(diameter 0)
@@
 	)
 	(junction
-		(at 88.9 161.29)
-		(diameter 0)
-		(color 0 0 0 0)
-	)
-	(junction
 		(at 193.04 50.8)
 		(diameter 0)
@@
 	)
 	(junction
-		(at 81.28 163.83)
-		(diameter 0)
-		(color 0 0 0 0)
-	)
-	(junction
 		(at 53.34 130.81)
 		(diameter 0)
@@
 	)
 	(junction
+		(at 81.28 154.94)
+		(diameter 0)
+		(color 0 0 0 0)
+	)
+	(junction
 		(at 120.65 105.41)
 		(diameter 0)
@@
 	(wire
 		(pts
-			(xy 81.28 163.83) (xy 81.28 161.29)
-		)
-		(stroke
-			(width 0)
-			(type default)
-		)
-	)
-	(wire
-		(pts
 			(xy 66.04 110.49) (xy 67.31 110.49)
 		)
@@
 	(wire
 		(pts
+			(xy 81.28 154.94) (xy 81.28 156.21)
+		)
+		(stroke
+			(width 0)
+			(type default)
+		)
+	)
+	(wire
+		(pts
 			(xy 82.55 130.81) (xy 71.12 130.81)
 		)
@@
 	(wire
 		(pts
-			(xy 81.28 163.83) (xy 81.28 165.1)
-		)
-		(stroke
-			(width 0)
-			(type default)
-		)
-	)
-	(wire
-		(pts
 			(xy 78.74 118.11) (xy 72.39 118.11)
 		)
@@
 	(wire
 		(pts
+			(xy 76.2 163.83) (xy 76.2 154.94)
+		)
+		(stroke
+			(width 0)
+			(type default)
+		)
+	)
+	(wire
+		(pts
 			(xy 66.04 115.57) (xy 77.47 115.57)
 		)
@@
 	(wire
 		(pts
+			(xy 88.9 161.29) (xy 88.9 154.94)
+		)
+		(stroke
+			(width 0)
+			(type default)
+		)
+	)
+	(wire
+		(pts
 			(xy 247.65 104.14) (xy 247.65 105.41)
 		)
@@
 	(wire
 		(pts
-			(xy 72.39 163.83) (xy 81.28 163.83)
-		)
-		(stroke
-			(width 0)
-			(type default)
-		)
-	)
-	(wire
-		(pts
 			(xy 99.06 162.56) (xy 99.06 161.29)
 		)
@@
 	(wire
 		(pts
+			(xy 88.9 154.94) (xy 81.28 154.94)
+		)
+		(stroke
+			(width 0)
+			(type default)
+		)
+	)
+	(wire
+		(pts
 			(xy 240.03 93.98) (xy 240.03 105.41)
 		)
@@
 	(wire
 		(pts
+			(xy 72.39 163.83) (xy 76.2 163.83)
+		)
+		(stroke
+			(width 0)
+			(type default)
+		)
+	)
+	(wire
+		(pts
 			(xy 254 38.1) (xy 264.16 38.1)
 		)
@@
 	(wire
 		(pts
+			(xy 81.28 163.83) (xy 81.28 165.1)
+		)
+		(stroke
+			(width 0)
+			(type default)
+		)
+	)
+	(wire
+		(pts
 			(xy 161.29 140.97) (xy 170.18 140.97)
 		)
@@
 	(wire
 		(pts
+			(xy 76.2 154.94) (xy 81.28 154.94)
+		)
+		(stroke
+			(width 0)
+			(type default)
+		)
+	)
+	(wire
+		(pts
 			(xy 200.66 102.87) (xy 200.66 110.49)
 		)
@@
 	(wire
 		(pts
-			(xy 81.28 161.29) (xy 88.9 161.29)
-		)
-		(stroke
-			(width 0)
-			(type default)
-		)
-	)
-	(wire
-		(pts
 			(xy 200.66 120.65) (xy 191.77 120.65)
 		)
@@
 					(unit 1)
 				)
+			)
+		)
+	)
+	(symbol
+		(lib_id "Device:R")
+		(at 81.28 160.02 0)
+		(unit 1)
+		(exclude_from_sim no)
+		(in_bom yes)
+		(on_board yes)
+		(dnp no)
+		(property "Reference" "R82"
+			(at 80.264 158.75 0)
+			(effects
+				(font
+					(size 1.27 1.27)
+				)
+				(justify right)
+			)
+		)
+		(property "Value" "402K"
+			(at 87.884 161.798 0)
+			(effects
+				(font
+					(size 1.27 1.27)
+				)
+				(justify right)
+			)
+		)
+		(property "Footprint" "Capacitor_SMD:C_0402_1005Metric_Pad0.74x0.62mm_HandSolder"
+			(at 79.502 160.02 90)
+			(effects
+				(font
+					(size 1.27 1.27)
+				)
+				(hide yes)
+			)
+		)
+		(property "Datasheet" "~"
+			(at 81.28 160.02 0)
+			(effects
+				(font
+					(size 1.27 1.27)
+				)
+				(hide yes)
+			)
+		)
+		(property "Description" "Resistor"
+			(at 81.28 160.02 0)
+			(effects
+				(font
+					(size 1.27 1.27)
+				)
+				(hide yes)
+			)
+		)
+		(pin "2"
+		)
+		(pin "1"
+		)
+		(instances
+			(project "coloryr"
+				(path "/9e6d55f4-a9e8-48fa-bb52-b4e4e3117f8b/45b885e8-026d-42f0-9271-c60672108a75"
+					(reference "R82")
+					(unit 1)
+				)

Commit message: up fix lcd pcb
Parts:
- added C80, C81: 1uF, Capacitor_SMD:C_0402_1005Metric_Pad0.74x0.62mm_HandSolder, symbol Device:C
- added U15: LP5907MFX-3.3, Package_TO_SOT_SMD:SOT-23-5, symbol Regulator_Linear:LP5907MFX-3.3
- R82: value 402K -> 12K
- R9: value 402K -> 390K
Connections:
- net 5V: now also C81.1, U15.1 (IN), U15.3 (EN)
- net GND: now also C80.2, C81.2, U15.2 (GND)
- new net DAC_3V3: C80.1, U15.5 (OUT)
Other:
- note added: "LDO 1.8V"
- note added: "LDO 3.3V"
- note added: "POWER 5V"
- note added: "POWER LED"
- note removed: "LDO"
- moved on the sheet: C25, D4, D5, D6, D7, J8, Q1, Q2, R15, R16, R23, R24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

Commit message: up
Parts:
- R25: value 100K -> 100K/NC
Changed lines of the file:
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@@
 		(dnp no)
 		(property "Reference" "R25"
-			(at 246.634 112.522 90)
+			(at 246.38 106.68 0)
 			(effects
 				(font
@@
 			)
 		)
-		(property "Value" "100K"
-			(at 246.634 107.696 90)
+		(property "Value" "100K/NC"
+			(at 254.762 113.792 0)
 			(effects
 				(font

Commit message: up
Parts:
- renumbered C5 to C10, C7 to C11, C9 to C12, C11 to C13, C13 to C14, C17 to C15, C18 to C16, C19 to C17, C21 to C18, C22 to C19, C24 to C20, C81 to C21, C80 to C22, C6 to C23, C8 to C24, C10 to C25, C12 to C26, C14 to C27, C15 to C5, C16 to C6, C20 to C7, C23 to C8, C25 to C9, D6 to D4, D7 to D5, D4 to D6, D5 to D7, J8 to J10, J5 to J11, J6 to J5, J9 to J6, J16 to J7, J17 to J8, J7 to J9, L2 to L1, L3 to L2, L1 to L3, R21 to R10, R22 to R11, R78 to R12, R12 to R13, R13 to R14, R17 to R15, R19 to R16, R20 to R17, R23 to R18, R24 to R19, R25 to R20, R26 to R21, R14 to R22, R82 to R23, R9 to R24, R10 to R25, R15 to R26, R16 to R27, R18 to R9, U4 to U2, U6 to U3, U5 to U4, U3 to U5, U15 to U6, U2 to U7
Other:
- moved on the sheet: C21, C22, D4, D5, J10, Q1, Q2, R18, R19, R20, R21, R22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

Commit message: up
Connections:
- net BAT_DP: now reaches U4.2 (D+)
- net BAT_DM: now reaches U4.3 (D-)
- net BAT_STAT: now reaches U4.4 (STAT)
- net USB0_DM renamed USB_DM
- net USB0_DP renamed USB_DP

Commit message: up
Parts:
- added J14: TestPoint, TestPoint:TestPoint_Pad_D2.0mm, symbol Connector_Generic:Conn_01x01
Connections:
- net DAC_3V3: now also J14.1 (Pin_1)
Changed lines of the file:
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@@
 	)
 	(junction
+		(at 259.08 69.85)
+		(diameter 0)
+		(color 0 0 0 0)
+	)
+	(junction
 		(at 193.04 50.8)
 		(diameter 0)
@@
 	(wire
 		(pts
+			(xy 260.35 59.69) (xy 259.08 59.69)
+		)
+		(stroke
+			(width 0)
+			(type default)
+		)
+	)
+	(wire
+		(pts
 			(xy 36.83 69.85) (xy 36.83 71.12)
 		)
@@
 	(wire
 		(pts
-			(xy 256.54 69.85) (xy 262.89 69.85)
+			(xy 256.54 69.85) (xy 259.08 69.85)
 		)
 		(stroke
@@
 	(wire
 		(pts
+			(xy 259.08 59.69) (xy 259.08 69.85)
+		)
+		(stroke
+			(width 0)
+			(type default)
+		)
+	)
+	(wire
+		(pts
 			(xy 137.16 123.19) (xy 140.97 123.19)
 		)
@@
 	(wire
 		(pts
+			(xy 259.08 69.85) (xy 262.89 69.85)
+		)
+		(stroke
+			(width 0)
+			(type default)
+		)
+	)
+	(wire
+		(pts
 			(xy 167.64 49.53) (xy 173.99 49.53)
 		)
@@
 					(unit 1)
 				)
+			)
+		)
+	)
+	(symbol
+		(lib_id "Connector_Generic:Conn_01x01")
+		(at 265.43 59.69 0)
+		(unit 1)
+		(exclude_from_sim no)
+		(in_bom yes)
+		(on_board yes)
+		(dnp no)
+		(property "Reference" "J14"
+			(at 275.082 62.484 0)
+			(effects
+				(font
+					(size 1.27 1.27)
+				)
+				(justify right)
+			)
+		)
+		(property "Value" "TestPoint"
+			(at 278.13 60.198 0)
+			(effects
+				(font
+					(size 1.27 1.27)
+				)
+				(justify right)
+			)
+		)
+		(property "Footprint" "TestPoint:TestPoint_Pad_D2.0mm"
+			(at 265.43 59.69 0)
+			(effects
+				(font
+					(size 1.27 1.27)
+				)
+				(hide yes)
+			)
+		)
+		(property "Datasheet" "~"
+			(at 265.43 59.69 0)
+			(effects
+				(font
+					(size 1.27 1.27)
+				)
+				(hide yes)
+			)
+		)
+		(property "Description" "Generic connector, single row, 01x01, script generated (kicad-library-utils/schlib/autogen/connector/)"
+			(at 265.43 59.69 0)
+			(effects
+				(font
+					(size 1.27 1.27)
+				)
+				(hide yes)
+			)
+		)
+		(pin "1"
+		)
+		(instances
+			(project "coloryr"
+				(path "/9e6d55f4-a9e8-48fa-bb52-b4e4e3117f8b/45b885e8-026d-42f0-9271-c60672108a75"
+					(reference "J14")
+					(unit 1)
+				)
