File: pcb/v2/rk3506.kicad_sch (KiCad schematic)
At the start: 15 parts, among them J1 Conn_01x02, J2 Conn_01x03, J3 Conn_01x02, U1 SOM3562_18

Commit message: up fix lcd pcb
Connections:
- net LCD_EN: now reaches U1.62 (SAI3_SDI/DSM_AUD_LN_M1/ETH_RMII0_MDC/GPIO2_B6_d)
Other:
- moved on the sheet: C1, C2, C3, C4, R1, R6, U1

Commit message: up
Parts:
- renumbered R6 to R2, R2 to R3, R3 to R4, R4 to R5, R5 to R6
Changed lines of the file:
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@@
 		(on_board yes)
 		(dnp no)
-		(property "Reference" "R3"
+		(property "Reference" "R4"
 			(at 146.304 251.206 90)
 			(effects
@@
 			(project "coloryr"
 				(path "/9e6d55f4-a9e8-48fa-bb52-b4e4e3117f8b/a64ce204-e78e-4a81-b82d-779b06b2e2e4"
-					(reference "R3")
+					(reference "R4")
 					(unit 1)
 				)
@@
 		(dnp no)
 		(fields_autoplaced yes)
-		(property "Reference" "#PWR06"
+		(property "Reference" "#PWR08"
 			(at 367.03 140.97 0)
 			(effects
@@
 			(project "coloryr"
 				(path "/9e6d55f4-a9e8-48fa-bb52-b4e4e3117f8b/a64ce204-e78e-4a81-b82d-779b06b2e2e4"
-					(reference "#PWR06")
+					(reference "#PWR08")
 					(unit 1)
 				)
@@
 		(dnp no)
 		(fields_autoplaced yes)
-		(property "Reference" "#PWR010"
+		(property "Reference" "#PWR05"
 			(at 304.8 213.36 0)
 			(effects
@@
 			(project "coloryr"
 				(path "/9e6d55f4-a9e8-48fa-bb52-b4e4e3117f8b/a64ce204-e78e-4a81-b82d-779b06b2e2e4"
-					(reference "#PWR010")
+					(reference "#PWR05")
 					(unit 1)
 				)
@@
 		(dnp no)
 		(fields_autoplaced yes)
-		(property "Reference" "#PWR047"
+		(property "Reference" "#PWR07"
 			(at 356.87 204.47 0)
 			(effects
@@
 			(project "coloryr"
 				(path "/9e6d55f4-a9e8-48fa-bb52-b4e4e3117f8b/a64ce204-e78e-4a81-b82d-779b06b2e2e4"
-					(reference "#PWR047")
+					(reference "#PWR07")
 					(unit 1)
 				)
@@
 		(dnp no)
 		(fields_autoplaced yes)
-		(property "Reference" "#PWR05"
+		(property "Reference" "#PWR06"
 			(at 350.52 220.98 0)
 			(effects
@@
 			(project "coloryr"
 				(path "/9e6d55f4-a9e8-48fa-bb52-b4e4e3117f8b/a64ce204-e78e-4a81-b82d-779b06b2e2e4"
-					(reference "#PWR05")
+					(reference "#PWR06")
 					(unit 1)
 				)
@@
 		(on_board yes)
 		(dnp no)
-		(property "Reference" "R2"
+		(property "Reference" "R3"
 			(at 96.012 248.666 90)
 			(effects
@@
 			(project "coloryr"
 				(path "/9e6d55f4-a9e8-48fa-bb52-b4e4e3117f8b/a64ce204-e78e-4a81-b82d-779b06b2e2e4"
-					(reference "R2")
+					(reference "R3")
 					(unit 1)
 				)
@@
 		(on_board yes)
 		(dnp no)
-		(property "Reference" "R5"
+		(property "Reference" "R6"
 			(at 203.962 248.666 90)
 			(effects
@@
 			(project "coloryr"
 				(path "/9e6d55f4-a9e8-48fa-bb52-b4e4e3117f8b/a64ce204-e78e-4a81-b82d-779b06b2e2e4"
-					(reference "R5")
+					(reference "R6")
 					(unit 1)
 				)
@@
 		(on_board yes)
 		(dnp no)
-		(property "Reference" "R6"
+		(property "Reference" "R2"
 			(at 357.632 143.256 90)
 			(effects
@@
 			(project "coloryr"
 				(path "/9e6d55f4-a9e8-48fa-bb52-b4e4e3117f8b/a64ce204-e78e-4a81-b82d-779b06b2e2e4"
-					(reference "R6")
+					(reference "R2")
 					(unit 1)
 				)
@@
 		(on_board yes)
 		(dnp no)
-		(property "Reference" "R4"
+		(property "Reference" "R5"
 			(at 157.226 241.046 90)
 			(effects
@@
 			(project "coloryr"
 				(path "/9e6d55f4-a9e8-48fa-bb52-b4e4e3117f8b/a64ce204-e78e-4a81-b82d-779b06b2e2e4"
-					(reference "R4")
-					(unit 1)
-				)
+					(reference "R5")
+					(unit 1)
+				)

Commit message: up
Connections:
- net DAC_PWM: now reaches U1.31 (RM_IO8/SPI1_CLK/SAI1_MCLK/GPIO0_B0_d)

Commit message: up
Connections:
- net GND: no longer R2.1
- net VCC_1V8_OUT: now also R2.1
- net WIFI_PWR: now reaches U1.30 (RM_IO9/SPI1_MOSI/SAI1_SCLK/GPIO0_B1_d)
Changed lines of the file:
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@@
+	(wire
+		(pts
+			(xy 342.9 77.47) (xy 353.06 77.47)
+		)
+		(stroke
+			(width 0)
+			(type default)
+		)
+	)
 	(wire
 		(pts
@@
 		)
 	)
+	(global_label "VCC_1V8_OUT"
+		(shape input)
+		(at 360.68 140.97 0)
+		(fields_autoplaced yes)
+		(effects
+			(font
+				(size 1.27 1.27)
+			)
+			(justify left)
+		)
+		(property "Intersheetrefs" "${INTERSHEET_REFS}"
+			(at 376.3652 140.97 0)
+			(effects
+				(font
+					(size 1.27 1.27)
+				)
+				(justify left)
+				(hide yes)
+			)
+		)
+	)
 	(global_label "LCD_DE"
 		(shape input)
@@
 		(property "Intersheetrefs" "${INTERSHEET_REFS}"
 			(at 363.4837 133.35 0)
+			(effects
+				(font
+					(size 1.27 1.27)
+				)
+				(justify left)
+				(hide yes)
+			)
+		)
+	)
+	(global_label "WIFI_PWR"
+		(shape input)
+		(at 353.06 77.47 0)
+		(fields_autoplaced yes)
+		(effects
+			(font
+				(size 1.27 1.27)
+			)
+			(justify left)
+		)
+		(property "Intersheetrefs" "${INTERSHEET_REFS}"
+			(at 364.7538 77.47 0)
 			(effects
 				(font
@@
 					(unit 1)
 				)
-			)
-		)
-	)
-	(symbol
-		(lib_id "power:GND")
-		(at 360.68 140.97 90)
-		(unit 1)
-		(exclude_from_sim no)
-		(in_bom yes)
-		(on_board yes)
-		(dnp no)
-		(fields_autoplaced yes)
-		(property "Reference" "#PWR08"
-			(at 367.03 140.97 0)
-			(effects
-				(font
-					(size 1.27 1.27)
-				)
-				(hide yes)
-			)
-		)
-		(property "Value" "GND"
-			(at 364.49 140.9699 90)
-			(effects
-				(font
-					(size 1.27 1.27)
-				)
-				(justify right)
-			)
-		)
-		(property "Footprint" ""
-			(at 360.68 140.97 0)
-			(effects
-				(font
-					(size 1.27 1.27)
-				)
-				(hide yes)
-			)
-		)
-		(property "Datasheet" ""
-			(at 360.68 140.97 0)
-			(effects
-				(font
-					(size 1.27 1.27)
-				)
-				(hide yes)
-			)
-		)
-		(property "Description" "Power symbol creates a global label with name \"GND\" , ground"
-			(at 360.68 140.97 0)
-			(effects
-				(font
-					(size 1.27 1.27)
-				)
-				(hide yes)
-			)
-		)
-		(pin "1"
-		)
-		(instances
-			(project "coloryr"
-				(path "/9e6d55f4-a9e8-48fa-bb52-b4e4e3117f8b/a64ce204-e78e-4a81-b82d-779b06b2e2e4"
-					(reference "#PWR08")
-					(unit 1)
-				)
