File: pcb/v2(out)/coloryr.kicad_pcb (KiCad board)
At the start: 2 copper layers, 118 x 67 mm, 240 parts, among them J1 Conn_01x02, J10 Conn_01x02, J11 TestPoint, J12 Conn_01x04, J13 Conn_01x05, J14 TestPoint, J2 Conn_01x03, J3 Conn_01x02, J4 Conn_01x02, J5 TestPoint, J6 TestPoint, J7 TestPoint, J8 TestPoint, J9 Conn_01x02, Q1 NPN, Q2 PMOS, U1 SOM3562_18, U10 STI9287, U11 TXS0102DCU, U12 TXS0102DCU, U13 AIC8800, U14 CS43198, U15 CS43198, U16 OPA1622, U17 CH422E, U2 TLV6213x, U4 BQ25895RTW, U5 LM27762, U6 LP5907MFX-3.3, U7 TPS61230DRC, U8 TCKE812, U9 CH334R, Y1 12M, Y2 24.576M

Commit message: up v3
Parts:
- added R91: 0, Resistor_SMD:R_0402_1005Metric_Pad0.72x0.64mm_HandSolder, F.Cu at (112.7, 121.2)
Connections:
- P2 pad 6: TP_RESET -> Net-(P2-SCL)
Routing:
- net TP_RESET: track 87.8 -> 84.1 mm
- net Net-(P2-SCL): track 0.00 -> 3.02 mm
Changed lines of the file:
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@@
 	(net 285 "DAC_PWM")
 	(net 286 "unconnected-(U1-RM_IO10{slash}SPI1_MISO{slash}SAI1_LRCK{slash}GPIO0_B2_d-Pad29)")
+	(net 287 "Net-(P2-SCL)")
 	(footprint "Capacitor_SMD:C_0402_1005Metric_Pad0.74x0.62mm_HandSolder"
 		(layer "F.Cu")
@@
 		)
 	)
+	(footprint "Resistor_SMD:R_0402_1005Metric_Pad0.72x0.64mm_HandSolder"
+		(layer "F.Cu")
+		(at 112.6625 121.15)
+		(descr "Resistor SMD 0402 (1005 Metric), square (rectangular) end terminal, IPC-7351 nominal with elongated pad for handsoldering. (Body size source: IPC-SM-782 page 72, https://www.pcb-3d.com/wordpress/wp-content/uploads/ipc-sm-782a_amendment_1_and_2.pdf), generated with kicad-footprint-generator")
+		(tags "resistor handsolder")
+		(property "Reference" "R91"
+			(at 0 -1.17 0)
+			(layer "F.SilkS")
+			(effects
+				(font
+					(size 1 1)
+					(thickness 0.15)
+				)
+			)
+		)
+		(property "Value" "0"
+			(at 0 1.17 0)
+			(layer "F.Fab")
+			(effects
+				(font
+					(size 1 1)
+					(thickness 0.15)
+				)
+			)
+		)
+		(property "Datasheet" ""
+			(at 0 0 0)
+			(layer "F.Fab")
+			(hide yes)
+			(effects
+				(font
+					(size 1.27 1.27)
+					(thickness 0.15)
+				)
+			)
+		)
+		(property "Description" "Resistor"
+			(at 0 0 0)
+			(layer "F.Fab")
+			(hide yes)
+			(effects
+				(font
+					(size 1.27 1.27)
+					(thickness 0.15)
+				)
+			)
+		)
+		(property ki_fp_filters "R_*")
+		(sheetname "/IO/")
+		(sheetfile "io.kicad_sch")
+		(attr smd)
+		(fp_line
+			(start -0.167621 -0.38)
+			(end 0.167621 -0.38)
+			(stroke
+				(width 0.12)
+				(type solid)
+			)
+			(layer "F.SilkS")
+		)
+		(fp_line
+			(start -0.167621 0.38)
+			(end 0.167621 0.38)
+			(stroke
+				(width 0.12)
+				(type solid)
+			)
+			(layer "F.SilkS")
+		)
+		(fp_line
+			(start -1.11 -0.47)
+			(end 1.11 -0.47)
+			(stroke
+				(width 0.05)
+				(type solid)
+			)
+			(layer "F.CrtYd")
+		)
+		(fp_line
+			(start -1.11 0.47)
+			(end -1.11 -0.47)
+			(stroke
+				(width 0.05)
+				(type solid)
+			)
+			(layer "F.CrtYd")
+		)
+		(fp_line
+			(start 1.11 -0.47)
+			(end 1.11 0.47)
+			(stroke
+				(width 0.05)
+				(type solid)
+			)
+			(layer "F.CrtYd")
+		)
+		(fp_line
+			(start 1.11 0.47)
+			(end -1.11 0.47)
+			(stroke
+				(width 0.05)
+				(type solid)
+			)
+			(layer "F.CrtYd")
+		)
+		(fp_line
+			(start -0.525 -0.27)
+			(end 0.525 -0.27)
+			(stroke
+				(width 0.1)
+				(type solid)
+			)
+			(layer "F.Fab")
+		)
+		(fp_line
+			(start -0.525 0.27)
+			(end -0.525 -0.27)
+			(stroke
+				(width 0.1)
+				(type solid)
+			)
+			(layer "F.Fab")
+		)
+		(fp_line
+			(start 0.525 -0.27)
+			(end 0.525 0.27)
+			(stroke
+				(width 0.1)
+				(type solid)
+			)
+			(layer "F.Fab")
+		)
+		(fp_line
+			(start 0.525 0.27)
+			(end -0.525 0.27)
+			(stroke
+				(width 0.1)
+				(type solid)
+			)
+			(layer "F.Fab")
+		)
+		(fp_text user "${REFERENCE}"
+			(at 0 0 0)
+			(layer "F.Fab")
+			(effects
+				(font
+					(size 0.26 0.26)
+					(thickness 0.04)
+				)
+			)
+		)
+		(pad "1" smd roundrect
+			(at -0.5975 0)
+			(size 0.715 0.64)
+			(layers "F.Cu" "F.Mask" "F.Paste")
+			(roundrect_rratio 0.25)
+			(net 287 "Net-(P2-SCL)")
+			(pintype "passive")
+		)
+		(pad "2" smd roundrect
+			(at 0.5975 0)
+			(size 0.715 0.64)
+			(layers "F.Cu" "F.Mask" "F.Paste")
+			(roundrect_rratio 0.25)
+			(net 62 "TP_RESET")
+			(pintype "passive")
+		)
+		(embedded_fonts no)
+		(model "${KICAD9_3DMODEL_DIR}/Resistor_SMD.3dshapes/R_0402_1005Metric.step"
+			(offset
+				(xyz 0 0 0)
+			)
+			(scale
+				(xyz 1 1 1)
+			)
+			(rotate
+				(xyz 0 0 0)
+			)
+		)
+	)
 	(footprint "Capacitor_SMD:C_0402_1005Metric_Pad0.74x0.62mm_HandSolder"
 		(layer "F.Cu")
@@
 		(tags "connector Hirose FH12 horizontal")
 		(property "Reference" "P2"
-			(at 3.18 -3.73 0)
+			(at -2.74 -3.9 0)
 			(layer "F.SilkS")
 			(effects
@@
 			(size 0.3 1.3)
 			(layers "F.Cu" "F.Mask" "F.Paste")
-			(net 62 "TP_RESET")
+			(net 287 "Net-(P2-SCL)")
 			(pinfunction "SCL")
 			(pintype "input")
@@
 	)
 	(segment
+		(start 115.572374 121.15)
+		(end 116.226187 120.496187)
+		(width 0.12)
+		(layer "F.Cu")
+		(net 62)
+	)
+	(segment
 		(start 132.08 83.034495)
 		(end 133.713 84.667495)
@@
 	(segment
 		(start 128.336376 108.386)
-		(end 113.192374 123.53)
+		(end 116.226187 120.496187)
 		(width 0.12)
 		(layer "F.Cu")
@@
 	)
 	(segment
-		(start 113.192374 123.53)
-		(end 110.53 123.53)
+		(start 113.26 121.15)
+		(end 115.572374 121.15)
 		(width 0.12)
 		(layer "F.Cu")
@@
 		(net 285)
 	)
+	(segment
+		(start 110.53 123.53)
+		(end 110.53 122.685)
+		(width 0.12)
+		(layer "F.Cu")
+		(net 287)
+	)
+	(segment
+		(start 110.53 122.685)
+		(end 112.065 121.15)
+		(width 0.12)
+		(layer "F.Cu")
+		(net 287)
+	)
 	(zone
