File: pcb/v2(out)/io.kicad_sch (KiCad schematic)
At the start: 59 parts, among them J12 Conn_01x04, J13 Conn_01x05, U10 STI9287, U8 TCKE812, U9 CH334R, Y1 12M

Commit message: up v3
Parts:
- added R91: 0, Resistor_SMD:R_0402_1005Metric_Pad0.72x0.64mm_HandSolder, symbol Device:R
Connections:
- net TP_RESET: now also R91.2; no longer P2.6 (SCL)
- new net: P2.6 (SCL), R91.1
Other:
- moved on the sheet: C37
Changed lines of the file:
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@@
 	)
 	(junction
-		(at 223.52 138.43)
-		(diameter 0)
-		(color 0 0 0 0)
-	)
-	(junction
 		(at 59.69 46.99)
 		(diameter 0)
@@
 	)
 	(junction
+		(at 222.25 138.43)
+		(diameter 0)
+		(color 0 0 0 0)
+	)
+	(junction
 		(at 160.02 177.8)
 		(diameter 0)
@@
 	(wire
 		(pts
-			(xy 223.52 138.43) (xy 223.52 130.81)
+			(xy 222.25 144.78) (xy 222.25 138.43)
 		)
 		(stroke
@@
 	(wire
 		(pts
-			(xy 232.41 130.81) (xy 236.22 130.81)
+			(xy 232.41 144.78) (xy 236.22 144.78)
 		)
 		(stroke
@@
 	(wire
 		(pts
+			(xy 236.22 133.35) (xy 240.03 133.35)
+		)
+		(stroke
+			(width 0)
+			(type default)
+		)
+	)
+	(wire
+		(pts
 			(xy 57.15 52.07) (xy 90.17 52.07)
 		)
@@
 	(wire
 		(pts
-			(xy 219.71 138.43) (xy 223.52 138.43)
-		)
-		(stroke
-			(width 0)
-			(type default)
-		)
-	)
-	(wire
-		(pts
-			(xy 250.19 133.35) (xy 259.08 133.35)
+			(xy 219.71 138.43) (xy 222.25 138.43)
 		)
 		(stroke
@@
 	(wire
 		(pts
+			(xy 247.65 133.35) (xy 259.08 133.35)
+		)
+		(stroke
+			(width 0)
+			(type default)
+		)
+	)
+	(wire
+		(pts
 			(xy 236.22 135.89) (xy 259.08 135.89)
 		)
@@
 	(wire
 		(pts
-			(xy 236.22 130.81) (xy 236.22 135.89)
+			(xy 236.22 144.78) (xy 236.22 135.89)
 		)
 		(stroke
@@
 	(wire
 		(pts
-			(xy 223.52 138.43) (xy 259.08 138.43)
+			(xy 177.8 133.35) (xy 184.15 133.35)
 		)
 		(stroke
@@
 	(wire
 		(pts
-			(xy 177.8 133.35) (xy 184.15 133.35)
+			(xy 222.25 138.43) (xy 259.08 138.43)
 		)
 		(stroke
@@
 	(wire
 		(pts
-			(xy 223.52 130.81) (xy 224.79 130.81)
+			(xy 222.25 144.78) (xy 224.79 144.78)
 		)
 		(stroke
@@
 		)
 	)
+	(global_label "TP_RESET"
+		(shape input)
+		(at 236.22 133.35 180)
+		(fields_autoplaced yes)
+		(effects
+			(font
+				(size 1.27 1.27)
+			)
+			(justify right)
+		)
+		(property "Intersheetrefs" "${INTERSHEET_REFS}"
+			(at 224.2845 133.35 0)
+			(effects
+				(font
+					(size 1.27 1.27)
+				)
+				(justify right)
+				(hide yes)
+			)
+		)
+	)
 	(global_label "DAC_SCL"
 		(shape input)
@@
 		)
 	)
-	(global_label "TP_RESET"
-		(shape input)
-		(at 250.19 133.35 180)
-		(fields_autoplaced yes)
-		(effects
-			(font
-				(size 1.27 1.27)
-			)
-			(justify right)
-		)
-		(property "Intersheetrefs" "${INTERSHEET_REFS}"
-			(at 238.2545 133.35 0)
-			(effects
-				(font
-					(size 1.27 1.27)
-				)
-				(justify right)
-				(hide yes)
-			)
-		)
-	)
 	(global_label "LCD_D1"
 		(shape input)
@@
 	)
 	(symbol
+		(lib_id "Device:R")
+		(at 243.84 133.35 270)
+		(unit 1)
+		(exclude_from_sim no)
+		(in_bom yes)
+		(on_board yes)
+		(dnp no)
+		(property "Reference" "R91"
+			(at 242.57 131.064 90)
+			(effects
+				(font
+					(size 1.27 1.27)
+				)
+			)
+		)
+		(property "Value" "0"
+			(at 246.126 131.064 90)
+			(effects
+				(font
+					(size 1.27 1.27)
+				)
+			)
+		)
+		(property "Footprint" "Resistor_SMD:R_0402_1005Metric_Pad0.72x0.64mm_HandSolder"
+			(at 243.84 131.572 90)
+			(effects
+				(font
+					(size 1.27 1.27)
+				)
+				(hide yes)
+			)
+		)
+		(property "Datasheet" "~"
+			(at 243.84 133.35 0)
+			(effects
+				(font
+					(size 1.27 1.27)
+				)
+				(hide yes)
+			)
+		)
+		(property "Description" "Resistor"
+			(at 243.84 133.35 0)
+			(effects
+				(font
+					(size 1.27 1.27)
+				)
+				(hide yes)
+			)
+		)
+		(pin "1"
+		)
+		(pin "2"
+		)
+		(instances
+			(project "coloryr"
+				(path "/9e6d55f4-a9e8-48fa-bb52-b4e4e3117f8b/d9c616e1-2298-455a-b24a-3007b8e9dd7b"
+					(reference "R91")
+					(unit 1)
+				)
+			)
+		)
+	)
+	(symbol
 		(lib_id "Diode:ESD9B5.0ST5G")
 		(at 81.28 135.89 90)
@@
 	(symbol
 		(lib_id "Device:C")
-		(at 228.6 130.81 90)
+		(at 228.6 144.78 90)
 		(unit 1)
 		(exclude_from_sim no)
@@
 		(dnp no)
 		(property "Reference" "C37"
-			(at 226.822 129.54 90)
+			(at 227.33 143.51 90)
 			(effects
 				(font
@@
 		)
 		(property "Value" "0.1uF"
-			(at 235.458 132.08 90)
+			(at 235.458 146.05 90)
 			(effects
 				(font
@@
 		)
 		(property "Footprint" "Capacitor_SMD:C_0402_1005Metric_Pad0.74x0.62mm_HandSolder"
-			(at 232.41 129.8448 0)
+			(at 232.41 143.8148 0)
 			(effects
 				(font
@@
 		)
 		(property "Datasheet" "~"
-			(at 228.6 130.81 0)
+			(at 228.6 144.78 0)
 			(effects
 				(font
@@
 		)
 		(property "Description" "Unpolarized capacitor"
-			(at 228.6 130.81 0)
+			(at 228.6 144.78 0)
 			(effects
 				(font
